File: Schematics/$ADAU1452.sch (KiCad schematic (older format))
At the start: 98 parts, among them CN201 COAX, P201 CONN_2x1, P202 CONN_2x1, P203 CONN_6X2, P204 CONN_6x1, SW201 SWITCH, SW202 SWITCH, U201 ADAU1452WBCPZ, U202 ADM13307-5ARZ, U203 25AA1024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

Commit message: PCB work
Parts:
- removed C225: 220u, OHDSP-Footprints-Pretty:SMD-0805, symbol CP1
- removed C240, C248: 220u, OHDSP-Footprints-Pretty:CAP-TH-D6.3mmP2.5mm, symbol CP1
- added C225, C240, C243: 22u, OHDSP-Footprints-Pretty:SMD-0805, symbol C
- C227: footprint OHDSP-Footprints-Pretty:SMD-0603 -> OHDSP-Footprints-Pretty:SMD-0805
- gave numbers to parts that had none: 1
Changed lines of the file:
@@
-$EndComp
-$Comp
-L CP1 C225
-U 1 1 54DB1F66
-P 7550 1650
-F 0 "C225" H 7600 1750 50  0000 L CNN
-F 1 "220u" H 7600 1550 50  0000 L CNN
-F 2 "OHDSP-Footprints-Pretty:SMD-0805" H 7550 1650 60  0000 C CNN
-F 3 "~" H 7550 1650 60  0000 C CNN
-	1    7550 1650
-	1    0    0    -1
 $EndComp
 $Comp
@@
 F 0 "C227" H 8200 1750 40  0000 L CNN
 F 1 "100n" H 8206 1565 40  0000 L CNN
-F 2 "OHDSP-Footprints-Pretty:SMD-0603" H 8238 1500 30  0000 C CNN
+F 2 "OHDSP-Footprints-Pretty:SMD-0805" H 8238 1500 30  0000 C CNN
 F 3 "~" H 8200 1650 60  0000 C CNN
 	1    8200 1650
@@
 $EndComp
 $Comp
-L CP1 C240
-U 1 1 54DB2FF5
-P 11850 1650
-F 0 "C240" H 11900 1750 50  0000 L CNN
-F 1 "220u" H 11900 1550 50  0000 L CNN
-F 2 "OHDSP-Footprints-Pretty:CAP-TH-D6.3mmP2.5mm" H 11850 1650 60  0000 C CNN
-F 3 "~" H 11850 1650 60  0000 C CNN
-	1    11850 1650
-	1    0    0    -1
-$EndComp
-$Comp
 L C C242
 U 1 1 54DB3007
@@
 F 3 "" H 14000 2200 60  0000 C CNN
 	1    14000 2200
-	1    0    0    -1
-$EndComp
-$Comp
-L CP1 C248
-U 1 1 54DB3C7D
-P 14350 1650
-F 0 "C248" H 14400 1750 50  0000 L CNN
-F 1 "220u" H 14400 1550 50  0000 L CNN
-F 2 "OHDSP-Footprints-Pretty:CAP-TH-D6.3mmP2.5mm" H 14350 1650 60  0000 C CNN
-F 3 "~" H 14350 1650 60  0000 C CNN
-	1    14350 1650
 	1    0    0    -1
 $EndComp
@@
 Connection ~ 14200 8600
 $Comp
-L R R?
+L R R233
 U 1 1 54F0DD27
 P 8700 10000
-F 0 "R?" V 8750 10300 40  0000 C CNN
+F 0 "R233" V 8750 10300 40  0000 C CNN
 F 1 "1k" V 8707 10001 40  0000 C CNN
 F 2 "OHDSP-Footprints-Pretty:SMD-0805" V 8630 10000 30  0001 C CNN
@@
 Wire Wire Line
 	8950 10000 9750 10000
+$Comp
+L C C240
+U 1 1 54F126E7
+P 11850 1650
+F 0 "C240" H 11850 1750 40  0000 L CNN
+F 1 "22u" H 11856 1565 40  0000 L CNN
+F 2 "OHDSP-Footprints-Pretty:SMD-0805" H 11888 1500 30  0000 C CNN
+F 3 "~" H 11850 1650 60  0000 C CNN
+	1    11850 1650
+	1    0    0    -1
+$EndComp
+$Comp
+L C C243
+U 1 1 54F127C8
+P 14350 1650
+F 0 "C243" H 14350 1750 40  0000 L CNN
+F 1 "22u" H 14356 1565 40  0000 L CNN
+F 2 "OHDSP-Footprints-Pretty:SMD-0805" H 14388 1500 30  0000 C CNN
+F 3 "~" H 14350 1650 60  0000 C CNN
+	1    14350 1650
+	1    0    0    -1
+$EndComp
+$Comp
+L C C225
+U 1 1 54F13D5F
+P 7550 1650
+F 0 "C225" H 7550 1750 40  0000 L CNN
+F 1 "22u" H 7556 1565 40  0000 L CNN
+F 2 "OHDSP-Footprints-Pretty:SMD-0805" H 7588 1500 30  0000 C CNN
+F 3 "~" H 7550 1650 60  0000 C CNN
+	1    7550 1650
+	1    0    0    -1
+$EndComp
 $EndSCHEMATC
