File: Schematics/OHDSP-ADAU1452.kicad_pcb (KiCad board)
At the start: 2 copper layers, 100 x 100 mm, 337 parts, among them CN201 COAX, CN401 COAX, CN402 COAX, CN403 COAX, CN404 COAX, CN405 COAX, CN406 COAX, CN407 COAX, CN408 COAX, P201 CONN_2x1, P202 CONN_2x1, P203 CONN_6X2, P204 CONN_6x1, P301 CONN_2x1, P302 CONN_2x1, P303 PIN, P304 PIN, P305 PIN, P306 PIN, P601 CONN_02X05, P602 CONN_02X05, P603 CONN_02X05, P604 CONN_02X05, P605 CONN_3x1, P606 CONN_6X2, P607 CONN_02X05, P608 CONN_02X05, P609 CONN_02X20, P610 CONN_02X05, P611 CONN_5x1, P613 CONN_02X05, P614 CONN_02X05, P615 CONN_02X05, P616 CONN_02X05, SW201 SWITCH, SW202 SWITCH, U201 ADAU1452WBCPZ, U202 ADM13307-5ARZ, U203 25AA1024, U301 IC-REG-XRP7659ISTR-F, U302 IC-REG-XRP7659ISTR-F, U303 XRP6272ITC5TR-F, U304 IC-REG-XC6210B332MR, U305 IC-REG-XC6210B332MR, U401 NB3L553, U402 NB3L553, U501 IC-SPDIF-RX-OPTO, U502 IC-SPDIF-TX-OPTO, X201 24M576

Commit message: Remove 1v2 LDO
Remove 1v2 LDO, not really needed...
Parts:
- removed C324, C332: 22u, OHDSP-Footprints-Pretty:SMD-0805
- removed C327: 1u, OHDSP-Footprints-Pretty:SMD-0805
- removed C336: 100n, OHDSP-Footprints-Pretty:SMD-0805
- removed C339: 220u, OHDSP-Footprints-Pretty:CAP-TH-D6.3mmP2.5mm
- removed R312: 100k, OHDSP-Footprints-Pretty:SMD-0805
- removed R315: 34k8, OHDSP-Footprints-Pretty:SMD-0805
- removed R316: 48k7, OHDSP-Footprints-Pretty:SMD-0805
- removed U303: XRP6272ITC5TR-F, OHDSP-Footprints-Pretty:IC-TO-252-5L
- C321: value 100n -> 1u
- moved C321 139.0 mm to (147.0, 70.0), turned to 90 degrees
- moved R301 118.8 mm to (144.5, 70.0), turned to 90 degrees
- moved C303 116.7 mm to (151.1, 74.0)
- moved C305 116.7 mm to (153.4, 74.0)
- moved C309 116.7 mm to (155.9, 67.6)
- moved C313 116.7 mm to (164.3, 71.4)
- moved C314 116.7 mm to (162.0, 71.5)
- moved C316 116.7 mm to (159.7, 71.4)
- moved D303 116.7 mm to (156.9, 74.7)
- moved L302 116.7 mm to (161.0, 64.0)
- moved R304 116.7 mm to (150.0, 64.5)
- moved R305 116.7 mm to (149.0, 67.5)
- moved U301 116.7 mm to (152.1, 69.7)
- moved C301 105.8 mm to (146.0, 75.0), turned to 270 degrees
- moved C304 78.0 mm to (148.5, 40.4)
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Connections:
- C313 pad 1: HT -> VDD
- C314 pad 1: HT -> VDD
- C316 pad 1: HT -> VDD
- C321 pad 1: HT -> Net-(C321-Pad1)
- L302 pad 2: HT -> VDD
- R301 pad 1: Net-(R301-Pad1) -> Net-(C321-Pad1)
- R301 pad 2: VCC -> VAA
- R304 pad 1: HT -> VDD
- R309 pad 1: HT -> VDD
- U301 pad 4: Net-(R301-Pad1) -> Net-(C321-Pad1)
Routing:
- net VCC: track 3.25 -> 0.00 mm

Commit message: Change ADAU1452 footprint, minor PCB changes
Parts:
- R305: value 51k -> 97k6
- U201: footprint OHDSP-Footprints-Pretty:IC-LFCSP72 -> OHDSP-Footprints-Pretty:IC-LFCSP72-HANDFIT
- moved L206 182.3 mm to (-30.5, 160.0)
- moved C249 135.7 mm to (-35.0, 172.0)
- moved C246 131.3 mm to (-45.0, 164.5)
- moved C247 125.4 mm to (-50.5, 171.5)
- moved C237 119.1 mm to (-103.4, 161.6)
- moved C238 119.1 mm to (-103.4, 166.7)
- moved XTAL201 99.9 mm to (-45.5, 158.5)
- moved CN201 91.2 mm to (-59.5, 172.5)
- moved R227 87.9 mm to (-80.5, 164.0)
- moved R230 79.5 mm to (-88.0, 157.5)
- moved X201 78.4 mm to (-90.5, 167.0)
- moved R233 75.2 mm to (-53.0, 161.0)
- moved R235 72.2 mm to (-43.0, 171.5)

Commit message: Rationalise the clock and clock fan-out schematics.
Rationalise the clock and clock fan-out schematics.
Removed one clock fan out buffer, still have 4 master audio clock
outputs. Also removed local crytsal oscialltor, a low jitter crystal
should perform as well, ADAU1452 has internal "dejittering" anyway.
Parts:
- removed C246: 10n, OHDSP-Footprints-Pretty:SMD-0805
- removed C247: 22u, OHDSP-Footprints-Pretty:SMD-0805
- removed C249: 100p, OHDSP-Footprints-Pretty:SMD-0805
- removed C406: 100n, OHDSP-Footprints-Pretty:SMD-0805
- removed CN403, CN404, CN407, CN408: COAX, OHDSP-Footprints-Pretty:CONN-RF-UFL
- removed L206: 600R@100MHz, OHDSP-Footprints-Pretty:SMD-0805
- removed R233: 0R, OHDSP-Footprints-Pretty:SMD-0805
- removed R235: 47R, OHDSP-Footprints-Pretty:SMD-0805
- removed R403: 75R, OHDSP-Footprints-Pretty:TH-RES-0W25
- removed R405: 1k, OHDSP-Footprints-Pretty:SMD-0805
- removed R410, R411, R412, R413: 27R, OHDSP-Footprints-Pretty:SMD-0805
- removed R416, R417, R420, R421: N/F, OHDSP-Footprints-Pretty:SMD-0805
- removed U402: NB3L553, OHDSP-Footprints-Pretty:IC_SOIC_8
- removed XTAL201: XTAL-OSC-4PIN, OHDSP-Footprints-Pretty:XTAL_5x3.2_4PIN
- moved C237 373.9 mm to (261.4, 79.5), turned to 180 degrees
- moved C238 371.2 mm to (257.4, 79.5)
- moved X201 360.0 mm to (259.4, 82.2), turned to 180 degrees
- moved R230 359.3 mm to (264.2, 86.0), turned to 45 degrees
- moved R227 347.2 mm to (258.1, 87.2), turned to 180 degrees
- moved R229 346.4 mm to (260.7, 85.1), turned to 180 degrees
- moved CN201 337.4 mm to (265.0, 80.1)
- moved R402 80.3 mm to (257.2, 93.5)
- moved C252 28.2 mm to (210.4, 118.0), turned to 0 degrees
- moved R231 25.1 mm to (215.5, 119.2), turned to 0 degrees
- moved P204 24.3 mm to (219.5, 122.5), turned to 180 degrees
- moved P608 22.4 mm to (234.5, 120.5)
- moved P607 22.4 mm to (234.5, 113.0)
- moved U203 20.3 mm to (213.0, 112.2), turned to 180 degrees
- moved R232 20.1 mm to (213.6, 112.9), turned to 90 degrees
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Connections:
- R229 pad 2: Net-(R229-Pad2) -> GNDD
Routing:
- net /ClockFanout/MCLKA1: track 12.7 -> 0.76 mm
- net /ClockFanout/MCLKC6: track 11.3 -> 0.00 mm
- net /ClockFanout/MCLKC7: track 11.2 -> 0.00 mm
- net /ClockFanout/MCLKB7: track 10.4 -> 0.00 mm
- net /ClockFanout/MCLKB6: track 10.1 -> 0.00 mm
- net /ADAU1452/XTALIN: track 0.00 -> 9.61 mm
- net /ADAU1452/XTALOUT: track 0.00 -> 8.53 mm
- net /ClockFanout/MCLKB5: track 8.32 -> 0.00 mm
- net /ClockFanout/MCLKB8: track 8.28 -> 0.00 mm
- net /ADAU1452/MCLK: track 13.2 -> 5.90 mm
- net /ClockFanout/MCLKC8: track 5.80 -> 0.00 mm
- net /ClockFanout/MCLKC5: track 5.76 -> 0.00 mm
- net Net-(CN201-Pad1): track 0.00 -> 4.19 mm
- net /ClockFanout/MCLKA2: track 3.78 -> 0.00 mm

Commit message: PCB work
Parts:
- moved C507 640.2 mm to (288.5, 71.1), turned to 90 degrees
- moved R503 637.7 mm to (286.0, 71.1), turned to 90 degrees
- moved R633 550.2 mm to (248.5, 82.0)
- moved R632 544.5 mm to (248.5, 79.0)
- moved R631 544.4 mm to (248.5, 76.0)
- moved R630 529.4 mm to (233.5, 76.5), turned to 90 degrees
- moved R629 526.9 mm to (231.0, 76.5), turned to 90 degrees
- moved R643 508.4 mm to (245.5, 66.7)
- moved R207 106.2 mm to (230.9, 99.4)
- moved R208 105.8 mm to (230.9, 101.9)
- moved R210 98.0 mm to (230.9, 105.9)
- moved R209 97.8 mm to (230.9, 103.9)
- moved R214 84.5 mm to (237.0, 107.4)
- moved R213 82.5 mm to (237.0, 104.4)
- moved R211 82.2 mm to (242.0, 108.4)
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Routing:
- net /Connectors/RPI_BCLK: track 0.00 -> 28.4 mm
- net Net-(R211-Pad2): track 0.00 -> 25.1 mm
- net Net-(R207-Pad2): track 0.00 -> 23.2 mm
- net Net-(R209-Pad2): track 0.00 -> 22.8 mm
- net /ADAU1452/ADAU_SPDIF_RX: track 0.00 -> 22.1 mm
- net Net-(R212-Pad2): track 0.00 -> 20.9 mm
- net /ADAU1452/ADAU_SPDIF_TX: track 0.00 -> 20.8 mm
- net /ADAU1452/M_MISO: track 0.00 -> 20.4 mm
- net /ADAU1452/M_SCLK: track 0.00 -> 20.3 mm
- net /ADAU1452/M_MOSI: track 0.00 -> 20.1 mm
- net /ADAU1452/M_SS: track 0.00 -> 20.0 mm
- net Net-(P609-Pad23): track 0.00 -> 12.8 mm
- net Net-(C507-Pad2): track 0.00 -> 11.8 mm
- net Net-(P609-Pad21): track 0.00 -> 8.78 mm
- net Net-(R503-Pad2): track 0.00 -> 7.15 mm
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Other:
- board text added: "This is the BCLK for the Pi - high speed.... Route carefully"

Commit message: Going 4 layer on small PCB
Going 4 layer on small PCB
Parts:
- D301, D302, R641: moved to B.Cu
- moved D301 6.54 mm to (223.0, 66.8), turned to 180 degrees
- moved C308 5.14 mm to (213.4, 76.6)
- moved C312 5.14 mm to (211.2, 76.6)
- moved C307 5.14 mm to (207.2, 79.7)
- moved C311 5.14 mm to (215.9, 76.7)
- moved L301 5.14 mm to (207.2, 71.7)
- moved R303 5.14 mm to (207.2, 75.7)
- moved D302 4.22 mm to (213.1, 66.8), turned to 180 degrees
- moved C235 0.92 mm to (283.7, 99.4)
- moved P301 0.48 mm to (223.5, 63.0)
- moved P302 0.39 mm to (213.1, 63.0)
- moved R641 0.11 mm to (228.6, 67.1)
Routing:
- net /ADAU1452/DVDD: track 3.81 -> 12.7 mm, vias 0 -> 1
- net /ADAU1452/IOVDD: track 10.0 -> 17.4 mm, vias 0 -> 1
Other:
- copper layers 2 -> 4
- net class 100ohm: clearance 0.1 -> 0.1524
- net class Default: clearance 0.1 -> 0.1524
- rule trace_clearance: 0.1 -> 0.1524
- board text added: "Lets go 4 layer and more SPI/I2C to back"

Commit message: PCB work
Parts:
- C303, C304, C305, C306, C307, C309, C310, C321, D303, D304, L301, R207, R208, R209, R210, R211, R212, R213, R214, R215, R216, R301, R302, R303, R304, R305, R306, R307, R308, U301, U302: moved to B.Cu
- C313, C315, C316, C319: moved to F.Cu
- moved R307 98.7 mm to (212.9, 104.9)
- moved R306 98.6 mm to (216.7, 104.9)
- moved R308 97.6 mm to (210.6, 102.9), turned to 180 degrees
- moved C310 91.1 mm to (213.6, 101.6)
- moved L303 88.8 mm to (217.7, 97.8), turned to 90 degrees
- moved U302 87.8 mm to (210.1, 99.6)
- moved R302 83.0 mm to (201.2, 96.5), turned to 90 degrees
- moved C304 81.4 mm to (209.8, 94.0), turned to 180 degrees
- moved C306 81.1 mm to (209.8, 96.0), turned to 180 degrees
- moved D304 78.6 mm to (213.4, 94.0), turned to 270 degrees
- moved C319 78.4 mm to (211.3, 96.0), turned to 180 degrees
- moved C317 75.8 mm to (215.1, 90.7), turned to 180 degrees
- moved C315 73.6 mm to (211.3, 94.0), turned to 180 degrees
- moved R304 67.4 mm to (213.6, 86.9)
- moved C301 64.2 mm to (208.5, 89.4), turned to 0 degrees
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Routing:
- net Net-(R211-Pad2): track 25.1 -> 0.00 mm
- net Net-(R207-Pad2): track 23.2 -> 0.00 mm
- net Net-(R209-Pad2): track 22.8 -> 0.00 mm
- net Net-(R212-Pad2): track 20.9 -> 0.00 mm
Other:
- rule via_min_drill: 0.5 -> 0.3
- rule via_min_size: 0.9 -> 0.6

Commit message: PCB work
Parts:
- C207, C210, C213, C219, C228, C230, C233, C235, C241, C250, C325, C326, C328, C329, C330, C331, R313, R314, R629, R630, R631, R632, R633, U304, U305: moved to B.Cu
- C321, R301: moved to F.Cu
- moved P610 545.0 mm to (241.0, 80.5), turned to 90 degrees
- moved C250 434.3 mm to (273.8, 87.1), turned to 270 degrees
- moved C241 409.5 mm to (270.0, 87.1), turned to 270 degrees
- moved C325 52.0 mm to (222.9, 89.2), turned to 90 degrees
- moved C328 51.9 mm to (225.2, 89.2), turned to 90 degrees
- moved C326 51.4 mm to (222.9, 95.5), turned to 90 degrees
- moved C329 51.1 mm to (225.0, 95.5), turned to 90 degrees
- moved C335 50.6 mm to (232.0, 95.1)
- moved C338 50.6 mm to (236.5, 95.1)
- moved C341 50.6 mm to (234.5, 95.1)
- moved U305 50.6 mm to (228.5, 95.1), turned to 90 degrees
- moved C334 50.6 mm to (232.5, 87.1)
- moved C337 50.6 mm to (236.5, 87.1)
- moved C340 50.6 mm to (234.5, 87.1)
- moved U304 50.6 mm to (228.5, 87.6), turned to 90 degrees
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Routing:
- net VCC: track 0.00 -> 46.5 mm
- net /ADAU1452/I2C_SCL: track 0.00 -> 41.3 mm
- net /ADAU1452/I2C_SDA: track 0.00 -> 36.7 mm
- net /ADAU1452/M_MISO: track 20.4 -> 49.9 mm
- net /ADAU1452/M_SCLK: track 20.3 -> 49.1 mm
- net /ADAU1452/M_MOSI: track 20.1 -> 48.3 mm
- net /ADAU1452/M_SS: track 20.0 -> 47.4 mm
- net /ADAU1452/SPI_SCLK: track 0.00 -> 26.7 mm
- net Net-(C315-Pad1): track 0.00 -> 26.5 mm
- net /ADAU1452/SPI_MISO: track 0.00 -> 24.9 mm
- net Net-(R209-Pad2): track 0.00 -> 15.7 mm, vias 0 -> 1
- net Net-(P609-Pad23): track 12.8 -> 0.00 mm
- net Net-(R207-Pad2): track 0.00 -> 10.9 mm, vias 0 -> 1
- net GNDD: track 0.00 -> 10.5 mm
- net Net-(P609-Pad21): track 8.78 -> 0.00 mm
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Other:
- board text removed: "Lets go 4 layer and more SPI/I2C to back"

Commit message: PCB work
Parts:
- added C243: 22u, OHDSP-Footprints-Pretty:SMD-0805, F.Cu at (255.0, 134.1)
- added R233: 1k, OHDSP-Footprints-Pretty:SMD-0805, B.Cu at (205.7, 159.3)
- added R642: 0R, OHDSP-Footprints-Pretty:SMD-0805, B.Cu at (240.4, 95.0)
- C203, C214, C216, C218, C224, C226, C231, L201, L202, L203, R204, R206, R218, R219, R220, R222, R223, R224, R225, R226, U202: moved to B.Cu
- C225: value 220u -> 22u; moved to B.Cu
- C227: footprint OHDSP-Footprints-Pretty:SMD-0603 -> OHDSP-Footprints-Pretty:SMD-0805; moved to B.Cu
- C240: value 220u -> 22u; footprint OHDSP-Footprints-Pretty:CAP-TH-D6.3mmP2.5mm -> OHDSP-Footprints-Pretty:SMD-0805
- moved R644 511.6 mm to (248.4, 80.3), turned to 270 degrees
- moved L203 456.1 mm to (259.3, 106.4), turned to 90 degrees
- moved C224 398.1 mm to (261.4, 106.4), turned to 270 degrees
- moved C225 393.5 mm to (258.3, 101.6), turned to 180 degrees
- moved C226 392.1 mm to (258.3, 99.6), turned to 180 degrees
- moved C227 391.4 mm to (257.6, 104.6), turned to 270 degrees
- moved L202 385.7 mm to (201.4, 155.1)
- moved C216 375.0 mm to (210.2, 148.1), turned to 90 degrees
- moved C214 351.6 mm to (200.4, 149.6), turned to 90 degrees
- moved C218 350.3 mm to (202.7, 149.8), turned to 90 degrees
- moved SW202 348.3 mm to (201.3, 183.0)
- moved C231 334.2 mm to (207.4, 163.4)
- moved R225 330.7 mm to (260.4, 103.6)
- moved U202 300.8 mm to (204.4, 146.5), turned to 270 degrees
- moved R206 282.9 mm to (201.4, 152.7), turned to 180 degrees
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Connections:
- P607 pad 7: /ADAU1452/I2C_SDA -> Net-(P607-Pad7)
- P608 pad 7: /ADAU1452/I2C_SDA -> Net-(P607-Pad7)
- R226 pad 1: /ADAU1452/RESET -> GNDD
- R226 pad 2: GNDD -> /ADAU1452/RESET
- U202 pad 7: Net-(C231-Pad1) -> Net-(R233-Pad1)
Routing:
- net /ADAU1452/DVDD: track 12.2 -> 78.3 mm, vias 0 -> 1
- net /ADAU1452/IOVDD: track 14.2 -> 78.1 mm
- net VDD: track 0.00 -> 41.7 mm, vias 0 -> 1
- net VPP: track 0.00 -> 32.9 mm, vias 0 -> 1
- net /ADAU1452/I2C_SCL: track 41.3 -> 72.1 mm
- net Net-(P607-Pad7): track 0.00 -> 28.0 mm
- net Net-(C315-Pad1): track 26.5 -> 6.70 mm
- net Net-(P609-Pad23): track 0.00 -> 17.7 mm
- net Net-(P609-Pad21): track 0.00 -> 16.3 mm
- net /ADAU1452/XTALIN: track 12.5 -> 26.1 mm
- net Net-(R220-Pad2): track 0.00 -> 11.2 mm
- net Net-(R219-Pad2): track 0.00 -> 8.41 mm
- net Net-(R218-Pad2): track 0.00 -> 7.54 mm
- net /ClockFanout/MCLKB1: track 9.50 -> 2.61 mm
- net /ClockFanout/MCLKB4: track 9.45 -> 2.74 mm
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