File: Schematics/OHDSP-ADAU1701.sch (KiCad schematic (older format))
At the start: 0 parts

Commit message: WIP
Connections:
- net labels added: ANA_IN1, ANA_IN2, ANA_OUT1, ANA_OUT2, ANA_OUT3, ANA_OUT4, GLB_RESET, MCLK1, MCLK2, MCLK3
- net labels removed: MCLK
- wire segments 33 -> 53
