File: Schematics/ADAU1701.sch (KiCad schematic (older format))
At the start: 99 parts, among them CN201 COAX, P201 CONN_2x1, P203 CONN_6X2, P204 CONN_6x1, SW202 SWITCH, U201 ADAU1452WBCPZ, U202 ADM13307-5ARZ, U203 25AA1024, X201 24M576

Commit message: Adding ADAU1701 version
Because its easier...
Parts:
- removed C213, C219, C230, C233, C235: 1u, OHDSP-Footprints-Pretty:SMD-0603, symbol C
- removed C215, C220, C232, C234, C236: 100n, OHDSP-Footprints-Pretty:SMD-0603, symbol C
- removed C217, C223: 10n, OHDSP-Footprints-Pretty:SMD-0603, symbol C
- removed U201: ADAU1452WBCPZ, OHDSP-Footprints-Pretty:IC-LFCSP72-HANDFIT, symbol IC-DSP-ADAU1452WBCPZ
- added C? (x2): 1u, OHDSP-Footprints-Pretty:SMD-0603, symbol C
- added C? (x2): 100n, OHDSP-Footprints-Pretty:SMD-0603, symbol C
- added R?: 7k5, OHDSP-Footprints-Pretty:SMD-0805, symbol R
- added U?: IC-DSP-ADAU1701JSTZ, symbol IC-DSP-ADAU1701JSTZ
Connections:
- net labels added: ANAIN0, ANAIN1, ANAVOUT0, ANAVOUT1, ANAVOUT2, ANAVOUT3
- net labels removed: ADAU_SPDIF_RX, ADAU_SPDIF_TX, ADCIN_BCLK1, ADCIN_BCLK2, ADCIN_BCLK3, ADCIN_LRCLK1, ADCIN_LRCLK2, ADCIN_LRCLK3, AUXADC_IN1, AUXADC_IN2, AUXADC_IN3, AUXADC_IN4, AUXADC_IN5, AUXADC_IN6, DACOUT_BCLK1, DACOUT_BCLK2, DACOUT_BCLK3, DACOUT_LRCLK1, DACOUT_LRCLK2, DACOUT_LRCLK3
- wire segments 327 -> 285
Other:
- moved on the sheet: C202, C221, C222, C224, C225, C226, C227, C228, C229, C239, C240, C241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

Commit message: WIP
Parts:
- removed P203: CONN_6X2, OHDSP-Footprints-Pretty:CONN_DIL_2X6, symbol CONN_6X2
- removed P204: CONN_6x1, OHDSP-Footprints-Pretty:CONN_SIL_6, symbol CONN_6x1
- removed R231, R232: 10k, OHDSP-Footprints-Pretty:SMD-0805, symbol R
- removed U203: 25AA1024, OHDSP-Footprints-Pretty:IC_DIP_8, symbol IC-EEPROM-SPI
- added U?: IC-EEPROM-I2C, symbol IC-EEPROM-I2C
Connections:
- net labels removed: EE_SO, EE_~CS, SPI_MISO, SPI_MOSI, SPI_SCLK, SPI_~CS
- wire segments 285 -> 247
Other:
- note added: "I2C Interface"
- note removed: "Allow choosing\nbetween the two\nfor Raspberry Pi\nor Arduino"
- note removed: "Allow for self boot\nUses master SPI"
- note removed: "Jumpers to allow \nexternal programming\n"
- note removed: "Programming\nHeader\n"
- note removed: "SPI"
- note removed: "SPI EEPROM"
- note removed: "Slave SPI and I2C"
- note removed: "Slave SPI/I2C"
- moved on the sheet: C201, C252, C254, R202, R203, R221, R235, R?, U?

Commit message: WIP
Connections:
- net labels added: ADC_IN0, ADC_IN1, DAC_VOUT0, DAC_VOUT1, DAC_VOUT2, DAC_VOUT3
- net labels removed: ANAIN0, ANAIN1, ANAVOUT0, ANAVOUT1, ANAVOUT2, ANAVOUT3
- wire segments 247 -> 253
Changed lines of the file:
@@
 $Descr A3 16535 11693
 encoding utf-8
-Sheet 2 6
+Sheet 2 5
 Title ""
 Date "10 feb 2015"
@@
 Connection ~ 9950 7200
 Text HLabel 11050 4300 2    60   Output ~ 0
-ANAVOUT0
+DAC_VOUT0
 Text HLabel 11050 4450 2    60   Output ~ 0
-ANAVOUT1
+DAC_VOUT1
 Text HLabel 11050 4600 2    60   Output ~ 0
-ANAVOUT2
+DAC_VOUT2
 Text HLabel 11050 4750 2    60   Output ~ 0
-ANAVOUT3
+DAC_VOUT3
 Text HLabel 8250 4300 0    60   Input ~ 0
-ANAIN0
+ADC_IN0
 Text HLabel 8250 4450 0    60   Input ~ 0
-ANAIN1
+ADC_IN1
 $Comp
 L R R?
@@
 	1    0    0    -1
 $EndComp
+Wire Wire Line
+	8250 4300 8350 4300
+Wire Wire Line
+	8350 4450 8250 4450
+Wire Wire Line
+	10850 4300 11050 4300
+Wire Wire Line
+	11050 4450 10850 4450
+Wire Wire Line
+	10850 4600 11050 4600
+Wire Wire Line
+	11050 4750 10850 4750
 $EndSCHEMATC

Commit message: WIP
Parts:
- removed C237, C238: 33p, OHDSP-Footprints-Pretty:SMD-0603, symbol C
- removed CN201: COAX, OHDSP-Footprints-Pretty:CONN-RF-UFL, symbol COAX
- removed R227: 100R, OHDSP-Footprints-Pretty:SMD-0805, symbol R
- removed R229, R230: N/F, OHDSP-Footprints-Pretty:SMD-0805, symbol R
- removed X201: 24M576, OHDSP-Footprints-Pretty:XTAL_HC49_TH, symbol CRYSTAL
- added R216: 0R, symbol R
- added TP201: TP, symbol PIN
- C201, L201, L202, L203, L204, L205, R201, R202, R203, R204, R205: footprint OHDSP-Footprints-Pretty:SMD-0805 -> (none)
- C202: renamed from C203; footprint OHDSP-Footprints-Pretty:SMD-0805 -> (none)
- C203: renamed from C204; footprint OHDSP-Footprints-Pretty:CAP-TH-D6.3mmP2.5mm -> (none)
- C204: renamed from C205; footprint OHDSP-Footprints-Pretty:SMD-0805 -> (none)
- C205: renamed from C206; footprint OHDSP-Footprints-Pretty:SMD-0805 -> (none)
- C206: renamed from C207; footprint OHDSP-Footprints-Pretty:SMD-0603 -> (none)
- C207: renamed from C208; footprint OHDSP-Footprints-Pretty:SMD-0603 -> (none)
- C208: renamed from C209; footprint OHDSP-Footprints-Pretty:SMD-0603 -> (none)
- C209: renamed from C210; footprint OHDSP-Footprints-Pretty:SMD-0603 -> (none)
- C210: renamed from C211; footprint OHDSP-Footprints-Pretty:SMD-0603 -> (none)
- C211: renamed from C212; footprint OHDSP-Footprints-Pretty:SMD-0603 -> (none)
- C212: renamed from C214; footprint OHDSP-Footprints-Pretty:SMD-0805 -> (none)
- C213: renamed from C216; footprint OHDSP-Footprints-Pretty:SMD-0805 -> (none)
- C214: renamed from C252; footprint OHDSP-Footprints-Pretty:SMD-0805 -> (none)
- C215: renamed from C218; footprint OHDSP-Footprints-Pretty:SMD-0805 -> (none)
- C216: renamed from C254; footprint OHDSP-Footprints-Pretty:SMD-0805 -> (none)
- C217: renamed from C224; footprint OHDSP-Footprints-Pretty:SMD-0805 -> (none)
- C218: renamed from C225; footprint OHDSP-Footprints-Pretty:SMD-0805 -> (none)
- C219: renamed from C226; footprint OHDSP-Footprints-Pretty:SMD-0805 -> (none)
- C220: renamed from C227; footprint OHDSP-Footprints-Pretty:SMD-0805 -> (none)
- C221: renamed from C228; footprint OHDSP-Footprints-Pretty:SMD-0603 -> (none)
- C222: renamed from C229; footprint OHDSP-Footprints-Pretty:SMD-0603 -> (none)
- C223: renamed from C231; footprint OHDSP-Footprints-Pretty:SMD-0805 -> (none)
- C224: renamed from C246; footprint OHDSP-Footprints-Pretty:SMD-0805 -> (none)
- C225: renamed from C239; footprint OHDSP-Footprints-Pretty:SMD-0805 -> (none)
- C226: renamed from C240; footprint OHDSP-Footprints-Pretty:SMD-0805 -> (none)
- C227: renamed from C244; footprint OHDSP-Footprints-Pretty:SMD-0805 -> (none)
- C228: renamed from C241; footprint OHDSP-Footprints-Pretty:SMD-0805 -> (none)
- C229: renamed from C242; footprint OHDSP-Footprints-Pretty:SMD-0603 -> (none)
- C230: renamed from C202; footprint OHDSP-Footprints-Pretty:CAP-TH-D6.3mmP2.5mm -> (none)
- C231: renamed from C245; footprint OHDSP-Footprints-Pretty:SMD-0805 -> (none)
- C232: renamed from C243; footprint OHDSP-Footprints-Pretty:SMD-0805 -> (none)
- C233: renamed from C250; footprint OHDSP-Footprints-Pretty:SMD-0805 -> (none)
- C234: renamed from C251; footprint OHDSP-Footprints-Pretty:SMD-0603 -> (none)
- C235, C236, C237, C238: renamed from C?; footprint OHDSP-Footprints-Pretty:SMD-0603 -> (none)
- C239: renamed from C221; footprint OHDSP-Footprints-Pretty:SMD-0603 -> (none)
- C240: renamed from C222; footprint OHDSP-Footprints-Pretty:SMD-0603 -> (none)
- P201: footprint OHDSP-Footprints-Pretty:CONN_SIL_2 -> (none)
- R206: renamed from R235; footprint OHDSP-Footprints-Pretty:SMD-0805 -> (none)
- R207: renamed from R206; footprint OHDSP-Footprints-Pretty:SMD-0805 -> (none)
- R208: renamed from R225; footprint OHDSP-Footprints-Pretty:SMD-0805 -> (none)
- R209: renamed from R218; footprint OHDSP-Footprints-Pretty:SMD-0805 -> (none)
- R210: renamed from R219; footprint OHDSP-Footprints-Pretty:SMD-0805 -> (none)
- R211: renamed from R220; value 3k3 -> 8k2; footprint OHDSP-Footprints-Pretty:SMD-0805 -> (none)
- R212: renamed from R222; footprint OHDSP-Footprints-Pretty:SMD-0805 -> (none)
- R213: renamed from R223; footprint OHDSP-Footprints-Pretty:SMD-0805 -> (none)
- R214: renamed from R224; value 3k6 -> 4k7; footprint OHDSP-Footprints-Pretty:SMD-0805 -> (none)
- R215: renamed from R?; footprint OHDSP-Footprints-Pretty:SMD-0805 -> (none)
- R217: renamed from R233; footprint OHDSP-Footprints-Pretty:SMD-0805 -> (none)
- R218: renamed from R228; footprint OHDSP-Footprints-Pretty:SMD-0805 -> (none)
- R219: renamed from R226; footprint OHDSP-Footprints-Pretty:SMD-0805 -> (none)
- R220: renamed from R221; footprint OHDSP-Footprints-Pretty:SMD-0805 -> (none)
- R221: renamed from R234; footprint OHDSP-Footprints-Pretty:SMD-0805 -> (none)
- R222: renamed from R207; footprint OHDSP-Footprints-Pretty:SMD-0805 -> (none)
- R223: renamed from R208; footprint OHDSP-Footprints-Pretty:SMD-0805 -> (none)
- R224: renamed from R209; footprint OHDSP-Footprints-Pretty:SMD-0805 -> (none)
- R225: renamed from R210; footprint OHDSP-Footprints-Pretty:SMD-0805 -> (none)
- R226: renamed from R211; footprint OHDSP-Footprints-Pretty:SMD-0805 -> (none)
- R227: renamed from R212; footprint OHDSP-Footprints-Pretty:SMD-0805 -> (none)
- R228: renamed from R213; footprint OHDSP-Footprints-Pretty:SMD-0805 -> (none)
- R229: renamed from R214; footprint OHDSP-Footprints-Pretty:SMD-0805 -> (none)
- R230: renamed from R215; footprint OHDSP-Footprints-Pretty:SMD-0805 -> (none)
- R231: renamed from R216; footprint OHDSP-Footprints-Pretty:SMD-0805 -> (none)
- R232: renamed from R217; footprint OHDSP-Footprints-Pretty:SMD-0603 -> (none)
- SW201: renamed from SW202; footprint OHDSP-Footprints-Pretty:SW_TACT_SMD -> (none)
- U202: footprint OHDSP-Footprints-Pretty:IC_SOIC_8 -> (none)
- gave numbers to parts that had none: 2
Connections:
- wire segments 253 -> 243
- no-connect marks 5 -> 4
Other:
- note added: "USE 0.1% RESISTORS\n\nSENSE2 Vmin=2.973V\nSENSE3 Vmin=1.632V"
- note removed: "External Clock"
- note removed: "Master Clock - Two Options"
- note removed: "Standard Crystal"
- note removed: "USE 0.1% RESISTORS\n\nSENSE2 Vmin=2.973\nSENSE3 Vmin=1.1396"

Commit message: WIP
Parts:
- removed R205: N/F, symbol R
- added R? (x4): 0R, symbol R
- added R? (x2): 1k, symbol R
- added R? (x2): N/F, symbol R
- U203: value IC-DSP-ADAU1701JSTZ -> ADAU1701JSTZ
Connections:
- net labels added: ADDR0, ADDR1, RST_IN, RST_OUT
- net labels removed: EE_SCK, EE_SI, MRST
- wire segments 243 -> 273
Other:
- note added: "I2C Address"
- note added: "Selfboot EEPROM"
- note added: "Selfboot Select"
- note removed: "Manual Control Switches"
- note removed: "SPI/I2C Select:\nSet SPI or I2C for selfboot\n10kR to 0V is I2C\nOpen is SPI"
- moved on the sheet: C201, C212, C213, C214, C215, C216, C223, C224, C227, L202, P201, R201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

Commit message: WIP
Parts:
- added R?: 1k, symbol R
- added R? (x2): 10k, symbol R
- added TR?: TRAN-NPN-BC847, symbol TRAN-NPN-BC847
- added TR? (x2): TRAN-PNP-BC857, symbol TRAN-PNP-BC857
Connections:
- net labels added: RST_IN1, RST_IN2
- net labels removed: RST_IN
- wire segments 273 -> 379

Commit message: WIP
Parts:
- added R? (x2): 100k, symbol R
Connections:
- wire segments 379 -> 293
Other:
- moved on the sheet: R?

Commit message: WIP
Parts:
- TR?: value TRAN-NPN-BC847 -> BC847
- TR? (x2): value TRAN-PNP-BC857 -> BC857
Connections:
- wire segments 293 -> 390
Other:
- moved on the sheet: R?, TR?
