File: Schematics/ADAU1701.sch (KiCad schematic (older format))
At the start: 98 parts, among them P201 CONN_2x1, SW201 SWITCH, U201 IC-EEPROM-I2C, U202 ADM13307-5ARZ, U203 ADAU1701JSTZ

Commit message: WIP
Parts:
- added C? (x3): 220u, symbol CP1
- added C? (x3): 100n, symbol C
- added C?: 10u, symbol C
- added C? (x2): 10v, symbol C
- added C?: 3n3, symbol C
- added C?: 56n, symbol C
- added R?: 475R, symbol R
- added R? (x2): 1k, symbol R
- added R? (x2): N/F, symbol R
- added R?: 0R, symbol R
- added TP?: TP, symbol PIN
Connections:
- net labels added: CM, FILTA, FILTD, PLL0, PLL1
- wire segments 390 -> 343
Other:
- note added: "Default 256xfs"
- note added: "Filters"
- note added: "PLL Mode"
- moved on the sheet: P201, R201, R?

Commit message: WIP
Parts:
- removed C239: 5n6, symbol C
- removed C240: 150p, symbol C
- removed R222, R223, R224, R225, R228, R229: 0R, symbol R
- removed R226, R227, R230, R231: N/F, symbol R
- removed R232: 4k3, symbol R
- C201, C202, C205, C206, C207, C210, C211, C212, C223, C224: renamed from C?; footprint (none) -> OHDSP-Footprints-Pretty:SMD-0805
- C203: renamed from C?; footprint (none) -> OHDSP-Footprints-Pretty:CAP-TH-D6.3mmP2.5mm
- C204: renamed from C202; footprint (none) -> OHDSP-Footprints-Pretty:SMD-0805
- C208: renamed from C203; footprint (none) -> OHDSP-Footprints-Pretty:SMD-0805
- C209: renamed from C212; footprint (none) -> OHDSP-Footprints-Pretty:SMD-0805
- C213, C215, L201, L202, L203, L204, L205: footprint (none) -> OHDSP-Footprints-Pretty:SMD-0805
- C214: renamed from C204; footprint (none) -> OHDSP-Footprints-Pretty:SMD-0805
- C216: renamed from C205; footprint (none) -> OHDSP-Footprints-Pretty:SMD-0805
- C217: renamed from C206; footprint (none) -> OHDSP-Footprints-Pretty:SMD-0805
- C218: renamed from C207; footprint (none) -> OHDSP-Footprints-Pretty:SMD-0805
- C219: renamed from C208; footprint (none) -> OHDSP-Footprints-Pretty:SMD-0805
- C220: renamed from C209; footprint (none) -> OHDSP-Footprints-Pretty:SMD-0805
- C221: renamed from C210; footprint (none) -> OHDSP-Footprints-Pretty:SMD-0805
- C222: renamed from C211; footprint (none) -> OHDSP-Footprints-Pretty:SMD-0805
- C225: renamed from C217; footprint (none) -> OHDSP-Footprints-Pretty:SMD-0805
- C226: renamed from C223; footprint (none) -> OHDSP-Footprints-Pretty:SMD-0805
- C227: renamed from C218; footprint (none) -> OHDSP-Footprints-Pretty:SMD-0805
- C228: renamed from C224; footprint (none) -> OHDSP-Footprints-Pretty:SMD-0805
- C229: renamed from C219; footprint (none) -> OHDSP-Footprints-Pretty:SMD-0805
- C230: renamed from C220; footprint (none) -> OHDSP-Footprints-Pretty:CAP-TH-D6.3mmP2.5mm
- C231: renamed from C221; footprint (none) -> OHDSP-Footprints-Pretty:SMD-0805
- C232: renamed from C227; footprint (none) -> OHDSP-Footprints-Pretty:SMD-0805
- C233: renamed from C222; footprint (none) -> OHDSP-Footprints-Pretty:SMD-0805
- C234: renamed from C225; footprint (none) -> OHDSP-Footprints-Pretty:SMD-0805
- C235: renamed from C226; footprint (none) -> OHDSP-Footprints-Pretty:SMD-0805
- C236: renamed from C228; footprint (none) -> OHDSP-Footprints-Pretty:SMD-0805
- C237: renamed from C229; footprint (none) -> OHDSP-Footprints-Pretty:SMD-0805
- C238: renamed from C230; footprint (none) -> OHDSP-Footprints-Pretty:SMD-0805
- C239: renamed from C231; footprint (none) -> OHDSP-Footprints-Pretty:SMD-0805
- C240: renamed from C232; footprint (none) -> OHDSP-Footprints-Pretty:SMD-0805
- P201: footprint (none) -> OHDSP-Footprints-Pretty:CONN_SIL_2
- R201: renamed from R204; footprint (none) -> OHDSP-Footprints-Pretty:SMD-0805
- R202: renamed from R207; footprint (none) -> OHDSP-Footprints-Pretty:SMD-0805
- R203: renamed from R209; footprint (none) -> OHDSP-Footprints-Pretty:SMD-0805
- R204: renamed from R210; footprint (none) -> OHDSP-Footprints-Pretty:SMD-0805
- R205: renamed from R211; footprint (none) -> OHDSP-Footprints-Pretty:SMD-0805
- R206: renamed from R212; footprint (none) -> OHDSP-Footprints-Pretty:SMD-0805
- R207: renamed from R213; footprint (none) -> OHDSP-Footprints-Pretty:SMD-0805
- R208: renamed from R214; footprint (none) -> OHDSP-Footprints-Pretty:SMD-0805
- R209, R210, R216, R218, R219, R221, R222, R223, R226, R227, R228, R229, R230, R231, R232: renamed from R?; footprint (none) -> OHDSP-Footprints-Pretty:SMD-0805
- R211: renamed from R215; footprint (none) -> OHDSP-Footprints-Pretty:SMD-0805
- R212: renamed from R208; footprint (none) -> OHDSP-Footprints-Pretty:SMD-0805
- R213: renamed from R216; footprint (none) -> OHDSP-Footprints-Pretty:SMD-0805
- R214: renamed from R217; footprint (none) -> OHDSP-Footprints-Pretty:SMD-0805
- R215: renamed from R219; footprint (none) -> OHDSP-Footprints-Pretty:SMD-0805
- R217: renamed from R220; footprint (none) -> OHDSP-Footprints-Pretty:SMD-0805
- R220: renamed from R218; footprint (none) -> OHDSP-Footprints-Pretty:SMD-0805
- R224: renamed from R201; footprint (none) -> OHDSP-Footprints-Pretty:SMD-0805
- R225: renamed from R221; footprint (none) -> OHDSP-Footprints-Pretty:SMD-0805
- SW201: footprint (none) -> OHDSP-Footprints-Pretty:SW_TACT_SMD
- U201: renamed from U202; footprint (none) -> OHDSP-Footprints-Pretty:IC_DIP_8
- U202: renamed from U203; footprint (none) -> OHDSP-Footprints-Pretty:IC_SOIC_8
- U203: renamed from U201; footprint (none) -> OHDSP-Footprints-Pretty:IC-LQFP48_7x7
- gave numbers to parts that had none: 8
- renumbered C233 to C241, C234 to C242, C235 to C243, C236 to C244, C237 to C245, C238 to C246, C214 to C247, C216 to C248, C201 to C249, R206 to R233, R203 to R236, R202 to R237, TP201 to TP202
Connections:
- net labels removed: MCLK_ADAU, M_MISO, M_MOSI, M_SCLK, M_SS, SL_MISO, SL_MOSI, SL_SCLK, SL_~SS, XTALIN, XTALOUT
- wire segments 343 -> 295
- no-connect marks 4 -> 0
Other:
- note removed: "Audio Master Clock Output"

Commit message: WIP
Parts:
- C201, C202, C208, C238: footprint OHDSP-Footprints-Pretty:SMD-0805 -> OHDSP-Footprints-Pretty:CAP-TH-D6.3mmP2.5mm
- C206, C207: value 10v -> 10u
- C230: footprint OHDSP-Footprints-Pretty:CAP-TH-D6.3mmP2.5mm -> OHDSP-Footprints-Pretty:SMD-0805
- C241, C242, C243, C244, C245, C246, C247, C248, C249, R233, R234, R235, R236, R237, R238, R239: footprint (none) -> OHDSP-Footprints-Pretty:SMD-0805
- TP201, TP202: footprint (none) -> OHDSP-Footprints-Pretty:TP-2mm
- TR201, TR202, TR203: footprint (none) -> OHDSP-Footprints-Pretty:IC-SOT23
- U202: footprint OHDSP-Footprints-Pretty:IC_SOIC_8 -> OHDSP-Footprints-Pretty:IC-LQFP48_7x7
- U203: footprint OHDSP-Footprints-Pretty:IC-LQFP48_7x7 -> OHDSP-Footprints-Pretty:IC_DIP_8

Commit message: WIP
Parts:
- added C250: N/F, OHDSP-Footprints-Pretty:SMD-0805, symbol C
- added R240: N/F, OHDSP-Footprints-Pretty:SMD-0805, symbol R
- added R241: 0R, OHDSP-Footprints-Pretty:SMD-0805, symbol R
- added TR204: N/F, OHDSP-Footprints-Pretty:IC-SOT23, symbol TRAN-NPN-BC847
- R230: value 1k -> 10k
- R231: value N/F -> 10k
- R232: value 1k -> N/F
Connections:
- net labels added: WP
- wire segments 295 -> 305
Other:
- note added: "Also add support for optional write back.\nThis will need high to low transistion\nsetting in the EEPROM selfboot messages."
- note added: "I2C Address Pins"
- note removed: "I2C Address"
- moved on the sheet: C238, C240, C241, C242, C243, C244, C245, C246, P201, R224, R229, R230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

Commit message: WIP
Parts:
- added R242, R243: 0R, OHDSP-Footprints-Pretty:SMD-0805, symbol R
- R211: footprint OHDSP-Footprints-Pretty:SMD-0805 -> OHDSP-Footprints-Pretty:SMD-1206
- U201: footprint OHDSP-Footprints-Pretty:IC_DIP_8 -> OHDSP-Footprints-Pretty:IC_SOIC_8
Connections:
- wire segments 305 -> 307
Changed lines of the file:
@@
 F 0 "U201" H 5000 9850 60  0000 C CNN
 F 1 "ADM13307-5ARZ" H 5350 9750 60  0000 C CNN
-F 2 "OHDSP-Footprints-Pretty:IC_DIP_8" H 4700 9600 60  0001 C CNN
+F 2 "OHDSP-Footprints-Pretty:IC_SOIC_8" H 4700 9600 60  0001 C CNN
 F 3 "" H 4700 9600 60  0000 C CNN
 	1    4700 9600
@@
 F 0 "R211" V 5350 4600 40  0000 C CNN
 F 1 "7k5" V 5257 4601 40  0000 C CNN
-F 2 "OHDSP-Footprints-Pretty:SMD-0805" V 5180 4600 30  0001 C CNN
+F 2 "OHDSP-Footprints-Pretty:SMD-1206" V 5180 4600 30  0001 C CNN
 F 3 "~" H 5250 4600 30  0000 C CNN
 	1    5250 4600
@@
 Text Label 15450 6600 0    60   ~ 0
 IOVDD
-Text Label 9100 6300 2    60   ~ 0
+Text Label 10000 6300 2    60   ~ 0
 SL_SCL
-Text Label 9100 6200 2    60   ~ 0
+Text Label 10000 6200 2    60   ~ 0
 SL_SDA
 $Comp
@@
 U 1 1 5519B9C0
 P 12700 6250
-F 0 "R226" V 12750 6450 40  0000 C CNN
+F 0 "R226" V 12800 6250 40  0000 C CNN
 F 1 "0R" V 12707 6251 40  0000 C CNN
 F 2 "OHDSP-Footprints-Pretty:SMD-0805" V 12630 6250 30  0001 C CNN
@@
 U 1 1 5519C1EE
 P 12850 6250
-F 0 "R227" V 12900 6450 40  0000 C CNN
+F 0 "R227" V 12900 6000 40  0000 C CNN
 F 1 "0R" V 12857 6251 40  0000 C CNN
 F 2 "OHDSP-Footprints-Pretty:SMD-0805" V 12780 6250 30  0001 C CNN
@@
 U 1 1 5519C2B4
 P 13000 6250
-F 0 "R228" V 13050 6450 40  0000 C CNN
+F 0 "R228" V 12900 6250 40  0000 C CNN
 F 1 "0R" V 13007 6251 40  0000 C CNN
 F 2 "OHDSP-Footprints-Pretty:SMD-0805" V 12930 6250 30  0001 C CNN
@@
 U 1 1 5519F434
 P 14600 6400
-F 0 "R241" V 14650 6600 40  0000 C CNN
+F 0 "R241" V 14700 6400 40  0000 C CNN
 F 1 "0R" V 14607 6401 40  0000 C CNN
 F 2 "OHDSP-Footprints-Pretty:SMD-0805" V 14530 6400 30  0001 C CNN
@@
 	12300 1900 12300 2200
 Connection ~ 12300 2200
+Connection ~ 8650 9300
+$Comp
+L R R242
+U 1 1 551E01DD
+P 9350 6200
+F 0 "R242" V 9450 6200 40  0000 C CNN
+F 1 "0R" V 9357 6201 40  0000 C CNN
+F 2 "OHDSP-Footprints-Pretty:SMD-0805" V 9280 6200 30  0001 C CNN
+F 3 "~" H 9350 6200 30  0000 C CNN
+	1    9350 6200
+	0    1    -1   0
+$EndComp
+$Comp
+L R R243
+U 1 1 551E0C1B
+P 9350 6300
+F 0 "R243" V 9250 6300 40  0000 C CNN
+F 1 "0R" V 9357 6301 40  0000 C CNN
+F 2 "OHDSP-Footprints-Pretty:SMD-0805" V 9280 6300 30  0001 C CNN
+F 3 "~" H 9350 6300 30  0000 C CNN
+	1    9350 6300
+	0    1    -1   0
+$EndComp
+Wire Wire Line
+	10000 6300 9600 6300
+Wire Wire Line
+	9600 6200 10000 6200
 $EndSCHEMATC

Commit message: WIP
Parts:
- U203: footprint OHDSP-Footprints-Pretty:IC_DIP_8 -> OHDSP-Footprints-Pretty:IC_SOIC_8
Changed lines of the file:
@@
 F 0 "U203" H 13550 6850 60  0000 C CNN
 F 1 "IC-EEPROM-I2C" H 13750 6750 60  0000 C CNN
-F 2 "OHDSP-Footprints-Pretty:IC_DIP_8" H 13300 6600 60  0001 C CNN
+F 2 "OHDSP-Footprints-Pretty:IC_SOIC_8" H 13300 6600 60  0001 C CNN
 F 3 "" H 13300 6600 60  0000 C CNN
 	1    13300 6600

Commit message: WIP
Parts:
- removed C204, C225, C234: 100p, OHDSP-Footprints-Pretty:SMD-0805, symbol C
- removed R201, R212, R220: 47R, OHDSP-Footprints-Pretty:SMD-0805, symbol R
- removed R210: 0R, OHDSP-Footprints-Pretty:SMD-0805, symbol R
Connections:
- wire segments 307 -> 297
Other:
- moved on the sheet: C208, C214, C216, C217, C218, C219, C220, C221, C222, C227, C229, C230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

Commit message: WIP
Parts:
- removed C219, C222: 10n, OHDSP-Footprints-Pretty:SMD-0805, symbol C
Changed lines of the file:
@@
-$EndComp
-$Comp
-L C C219
-U 1 1 54DAD63D
-P 3050 1650
-F 0 "C219" H 3050 1750 40  0000 L CNN
-F 1 "10n" H 3056 1565 40  0000 L CNN
-F 2 "OHDSP-Footprints-Pretty:SMD-0805" H 3088 1500 30  0001 C CNN
-F 3 "~" H 3050 1650 60  0000 C CNN
-	1    3050 1650
-	1    0    0    -1
 $EndComp
 $Comp
@@
 F 3 "~" H 3600 1650 60  0000 C CNN
 	1    3600 1650
-	1    0    0    -1
-$EndComp
-$Comp
-L C C222
-U 1 1 54DAE4B8
-P 3850 1650
-F 0 "C222" H 3850 1750 40  0000 L CNN
-F 1 "10n" H 3856 1565 40  0000 L CNN
-F 2 "OHDSP-Footprints-Pretty:SMD-0805" H 3888 1500 30  0001 C CNN
-F 3 "~" H 3850 1650 60  0000 C CNN
-	1    3850 1650
 	1    0    0    -1
 $EndComp
@@
 	2800 2150 2800 1850
 Connection ~ 2550 2150
-Wire Wire Line
-	3050 2150 3050 1850
 Connection ~ 2800 2150
 Wire Wire Line
@@
 	2800 1050 2800 1450
 Connection ~ 2550 1050
-Wire Wire Line
-	3050 1050 3050 1450
 Connection ~ 2800 1050
 Wire Wire Line
@@
 Connection ~ 3350 2150
 Wire Wire Line
-	3850 2150 3850 1850
-Connection ~ 3600 2150
-Wire Wire Line
 	3350 1050 3350 1450
 Wire Wire Line
 	3600 1050 3600 1450
 Connection ~ 3350 1050
-Wire Wire Line
-	3850 1050 3850 1450
 Connection ~ 3600 1050
-Connection ~ 3050 1050
-Connection ~ 3050 2150
 Wire Wire Line
 	800  900  800  1050
@@
 Wire Wire Line
 	1500 1050 3850 1050
-Wire Wire Line
-	1600 2150 3850 2150
 Wire Wire Line
 	6750 3550 6950 3550
@@
 Wire Wire Line
 	7250 2150 7900 2150
+Wire Wire Line
+	1600 2150 3600 2150
 $EndSCHEMATC
