File: Schematics/ADAU1701.sch (KiCad schematic (older format))
At the start: 100 parts, among them P201 CONN_2x1, SW201 SWITCH, U201 ADM13307-5ARZ, U202 ADAU1701JSTZ, U203 IC-EEPROM-I2C

Commit message: Change reset chip to ADM811
Parts:
- removed R203: 0R, OHDSP-Footprints-Pretty:SMD-0805, symbol R
- removed R204: 12k, OHDSP-Footprints-Pretty:SMD-0805, symbol R
- removed R205: 8k2, OHDSP-Footprints-Pretty:SMD-0805, symbol R
- removed R206: N/F, OHDSP-Footprints-Pretty:SMD-0805, symbol R
- removed R207: 3k, OHDSP-Footprints-Pretty:SMD-0805, symbol R
- removed R208: 4k7, OHDSP-Footprints-Pretty:SMD-0805, symbol R
- removed TP202: TP, OHDSP-Footprints-Pretty:TP-2mm, symbol PIN
- removed U201: ADM13307-5ARZ, OHDSP-Footprints-Pretty:IC_SOIC_8, symbol IC-RST-ADM13307
- added U201: IC-RST-ADM811, symbol IC-RST-ADM811
Connections:
- wire segments 293 -> 277
Other:
- note added: "Generate a global reset based, monitors 3v3 rail"
- note removed: "Generate a global reset based on voltage rails.\nUse ADM13307-5ARZ only! (Sense1=3v3, Sense2/3=Adj)"
- note removed: "USE 0.1% RESISTORS\n\nSENSE2 Vmin=2.973V\nSENSE3 Vmin=1.632V"
- moved on the sheet: C209, C213, C215, L202, R202

Commit message: Change to box headers
Parts:
- U201: footprint (none) -> OHDSP-Footprints-Pretty:IC-SOT143
Changed lines of the file:
@@
 ADCIN_SDATA0
 $Comp
-L GNDD #PWR202
+L GNDD #PWR01
 U 1 1 54DACD02
 P 1600 2200
-F 0 "#PWR202" H 1600 1950 60  0001 C CNN
+F 0 "#PWR01" H 1600 1950 60  0001 C CNN
 F 1 "GNDD" H 1600 2050 60  0000 C CNN
 F 2 "" H 1600 2200 60  0000 C CNN
@@
 DVDD
 $Comp
-L VDD #PWR201
+L VDD #PWR02
 U 1 1 54DB0DB8
 P 800 900
-F 0 "#PWR201" H 800 750 60  0001 C CNN
+F 0 "#PWR02" H 800 750 60  0001 C CNN
 F 1 "VDD" H 800 1050 60  0000 C CNN
 F 2 "" H 800 900 60  0000 C CNN
@@
 $EndComp
 $Comp
-L VPP #PWR207
+L VPP #PWR03
 U 1 1 54DB1373
 P 4050 900
-F 0 "#PWR207" H 4050 750 60  0001 C CNN
+F 0 "#PWR03" H 4050 750 60  0001 C CNN
 F 1 "VPP" H 4050 1050 60  0000 C CNN
 F 2 "" H 4050 900 60  0000 C CNN
@@
 $EndComp
 $Comp
-L GNDD #PWR210
+L GNDD #PWR04
 U 1 1 54DB1F60
 P 4850 2200
-F 0 "#PWR210" H 4850 1950 60  0001 C CNN
+F 0 "#PWR04" H 4850 1950 60  0001 C CNN
 F 1 "GNDD" H 4850 2050 60  0000 C CNN
 F 2 "" H 4850 2200 60  0000 C CNN
@@
 IOVDD
 $Comp
-L VAA #PWR214
+L VAA #PWR05
 U 1 1 54DB2FD4
 P 6450 900
-F 0 "#PWR214" H 6450 750 60  0001 C CNN
+F 0 "#PWR05" H 6450 750 60  0001 C CNN
 F 1 "VAA" H 6450 1050 60  0000 C CNN
 F 2 "" H 6450 900 60  0000 C CNN
@@
 $EndComp
 $Comp
-L GNDD #PWR218
+L GNDD #PWR06
 U 1 1 54DB2FEF
 P 7250 2200
-F 0 "#PWR218" H 7250 1950 60  0001 C CNN
+F 0 "#PWR06" H 7250 1950 60  0001 C CNN
 F 1 "GNDD" H 7250 2050 60  0000 C CNN
 F 2 "" H 7250 2200 60  0000 C CNN
@@
 PVDD
 $Comp
-L VAA #PWR227
+L VAA #PWR07
 U 1 1 54DB3C56
 P 11050 950
-F 0 "#PWR227" H 11050 800 60  0001 C CNN
+F 0 "#PWR07" H 11050 800 60  0001 C CNN
 F 1 "VAA" H 11050 1100 60  0000 C CNN
 F 2 "" H 11050 950 60  0000 C CNN
@@
 $EndComp
 $Comp
-L GNDD #PWR228
+L GNDD #PWR08
 U 1 1 54DB3C77
 P 11900 2250
-F 0 "#PWR228" H 11900 2000 60  0001 C CNN
+F 0 "#PWR08" H 11900 2000 60  0001 C CNN
 F 1 "GNDD" H 11900 2100 60  0000 C CNN
 F 2 "" H 11900 2250 60  0000 C CNN
@@
 $EndComp
 $Comp
-L GNDD #PWR223
+L GNDD #PWR09
 U 1 1 54DB551F
 P 8750 3600
-F 0 "#PWR223" H 8750 3350 60  0001 C CNN
+F 0 "#PWR09" H 8750 3350 60  0001 C CNN
 F 1 "GNDD" H 8750 3450 60  0000 C CNN
 F 2 "" H 8750 3600 60  0000 C CNN
@@
 $EndComp
 $Comp
-L GNDD #PWR215
+L GNDD #PWR010
 U 1 1 54DB589A
 P 6700 7250
-F 0 "#PWR215" H 6700 7000 60  0001 C CNN
+F 0 "#PWR010" H 6700 7000 60  0001 C CNN
 F 1 "GNDD" H 6700 7100 60  0000 C CNN
 F 2 "" H 6700 7250 60  0000 C CNN
@@
 $EndComp
 $Comp
-L GNDD #PWR226
+L GNDD #PWR011
 U 1 1 54DB858F
 P 10350 9400
-F 0 "#PWR226" H 10350 9150 60  0001 C CNN
+F 0 "#PWR011" H 10350 9150 60  0001 C CNN
 F 1 "GNDD" H 10350 9250 60  0000 C CNN
 F 2 "" H 10350 9400 60  0000 C CNN
@@
 $EndComp
 $Comp
-L GNDD #PWR221
+L GNDD #PWR012
 U 1 1 54DF7B4A
 P 7900 9900
-F 0 "#PWR221" H 7900 9650 60  0001 C CNN
+F 0 "#PWR012" H 7900 9650 60  0001 C CNN
 F 1 "GNDD" H 7900 9750 60  0000 C CNN
 F 2 "" H 7900 9900 60  0000 C CNN
@@
 $EndComp
 $Comp
-L GNDD #PWR232
+L GNDD #PWR013
 U 1 1 54DFF973
 P 15000 7100
-F 0 "#PWR232" H 15000 6850 60  0001 C CNN
+F 0 "#PWR013" H 15000 6850 60  0001 C CNN
 F 1 "GNDD" H 15000 6950 60  0000 C CNN
 F 2 "" H 15000 7100 60  0000 C CNN
@@
 $EndComp
 $Comp
-L GNDD #PWR235
+L GNDD #PWR014
 U 1 1 54E277D2
 P 15350 5100
-F 0 "#PWR235" H 15350 4850 60  0001 C CNN
+F 0 "#PWR014" H 15350 4850 60  0001 C CNN
 F 1 "GNDD" H 15350 4950 60  0000 C CNN
 F 2 "" H 15350 5100 60  0000 C CNN
@@
 I2C
 $Comp
-L VPP #PWR234
+L VPP #PWR015
 U 1 1 54E57AC0
 P 15350 4500
-F 0 "#PWR234" H 15350 4350 60  0001 C CNN
+F 0 "#PWR015" H 15350 4350 60  0001 C CNN
 F 1 "VPP" H 15350 4650 60  0000 C CNN
 F 2 "" H 15350 4500 60  0000 C CNN
@@
 $EndComp
 $Comp
-L GNDD #PWR233
+L GNDD #PWR016
 U 1 1 54E66110
 P 15300 7100
-F 0 "#PWR233" H 15300 6850 60  0001 C CNN
+F 0 "#PWR016" H 15300 6850 60  0001 C CNN
 F 1 "GNDD" H 15300 6950 60  0000 C CNN
 F 2 "" H 15300 7100 60  0000 C CNN
@@
 $EndComp
 $Comp
-L VPP #PWR225
+L VPP #PWR017
 U 1 1 54E9D3D9
 P 10350 8000
-F 0 "#PWR225" H 10350 7850 60  0001 C CNN
+F 0 "#PWR017" H 10350 7850 60  0001 C CNN
 F 1 "VPP" H 10350 8150 60  0000 C CNN
 F 2 "" H 10350 8000 60  0000 C CNN
@@
 Manual\nreset
 $Comp
-L GNDD #PWR217
+L GNDD #PWR018
 U 1 1 54EA0E15
 P 7050 10650
-F 0 "#PWR217" H 7050 10400 60  0001 C CNN
+F 0 "#PWR018" H 7050 10400 60  0001 C CNN
 F 1 "GNDD" H 7050 10500 60  0000 C CNN
 F 2 "" H 7050 10650 60  0000 C CNN
@@
 $EndComp
 $Comp
-L GNDD #PWR213
+L GNDD #PWR019
 U 1 1 54EA141D
 P 6100 10650
-F 0 "#PWR213" H 6100 10400 60  0001 C CNN
+F 0 "#PWR019" H 6100 10400 60  0001 C CNN
 F 1 "GNDD" H 6100 10500 60  0000 C CNN
 F 2 "" H 6100 10650 60  0000 C CNN
@@
 $EndComp
 $Comp
-L GNDD #PWR208
+L GNDD #PWR020
 U 1 1 54EA28F6
 P 4200 10800
-F 0 "#PWR208" H 4200 10550 60  0001 C CNN
+F 0 "#PWR020" H 4200 10550 60  0001 C CNN
 F 1 "GNDD" H 4200 10650 60  0000 C CNN
 F 2 "" H 4200 10800 60  0000 C CNN
@@
 $EndComp
 $Comp
-L GNDD #PWR209
+L GNDD #PWR021
 U 1 1 54EA2F14
 P 4400 10350
-F 0 "#PWR209" H 4400 10100 60  0001 C CNN
+F 0 "#PWR021" H 4400 10100 60  0001 C CNN
 F 1 "GNDD" H 4400 10200 60  0000 C CNN
 F 2 "" H 4400 10350 60  0000 C CNN
@@
 $EndComp
 $Comp
-L GNDD #PWR212
+L GNDD #PWR022
 U 1 1 54EA451E
 P 5050 10000
-F 0 "#PWR212" H 5050 9750 60  0001 C CNN
+F 0 "#PWR022" H 5050 9750 60  0001 C CNN
 F 1 "GNDD" H 5050 9850 60  0000 C CNN
 F 2 "" H 5050 10000 60  0000 C CNN
@@
 RST_OUT
 $Comp
-L VPP #PWR206
+L VPP #PWR023
 U 1 1 54E404E0
 P 3500 9650
-F 0 "#PWR206" H 3500 9500 60  0001 C CNN
+F 0 "#PWR023" H 3500 9500 60  0001 C CNN
 F 1 "VPP" H 3500 9800 60  0000 C CNN
 F 2 "" H 3500 9650 60  0000 C CNN
@@
 $EndComp
 $Comp
-L GNDD #PWR219
+L GNDD #PWR024
 U 1 1 54FF363C
 P 7450 10750
-F 0 "#PWR219" H 7450 10500 60  0001 C CNN
+F 0 "#PWR024" H 7450 10500 60  0001 C CNN
 F 1 "GNDD" H 7450 10600 60  0000 C CNN
 F 2 "" H 7450 10750 60  0000 C CNN
@@
 $EndComp
 $Comp
-L GNDD #PWR216
+L GNDD #PWR025
 U 1 1 54FF7C76
 P 6750 10700
-F 0 "#PWR216" H 6750 10450 60  0001 C CNN
+F 0 "#PWR025" H 6750 10450 60  0001 C CNN
 F 1 "GNDD" H 6750 10550 60  0000 C CNN
 F 2 "" H 6750 10700 60  0000 C CNN
@@
 $EndComp
 $Comp
-L GNDD #PWR211
+L GNDD #PWR026
 U 1 1 55163566
 P 4900 4650
-F 0 "#PWR211" H 4900 4400 60  0001 C CNN
+F 0 "#PWR026" H 4900 4400 60  0001 C CNN
 F 1 "GNDD" H 4900 4500 60  0000 C CNN
 F 2 "" H 4900 4650 60  0000 C CNN
@@
 $EndComp
 $Comp
-L GNDD #PWR224
+L GNDD #PWR027
 U 1 1 5516ACC7
 P 8750 7150
-F 0 "#PWR224" H 8750 6900 60  0001 C CNN
+F 0 "#PWR027" H 8750 6900 60  0001 C CNN
 F 1 "GNDD" H 8750 7000 60  0000 C CNN
 F 2 "" H 8750 7150 60  0000 C CNN
@@
 $EndComp
 $Comp
-L GNDD #PWR229
+L GNDD #PWR028
 U 1 1 55170343
 P 12050 9400
-F 0 "#PWR229" H 12050 9150 60  0001 C CNN
+F 0 "#PWR028" H 12050 9150 60  0001 C CNN
 F 1 "GNDD" H 12050 9250 60  0000 C CNN
 F 2 "" H 12050 9400 60  0000 C CNN
@@
 $EndComp
 $Comp
-L GNDD #PWR230
+L GNDD #PWR029
 U 1 1 5519C877
 P 13200 6950
-F 0 "#PWR230" H 13200 6700 60  0001 C CNN
+F 0 "#PWR029" H 13200 6700 60  0001 C CNN
 F 1 "GNDD" H 13200 6800 60  0000 C CNN
 F 2 "" H 13200 6950 60  0000 C CNN
@@
 $EndComp
 $Comp
-L GNDD #PWR220
+L GNDD #PWR030
 U 1 1 551483F9
 P 7750 10850
-F 0 "#PWR220" H 7750 10600 60  0001 C CNN
+F 0 "#PWR030" H 7750 10600 60  0001 C CNN
 F 1 "GNDD" H 7750 10700 60  0000 C CNN
 F 2 "" H 7750 10850 60  0000 C CNN
@@
 $EndComp
 $Comp
-L VPP #PWR222
+L VPP #PWR031
 U 1 1 551493D2
 P 8650 9250
-F 0 "#PWR222" H 8650 9100 60  0001 C CNN
+F 0 "#PWR031" H 8650 9100 60  0001 C CNN
 F 1 "VPP" H 8650 9400 60  0000 C CNN
 F 2 "" H 8650 9250 60  0000 C CNN
@@
 $EndComp
 $Comp
-L GNDD #PWR203
+L GNDD #PWR032
 U 1 1 55163561
 P 1650 4750
-F 0 "#PWR203" H 1650 4500 60  0001 C CNN
+F 0 "#PWR032" H 1650 4500 60  0001 C CNN
 F 1 "GNDD" H 1650 4600 60  0000 C CNN
 F 2 "" H 1650 4750 60  0000 C CNN
@@
 $EndComp
 $Comp
-L GNDD #PWR204
+L GNDD #PWR033
 U 1 1 55164F29
 P 1650 5600
-F 0 "#PWR204" H 1650 5350 60  0001 C CNN
+F 0 "#PWR033" H 1650 5350 60  0001 C CNN
 F 1 "GNDD" H 1650 5450 60  0000 C CNN
 F 2 "" H 1650 5600 60  0000 C CNN
@@
 $EndComp
 $Comp
-L GNDD #PWR205
+L GNDD #PWR034
 U 1 1 55165032
 P 1650 6500
-F 0 "#PWR205" H 1650 6250 60  0001 C CNN
+F 0 "#PWR034" H 1650 6250 60  0001 C CNN
 F 1 "GNDD" H 1650 6350 60  0000 C CNN
 F 2 "" H 1650 6500 60  0000 C CNN
@@
 $EndComp
 $Comp
-L GNDD #PWR231
+L GNDD #PWR035
 U 1 1 5516EC7A
 P 14600 9400
-F 0 "#PWR231" H 14600 9150 60  0001 C CNN
+F 0 "#PWR035" H 14600 9150 60  0001 C CNN
 F 1 "GNDD" H 14600 9250 60  0000 C CNN
 F 2 "" H 14600 9400 60  0000 C CNN
@@
 F 0 "U201" H 5350 10000 60  0000 C CNN
 F 1 "IC-RST-ADM811" H 5600 9900 60  0000 C CNN
-F 2 "" H 5100 9900 60  0000 C CNN
+F 2 "OHDSP-Footprints-Pretty:IC-SOT143" H 5100 9900 60  0001 C CNN
 F 3 "" H 5100 9900 60  0000 C CNN
 	1    5100 9750

Commit message: WIP
Other:
- moved on the sheet: C209, C213, C215, C226, C228, C232, L202, P201, R202, R213, R214, R215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

Commit message: WIP
Parts:
- added P?: CONN_02X05, OHDSP-Footprints-Pretty:CONN_DIL_2X5_BOX, symbol CONN_02X05
- added R? (x6): 27R, OHDSP-Footprints-Pretty:SMD-0805, symbol R
- added R?: 1k, OHDSP-Footprints-Pretty:SMD-0805, symbol R
Connections:
- net labels added: ADIRST
- net labels removed: RST_IN1
- wire segments 277 -> 382
- no-connect marks 0 -> 6
Other:
- note added: "ADI EVAL-ADUSB2Z USB/I2C"

Commit message: WIP
Parts:
- removed C202: 220u, OHDSP-Footprints-Pretty:CAP-TH-D6.3mmP2.5mm, symbol CP1
- removed C207: 10u, OHDSP-Footprints-Pretty:SMD-0805, symbol C
- removed C212, C221, C242: 100n, OHDSP-Footprints-Pretty:SMD-0805, symbol C
- removed C214: 22u, OHDSP-Footprints-Pretty:SMD-0805, symbol C
- removed C220, C243: 1u, OHDSP-Footprints-Pretty:SMD-0805, symbol C
- removed C224: 3n3, OHDSP-Footprints-Pretty:SMD-0805, symbol C
- removed R224: 1k, OHDSP-Footprints-Pretty:SMD-0805, symbol R
- removed R225: 47R, OHDSP-Footprints-Pretty:SMD-0805, symbol R
- removed R236: 2k2, OHDSP-Footprints-Pretty:SMD-0805, symbol R
- added C204: 220u, OHDSP-Footprints-Pretty:CAP-TH-D6.3mmP2.5mm, symbol CP1
- added C209, C210: 10u, OHDSP-Footprints-Pretty:SMD-0805, symbol C
- added C215, C219, C237: 100n, OHDSP-Footprints-Pretty:SMD-0805, symbol C
- added C218, C239: 1u, OHDSP-Footprints-Pretty:SMD-0805, symbol C
- added C225: 3n3, OHDSP-Footprints-Pretty:SMD-0805, symbol C
- added R222: 1k, OHDSP-Footprints-Pretty:SMD-0805, symbol R
- added R223: 47R, OHDSP-Footprints-Pretty:SMD-0805, symbol R
- added R237: 2k2, OHDSP-Footprints-Pretty:SMD-0805, symbol R
- C206: value 10u -> 22u
- R206: renamed from R211; footprint OHDSP-Footprints-Pretty:SMD-1206 -> OHDSP-Footprints-Pretty:SMD-0805
- U203: footprint OHDSP-Footprints-Pretty:IC_SOIC_8 -> OHDSP-Footprints-Pretty:IC_DIP_8
- gave numbers to parts that had none: 8
- renumbered C208 to C201, C201 to C202, C209 to C205, C213 to C207, C205 to C208, C215 to C211, C216 to C212, C210 to C213, C211 to C214, C217 to C216, C218 to C217, C226 to C220, C228 to C221, C227 to C222, C232 to C223, C223 to C224, C229 to C226, C230 to C227, C231 to C228, C233 to C229, C235 to C230, C236 to C231, C237 to C232, C239 to C233, C238 to C234, C240 to C235, C241 to C236, C250 to C238, C244 to C240, C245 to C241, C246 to C242, C247 to C243, C248 to C244, C249 to C245, R202 to R201, R213 to R202, R214 to R203, R209 to R204, R215 to R205, R216 to R207, R219 to R208, R221 to R209, R222 to R210, R223 to R211, R217 to R212, R218 to R213, R242 to R220, R243 to R221, R226 to R224, R229 to R225, R230 to R226, R231 to R230, R232 to R231, R240 to R232, R241 to R233, R233 to R234, R234 to R235, R235 to R236, R237 to R238, R238 to R239, R239 to R240
Connections:
- net AVDD: now also C237.1, C239.1, R223.1
- net CM: now also C204.1, C210.1, C215.1; no longer C203.1
- net DVDD: now also C206.1, C218.1, C219.1
- net FILTD: now also C203.1, C209.1; no longer C206.1
- net GNDD: now also C204.2, C209.2, C210.2, C215.2, C218.2, C219.2, C237.2, C239.2
- net I2C_SDA: now also R237.2
- net PVDD: now also C225.2
- net VPP: now also R222.1, R237.1
- net at C233.1: now also R223.2
- net at C224.1, U202.35 (PLL_LF): now also C225.1
- net SELFBOOT renamed SELFBOOT_EN
- net SELFBOOT_EN: now also R222.2
- net WP renamed SELFBOOT_WP
Other:
- moved on the sheet: C243, C244, R224, R227, R228, R233, R234, U203
