File: Schematics/Connectors.sch (KiCad schematic (older format))
At the start: 84 parts, among them P501 CONN_02X10, P502 CONN_02X05, P503 CONN_02X05, P504 CONN_02X05, P505 CONN_02X10, P506 CONN_2x1, P507 CONN_2x1, P508 CONN_02X20, P509 CONN_02X05, P510 CONN_02X05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

Commit message: WIP
Parts:
- added R?: 1k, symbol R
Connections:
- net labels added: ADI_RST, PI_RST, RST_OUT
- net labels removed: MRST
- wire segments 322 -> 326
- no-connect marks 5 -> 4
Changed lines of the file:
@@
 Text Label 1550 9600 0    60   ~ 0
 SL_~SS
-Text Label 2500 9500 0    60   ~ 0
+Text Label 3200 9500 0    60   ~ 0
 SL_MOSI
 $Comp
@@
 $EndComp
 Text HLabel 10200 2050 0    60   Output ~ 0
-MRST
+PI_RST
 $Comp
 L CONN_02X05 P509
@@
 	1550 9200 1900 9200
 Wire Wire Line
-	2400 9500 2700 9500
+	2400 9500 3550 9500
 Wire Wire Line
 	2500 9600 2400 9600
@@
 	11050 2150 11200 2150
 NoConn ~ 2400 9200
-NoConn ~ 2400 9400
 Wire Wire Line
 	13600 1500 14100 1500
@@
 Wire Wire Line
 	2350 3000 1600 3000
+Text HLabel 3250 9350 2    60   Output ~ 0
+ADI_RST
+$Comp
+L R R?
+U 1 1 5517B867
+P 2750 9400
+F 0 "R?" V 2830 9400 40  0000 C CNN
+F 1 "1k" V 2757 9401 40  0000 C CNN
+F 2 "" V 2680 9400 30  0001 C CNN
+F 3 "~" H 2750 9400 30  0000 C CNN
+	1    2750 9400
+	0    1    -1   0
+$EndComp
+Wire Wire Line
+	3250 9350 3100 9350
+Wire Wire Line
+	3100 9350 3100 9400
+Wire Wire Line
+	3100 9400 3000 9400
+Wire Wire Line
+	2500 9400 2400 9400
+Text HLabel 5650 9300 2    60   Output ~ 0
+RST_OUT
 $EndSCHEMATC

Commit message: WIP
Connections:
- net labels added: ANA_IN1, ANA_IN2, ANA_OUT1, ANA_OUT2, ANA_OUT3, ANA_OUT4
- net labels removed: ANAIN1, ANAIN2, ANAOUT1, ANAOUT2, ANAOUT3, ANAOUT4, RST_OUT
Changed lines of the file:
@@
 $EndComp
 Text HLabel 11400 7250 2    60   Output ~ 0
-ANAIN1
+ANA_IN1
 Wire Wire Line
 	10500 7250 10600 7250
@@
 $EndComp
 Text HLabel 11400 8950 2    60   Output ~ 0
-ANAIN2
+ANA_IN2
 Wire Wire Line
 	10500 8950 10600 8950
@@
 $EndComp
 Text HLabel 12550 6450 0    60   Input ~ 0
-ANAOUT1
+ANA_OUT1
 Wire Wire Line
 	13450 6450 13350 6450
@@
 $EndComp
 Text HLabel 12550 7300 0    60   Input ~ 0
-ANAOUT2
+ANA_OUT2
 Wire Wire Line
 	13450 7300 13350 7300
@@
 $EndComp
 Text HLabel 12550 8100 0    60   Input ~ 0
-ANAOUT3
+ANA_OUT3
 Wire Wire Line
 	13450 8100 13350 8100
@@
 $EndComp
 Text HLabel 12550 8950 0    60   Input ~ 0
-ANAOUT4
+ANA_OUT4
 Wire Wire Line
 	13450 8950 13350 8950
@@
 Wire Wire Line
 	2500 9400 2400 9400
-Text HLabel 5650 9300 2    60   Output ~ 0
-RST_OUT
 $EndSCHEMATC

Commit message: WIP
Parts:
- C501, C502, C503, C505, C512, C513, C514, C515, L501, R501, R502, R503, R504, R505, R506, R507, R508, R509, R510, R511, R512: footprint (none) -> OHDSP-Footprints-Pretty:SMD-0805
- C504: footprint (none) -> OHDSP-Footprints-Pretty:CAP-TH-D6.3mmP2.5mm
- C506, C507, C508, C509, C510, C511: footprint (none) -> OHDSP-Footprints-Pretty:CAP-TH-D8mmP3.5mm
- D501, D502, D503, D504: footprint (none) -> OHDSP-Footprints-Pretty:DIODE-DO-41
- P501, P505: footprint (none) -> OHDSP-Footprints-Pretty:CONN_DIL_2X10
- P502, P503, P504, P509, P510, P511: footprint (none) -> OHDSP-Footprints-Pretty:CONN_DIL_2X5
- P506, P507, P512, P513, P514, P515: footprint (none) -> OHDSP-Footprints-Pretty:CONN_SIL_2
- P508: footprint (none) -> OHDSP-Footprints-Pretty:CONN_DIL_2X20
- R513: renamed from R?; footprint (none) -> OHDSP-Footprints-Pretty:SMD-0805
- R514: renamed from R513; footprint (none) -> OHDSP-Footprints-Pretty:SMD-0805
- R515: renamed from R514; footprint (none) -> OHDSP-Footprints-Pretty:SMD-0805
- R516: renamed from R515; footprint (none) -> OHDSP-Footprints-Pretty:SMD-0805
- R517: renamed from R516; footprint (none) -> OHDSP-Footprints-Pretty:SMD-0805
- R518: renamed from R517; footprint (none) -> OHDSP-Footprints-Pretty:SMD-0805
- R519: renamed from R518; footprint (none) -> OHDSP-Footprints-Pretty:SMD-0805
- R520: renamed from R519; footprint (none) -> OHDSP-Footprints-Pretty:SMD-0805
- R521: renamed from R520; footprint (none) -> OHDSP-Footprints-Pretty:SMD-0805
- R522: renamed from R521; footprint (none) -> OHDSP-Footprints-Pretty:SMD-0805
- R523: renamed from R522; footprint (none) -> OHDSP-Footprints-Pretty:SMD-0805
- R524: renamed from R523; footprint (none) -> OHDSP-Footprints-Pretty:SMD-0805
- R525: renamed from R524; footprint (none) -> OHDSP-Footprints-Pretty:SMD-0805
- R526: renamed from R525; footprint (none) -> OHDSP-Footprints-Pretty:SMD-0805
- R527: renamed from R526; footprint (none) -> OHDSP-Footprints-Pretty:SMD-0805
- R528: renamed from R527; footprint (none) -> OHDSP-Footprints-Pretty:SMD-0805
- R529: renamed from R528; footprint (none) -> OHDSP-Footprints-Pretty:SMD-0805
- R530: renamed from R529; footprint (none) -> OHDSP-Footprints-Pretty:SMD-0805
- R531: renamed from R530; footprint (none) -> OHDSP-Footprints-Pretty:SMD-0805
- R532: renamed from R531; footprint (none) -> OHDSP-Footprints-Pretty:SMD-0805
- R533: renamed from R532; footprint (none) -> OHDSP-Footprints-Pretty:SMD-0805
- R534: renamed from R533; footprint (none) -> OHDSP-Footprints-Pretty:SMD-0805
- R535: renamed from R534; footprint (none) -> OHDSP-Footprints-Pretty:SMD-0805
- R536: renamed from R535; footprint (none) -> OHDSP-Footprints-Pretty:SMD-0805
- R537: renamed from R536; footprint (none) -> OHDSP-Footprints-Pretty:SMD-0805
- R538: renamed from R537; footprint (none) -> OHDSP-Footprints-Pretty:SMD-0805
- R539: renamed from R538; footprint (none) -> OHDSP-Footprints-Pretty:SMD-0805
- R540: renamed from R539; footprint (none) -> OHDSP-Footprints-Pretty:SMD-0805
- R541: renamed from R540; footprint (none) -> OHDSP-Footprints-Pretty:SMD-0805
- R542: renamed from R541; footprint (none) -> OHDSP-Footprints-Pretty:SMD-0805
- R543: renamed from R542; footprint (none) -> OHDSP-Footprints-Pretty:SMD-0805
- R544: renamed from R543; footprint (none) -> OHDSP-Footprints-Pretty:SMD-0805
- R545: renamed from R544; footprint (none) -> OHDSP-Footprints-Pretty:SMD-0805
- R546: renamed from R545; footprint (none) -> OHDSP-Footprints-Pretty:SMD-0805
- R547: renamed from R546; footprint (none) -> OHDSP-Footprints-Pretty:SMD-0805
- R548: renamed from R547; footprint (none) -> OHDSP-Footprints-Pretty:SMD-0805
- R549: renamed from R548; footprint (none) -> OHDSP-Footprints-Pretty:SMD-0805
- renumbered R549 to R550
