File: Schematics/Connectors.sch (KiCad schematic (older format))
At the start: 85 parts, among them P501 CONN_02X10, P502 CONN_02X05, P503 CONN_02X05, P504 CONN_02X05, P505 CONN_02X10, P506 CONN_2x1, P507 CONN_2x1, P508 CONN_02X20, P509 CONN_02X05, P510 CONN_02X05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

Commit message: WIP
Parts:
- R543: value 0R -> N/F
Changed lines of the file:
@@
 SL_SDA
 $Comp
-L GNDD #PWR096
+L GNDD #PWR093
 U 1 1 54DC2149
 P 2500 9700
-F 0 "#PWR096" H 2500 9450 60  0001 C CNN
+F 0 "#PWR093" H 2500 9450 60  0001 C CNN
 F 1 "GNDD" H 2500 9550 60  0000 C CNN
 F 2 "" H 2500 9700 60  0000 C CNN
@@
 $EndComp
 $Comp
-L GNDD #PWR097
+L GNDD #PWR094
 U 1 1 54DC87F8
 P 11800 3450
-F 0 "#PWR097" H 11800 3200 60  0001 C CNN
+F 0 "#PWR094" H 11800 3200 60  0001 C CNN
 F 1 "GNDD" H 11800 3300 60  0000 C CNN
 F 2 "" H 11800 3450 60  0000 C CNN
@@
 $EndComp
 $Comp
-L GNDD #PWR098
+L GNDD #PWR095
 U 1 1 54DC884A
 P 11100 3450
-F 0 "#PWR098" H 11100 3200 60  0001 C CNN
+F 0 "#PWR095" H 11100 3200 60  0001 C CNN
 F 1 "GNDD" H 11100 3300 60  0000 C CNN
 F 2 "" H 11100 3450 60  0000 C CNN
@@
 $EndComp
 $Comp
-L GNDD #PWR099
+L GNDD #PWR096
 U 1 1 54DCE262
 P 2950 3900
-F 0 "#PWR099" H 2950 3650 60  0001 C CNN
+F 0 "#PWR096" H 2950 3650 60  0001 C CNN
 F 1 "GNDD" H 2950 3750 60  0000 C CNN
 F 2 "" H 2950 3900 60  0000 C CNN
@@
 These go to the slave port\nThese are 3v3 lines only!
 $Comp
-L GNDD #PWR0100
+L GNDD #PWR097
 U 1 1 54E4935B
 P 900 3000
-F 0 "#PWR0100" H 900 2750 60  0001 C CNN
+F 0 "#PWR097" H 900 2750 60  0001 C CNN
 F 1 "GNDD" H 900 2850 60  0000 C CNN
 F 2 "" H 900 3000 60  0000 C CNN
@@
 $EndComp
 $Comp
-L GNDD #PWR0101
+L GNDD #PWR098
 U 1 1 54E56282
 P 6450 3850
-F 0 "#PWR0101" H 6450 3600 60  0001 C CNN
+F 0 "#PWR098" H 6450 3600 60  0001 C CNN
 F 1 "GNDD" H 6450 3700 60  0000 C CNN
 F 2 "" H 6450 3850 60  0000 C CNN
@@
 P 12150 1450
 F 0 "R543" V 12200 1750 40  0000 C CNN
-F 1 "0R" V 12157 1451 40  0000 C CNN
+F 1 "N/F" V 12157 1451 40  0000 C CNN
 F 2 "OHDSP-Footprints-Pretty:SMD-0805" V 12080 1450 30  0001 C CNN
 F 3 "~" H 12150 1450 30  0000 C CNN
@@
 $EndComp
 $Comp
-L PWR_FLAG #FLG0102
+L PWR_FLAG #FLG099
 U 1 1 54E974DE
 P 12450 1500
-F 0 "#FLG0102" H 12450 1595 30  0001 C CNN
+F 0 "#FLG099" H 12450 1595 30  0001 C CNN
 F 1 "PWR_FLAG" H 12450 1680 30  0000 C CNN
 F 2 "" H 12450 1500 60  0000 C CNN
@@
 $EndComp
 $Comp
-L +5V #PWR0103
+L +5V #PWR0100
 U 1 1 54E47415
 P 12450 1350
-F 0 "#PWR0103" H 12450 1200 60  0001 C CNN
+F 0 "#PWR0100" H 12450 1200 60  0001 C CNN
 F 1 "+5V" H 12450 1490 60  0000 C CNN
 F 2 "" H 12450 1350 60  0000 C CNN
@@
 $EndComp
 $Comp
-L GNDD #PWR0104
+L GNDD #PWR0101
 U 1 1 54E3EEEB
 P 8500 2800
-F 0 "#PWR0104" H 8500 2550 60  0001 C CNN
+F 0 "#PWR0101" H 8500 2550 60  0001 C CNN
 F 1 "GNDD" H 8500 2650 60  0000 C CNN
 F 2 "" H 8500 2800 60  0000 C CNN
@@
 $EndComp
 $Comp
-L GNDD #PWR0105
+L GNDD #PWR0102
 U 1 1 54E480D0
 P 1850 7100
-F 0 "#PWR0105" H 1850 6850 60  0001 C CNN
+F 0 "#PWR0102" H 1850 6850 60  0001 C CNN
 F 1 "GNDD" H 1850 6950 60  0000 C CNN
 F 2 "" H 1850 7100 60  0000 C CNN
@@
 SL_SDA
 $Comp
-L VPP #PWR0106
+L VPP #PWR0103
 U 1 1 54E4FE28
 P 4350 6600
-F 0 "#PWR0106" H 4350 6450 60  0001 C CNN
+F 0 "#PWR0103" H 4350 6450 60  0001 C CNN
 F 1 "VPP" H 4350 6750 60  0000 C CNN
 F 2 "" H 4350 6600 60  0000 C CNN
@@
 $EndComp
 $Comp
-L GNDD #PWR0107
+L GNDD #PWR0104
 U 1 1 54E50905
 P 1150 7100
-F 0 "#PWR0107" H 1150 6850 60  0001 C CNN
+F 0 "#PWR0104" H 1150 6850 60  0001 C CNN
 F 1 "GNDD" H 1150 6950 60  0000 C CNN
 F 2 "" H 1150 7100 60  0000 C CNN
@@
 $EndComp
 $Comp
-L GNDD #PWR0108
+L GNDD #PWR0105
 U 1 1 54E5413C
 P 3450 7100
-F 0 "#PWR0108" H 3450 6850 60  0001 C CNN
+F 0 "#PWR0105" H 3450 6850 60  0001 C CNN
 F 1 "GNDD" H 3450 6950 60  0000 C CNN
 F 2 "" H 3450 7100 60  0000 C CNN
@@
 $EndComp
 $Comp
-L GNDD #PWR0109
+L GNDD #PWR0106
 U 1 1 54E54645
 P 3200 7200
-F 0 "#PWR0109" H 3200 6950 60  0001 C CNN
+F 0 "#PWR0106" H 3200 6950 60  0001 C CNN
 F 1 "GNDD" H 3200 7050 60  0000 C CNN
 F 2 "" H 3200 7200 60  0000 C CNN
@@
 $EndComp
 $Comp
-L GNDD #PWR0110
+L GNDD #PWR0107
 U 1 1 54E55D4A
 P 1850 8150
-F 0 "#PWR0110" H 1850 7900 60  0001 C CNN
+F 0 "#PWR0107" H 1850 7900 60  0001 C CNN
 F 1 "GNDD" H 1850 8000 60  0000 C CNN
 F 2 "" H 1850 8150 60  0000 C CNN
@@
 SL_SCL
 $Comp
-L GNDD #PWR0111
+L GNDD #PWR0108
 U 1 1 54E55D5C
 P 1150 8150
-F 0 "#PWR0111" H 1150 7900 60  0001 C CNN
+F 0 "#PWR0108" H 1150 7900 60  0001 C CNN
 F 1 "GNDD" H 1150 8000 60  0000 C CNN
 F 2 "" H 1150 8150 60  0000 C CNN
@@
 $EndComp
 $Comp
-L GNDD #PWR0112
+L GNDD #PWR0109
 U 1 1 54F77292
 P 2150 8200
-F 0 "#PWR0112" H 2150 7950 60  0001 C CNN
+F 0 "#PWR0109" H 2150 7950 60  0001 C CNN
 F 1 "GNDD" H 2150 8050 60  0000 C CNN
 F 2 "" H 2150 8200 60  0000 C CNN
@@
 PI_GP16
 $Comp
-L GNDD #PWR0113
+L GNDD #PWR0110
 U 1 1 54FFB4F8
 P 14650 3250
-F 0 "#PWR0113" H 14650 3000 60  0001 C CNN
+F 0 "#PWR0110" H 14650 3000 60  0001 C CNN
 F 1 "GNDD" H 14650 3100 60  0000 C CNN
 F 2 "" H 14650 3250 60  0000 C CNN
@@
 $EndComp
 $Comp
-L GNDD #PWR0114
+L GNDD #PWR0111
 U 1 1 55149DF3
 P 3400 3900
-F 0 "#PWR0114" H 3400 3650 60  0001 C CNN
+F 0 "#PWR0111" H 3400 3650 60  0001 C CNN
 F 1 "GNDD" H 3400 3750 60  0000 C CNN
 F 2 "" H 3400 3900 60  0000 C CNN
@@
 $EndComp
 $Comp
-L GNDD #PWR0115
+L GNDD #PWR0112
 U 1 1 55152108
 P 6000 3850
-F 0 "#PWR0115" H 6000 3600 60  0001 C CNN
+F 0 "#PWR0112" H 6000 3600 60  0001 C CNN
 F 1 "GNDD" H 6000 3700 60  0000 C CNN
 F 2 "" H 6000 3850 60  0000 C CNN
@@
 	10500 7250 10600 7250
 $Comp
-L GNDD #PWR0116
+L GNDD #PWR0113
 U 1 1 55157B54
 P 9950 7400
-F 0 "#PWR0116" H 9950 7150 60  0001 C CNN
+F 0 "#PWR0113" H 9950 7150 60  0001 C CNN
 F 1 "GNDD" H 9950 7250 60  0000 C CNN
 F 2 "" H 9950 7400 60  0000 C CNN
@@
 Connection ~ 11100 7250
 $Comp
-L GNDD #PWR0117
+L GNDD #PWR0114
 U 1 1 551582D5
 P 11100 7800
-F 0 "#PWR0117" H 11100 7550 60  0001 C CNN
+F 0 "#PWR0114" H 11100 7550 60  0001 C CNN
 F 1 "GNDD" H 11100 7650 60  0000 C CNN
 F 2 "" H 11100 7800 60  0000 C CNN
@@
 	11100 7800 11100 7750
 $Comp
-L VPP #PWR0118
+L VPP #PWR0115
 U 1 1 5515886B
 P 11200 6750
-F 0 "#PWR0118" H 11200 6600 60  0001 C CNN
+F 0 "#PWR0115" H 11200 6600 60  0001 C CNN
 F 1 "VPP" H 11200 6900 60  0000 C CNN
 F 2 "" H 11200 6750 60  0000 C CNN
@@
 	10500 8950 10600 8950
 $Comp
-L GNDD #PWR0119
+L GNDD #PWR0116
 U 1 1 55159842
 P 9950 9100
-F 0 "#PWR0119" H 9950 8850 60  0001 C CNN
+F 0 "#PWR0116" H 9950 8850 60  0001 C CNN
 F 1 "GNDD" H 9950 8950 60  0000 C CNN
 F 2 "" H 9950 9100 60  0000 C CNN
@@
 Connection ~ 11100 8950
 $Comp
-L GNDD #PWR0120
+L GNDD #PWR0117
 U 1 1 55159855
 P 11100 9500
-F 0 "#PWR0120" H 11100 9250 60  0001 C CNN
+F 0 "#PWR0117" H 11100 9250 60  0001 C CNN
 F 1 "GNDD" H 11100 9350 60  0000 C CNN
 F 2 "" H 11100 9500 60  0000 C CNN
@@
 	11100 9500 11100 9450
 $Comp
-L VPP #PWR0121
+L VPP #PWR0118
 U 1 1 5515985C
 P 11200 8450
-F 0 "#PWR0121" H 11200 8300 60  0001 C CNN
+F 0 "#PWR0118" H 11200 8300 60  0001 C CNN
 F 1 "VPP" H 11200 8600 60  0000 C CNN
 F 2 "" H 11200 8450 60  0000 C CNN
@@
 	13450 6450 13350 6450
 $Comp
-L GNDD #PWR0122
+L GNDD #PWR0119
 U 1 1 5515A1E8
 P 14500 6600
-F 0 "#PWR0122" H 14500 6350 60  0001 C CNN
+F 0 "#PWR0119" H 14500 6350 60  0001 C CNN
 F 1 "GNDD" H 14500 6450 60  0000 C CNN
 F 2 "" H 14500 6600 60  0000 C CNN
@@
 	14100 6550 14100 6450
 $Comp
-L GNDD #PWR0123
+L GNDD #PWR0120
 U 1 1 5515DB03
 P 14100 7000
-F 0 "#PWR0123" H 14100 6750 60  0001 C CNN
+F 0 "#PWR0120" H 14100 6750 60  0001 C CNN
 F 1 "GNDD" H 14100 6850 60  0000 C CNN
 F 2 "" H 14100 7000 60  0000 C CNN
@@
 	13450 7300 13350 7300
 $Comp
-L GNDD #PWR0124
+L GNDD #PWR0121
 U 1 1 5515EC44
 P 14500 7450
-F 0 "#PWR0124" H 14500 7200 60  0001 C CNN
+F 0 "#PWR0121" H 14500 7200 60  0001 C CNN
 F 1 "GNDD" H 14500 7300 60  0000 C CNN
 F 2 "" H 14500 7450 60  0000 C CNN
@@
 	14100 7400 14100 7300
 $Comp
-L GNDD #PWR0125
+L GNDD #PWR0122
 U 1 1 5515EC5B
 P 14100 7850
-F 0 "#PWR0125" H 14100 7600 60  0001 C CNN
+F 0 "#PWR0122" H 14100 7600 60  0001 C CNN
 F 1 "GNDD" H 14100 7700 60  0000 C CNN
 F 2 "" H 14100 7850 60  0000 C CNN
@@
 	13450 8100 13350 8100
 $Comp
-L GNDD #PWR0126
+L GNDD #PWR0123
 U 1 1 5515F0C7
 P 14500 8250
-F 0 "#PWR0126" H 14500 8000 60  0001 C CNN
+F 0 "#PWR0123" H 14500 8000 60  0001 C CNN
 F 1 "GNDD" H 14500 8100 60  0000 C CNN
 F 2 "" H 14500 8250 60  0000 C CNN
@@
 	14100 8200 14100 8100
 $Comp
-L GNDD #PWR0127
+L GNDD #PWR0124
 U 1 1 5515F0DE
 P 14100 8650
-F 0 "#PWR0127" H 14100 8400 60  0001 C CNN
+F 0 "#PWR0124" H 14100 8400 60  0001 C CNN
 F 1 "GNDD" H 14100 8500 60  0000 C CNN
 F 2 "" H 14100 8650 60  0000 C CNN
@@
 	13450 8950 13350 8950
 $Comp
-L GNDD #PWR0128
+L GNDD #PWR0125
 U 1 1 5515F0F4
 P 14500 9100
-F 0 "#PWR0128" H 14500 8850 60  0001 C CNN
+F 0 "#PWR0125" H 14500 8850 60  0001 C CNN
 F 1 "GNDD" H 14500 8950 60  0000 C CNN
 F 2 "" H 14500 9100 60  0000 C CNN
@@
 	14100 9050 14100 8950
 $Comp
-L GNDD #PWR0129
+L GNDD #PWR0126
 U 1 1 5515F10B
 P 14100 9500
-F 0 "#PWR0129" H 14100 9250 60  0001 C CNN
+F 0 "#PWR0126" H 14100 9250 60  0001 C CNN
 F 1 "GNDD" H 14100 9350 60  0000 C CNN
 F 2 "" H 14100 9500 60  0000 C CNN
@@
 Connection ~ 2150 1600
 $Comp
-L GNDD #PWR0130
+L GNDD #PWR0127
 U 1 1 55143B7B
 P 2150 3900
-F 0 "#PWR0130" H 2150 3650 60  0001 C CNN
+F 0 "#PWR0127" H 2150 3650 60  0001 C CNN
 F 1 "GNDD" H 2150 3750 60  0000 C CNN
 F 2 "" H 2150 3900 60  0000 C CNN

Commit message: WIP
Parts:
- removed C501, C502: 100n, OHDSP-Footprints-Pretty:SMD-0805, symbol C
- removed C503: 22u, OHDSP-Footprints-Pretty:SMD-0805, symbol C
- removed C504: 220u, OHDSP-Footprints-Pretty:CAP-TH-D6.3mmP2.5mm, symbol CP1
- removed C505: 100p, OHDSP-Footprints-Pretty:SMD-0805, symbol C
- removed L501: 600R@100MHz, OHDSP-Footprints-Pretty:SMD-0805, symbol INDUCTOR
- added C516, C517: 100p, OHDSP-Footprints-Pretty:SMD-0805, symbol C
- added R551, R552, R553, R554, R555, R556: 0R, OHDSP-Footprints-Pretty:SMD-1206, symbol R
- added R557, R558: 47R, OHDSP-Footprints-Pretty:SMD-0805, symbol R
- added R559: 1k, OHDSP-Footprints-Pretty:SMD-0805, symbol R
- R519: value 47R -> 1k
- R537, R538, R547, R548, R549, R550: footprint OHDSP-Footprints-Pretty:SMD-0805 -> OHDSP-Footprints-Pretty:SMD-1206
Connections:
- wire segments 322 -> 302
- no-connect marks 8 -> 20
Other:
- note added: "External I2C headers\nFor ADC and DAC"
- note added: "I2C Connectors\n"
- note removed: "Generic I2S and SPI connectors\n"
- note removed: "Some handy external connectors\nwith I2C and power"
- moved on the sheet: C506, C507, D501, D502, D503, D504, P506, P507, R537, R538

Commit message: WIP
Parts:
- added R560, R561: 0R, OHDSP-Footprints-Pretty:SMD-1206, symbol R
Connections:
- wire segments 302 -> 303
Other:
- moved on the sheet: R504, R505, R506, R507, R508, R509, R510, R511, R512, R514, R515, R516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

Commit message: WIP
Changed lines of the file:
@@
 U 1 1 55157505
 P 10050 7550
-F 0 "D501" H 9850 7600 40  0000 C CNN
+F 0 "D501" H 10050 7650 40  0000 C CNN
 F 1 "1N5818" H 10050 7450 40  0000 C CNN
 F 2 "OHDSP-Footprints-Pretty:DIODE-DO-41" H 10050 7550 60  0001 C CNN
@@
 U 1 1 551575DD
 P 10150 7000
-F 0 "D503" H 9950 7050 40  0000 C CNN
+F 0 "D503" H 10150 7100 40  0000 C CNN
 F 1 "1N5818" H 10150 6900 40  0000 C CNN
 F 2 "OHDSP-Footprints-Pretty:DIODE-DO-41" H 10150 7000 60  0001 C CNN

Commit message: Change to box headers
Parts:
- P501, P505: footprint OHDSP-Footprints-Pretty:CONN_DIL_2X10 -> OHDSP-Footprints-Pretty:CONN_DIL_2X10_BOX
- P502, P503, P504: footprint OHDSP-Footprints-Pretty:CONN_DIL_2X5 -> OHDSP-Footprints-Pretty:CONN_DIL_2X5_BOX
Changed lines of the file:
@@
 F 0 "P504" H 2150 9700 50  0000 C CNN
 F 1 "CONN_02X05" H 2150 9100 50  0000 C CNN
-F 2 "OHDSP-Footprints-Pretty:CONN_DIL_2X5" H 2150 8200 60  0001 C CNN
+F 2 "OHDSP-Footprints-Pretty:CONN_DIL_2X5_BOX" H 2150 8200 60  0001 C CNN
 F 3 "" H 2150 8200 60  0000 C CNN
 	1    2150 9400
@@
 SL_SDA
 $Comp
-L GNDD #PWR506
+L GNDD #PWR083
 U 1 1 54DC2149
 P 2500 9700
-F 0 "#PWR506" H 2500 9450 60  0001 C CNN
+F 0 "#PWR083" H 2500 9450 60  0001 C CNN
 F 1 "GNDD" H 2500 9550 60  0000 C CNN
 F 2 "" H 2500 9700 60  0000 C CNN
@@
 $EndComp
 $Comp
-L GNDD #PWR520
+L GNDD #PWR084
 U 1 1 54DC87F8
 P 11800 3450
-F 0 "#PWR520" H 11800 3200 60  0001 C CNN
+F 0 "#PWR084" H 11800 3200 60  0001 C CNN
 F 1 "GNDD" H 11800 3300 60  0000 C CNN
 F 2 "" H 11800 3450 60  0000 C CNN
@@
 $EndComp
 $Comp
-L GNDD #PWR519
+L GNDD #PWR085
 U 1 1 54DC884A
 P 11100 3450
-F 0 "#PWR519" H 11100 3200 60  0001 C CNN
+F 0 "#PWR085" H 11100 3200 60  0001 C CNN
 F 1 "GNDD" H 11100 3300 60  0000 C CNN
 F 2 "" H 11100 3450 60  0000 C CNN
@@
 $EndComp
 $Comp
-L GNDD #PWR505
+L GNDD #PWR086
 U 1 1 54DCE262
 P 2100 3900
-F 0 "#PWR505" H 2100 3650 60  0001 C CNN
+F 0 "#PWR086" H 2100 3650 60  0001 C CNN
 F 1 "GNDD" H 2100 3750 60  0000 C CNN
 F 2 "" H 2100 3900 60  0000 C CNN
@@
 These go to the slave port\nThese are 3v3 lines only!
 $Comp
-L GNDD #PWR501
+L GNDD #PWR087
 U 1 1 54E4935B
 P 900 3000
-F 0 "#PWR501" H 900 2750 60  0001 C CNN
+F 0 "#PWR087" H 900 2750 60  0001 C CNN
 F 1 "GNDD" H 900 2850 60  0000 C CNN
 F 2 "" H 900 3000 60  0000 C CNN
@@
 $EndComp
 $Comp
-L GNDD #PWR510
+L GNDD #PWR088
 U 1 1 54E56282
 P 5800 3850
-F 0 "#PWR510" H 5800 3600 60  0001 C CNN
+F 0 "#PWR088" H 5800 3600 60  0001 C CNN
 F 1 "GNDD" H 5800 3700 60  0000 C CNN
 F 2 "" H 5800 3850 60  0000 C CNN
@@
 $EndComp
 $Comp
-L PWR_FLAG #FLG501
+L PWR_FLAG #FLG089
 U 1 1 54E974DE
 P 12450 1500
-F 0 "#FLG501" H 12450 1595 30  0001 C CNN
+F 0 "#FLG089" H 12450 1595 30  0001 C CNN
 F 1 "PWR_FLAG" H 12450 1680 30  0000 C CNN
 F 2 "" H 12450 1500 60  0000 C CNN
@@
 $EndComp
 $Comp
-L +5V #PWR521
+L +5V #PWR090
 U 1 1 54E47415
 P 12450 1350
-F 0 "#PWR521" H 12450 1200 60  0001 C CNN
+F 0 "#PWR090" H 12450 1200 60  0001 C CNN
 F 1 "+5V" H 12450 1490 60  0000 C CNN
 F 2 "" H 12450 1350 60  0000 C CNN
@@
 $EndComp
 $Comp
-L GNDD #PWR512
+L GNDD #PWR091
 U 1 1 54E3EEEB
 P 8500 2800
-F 0 "#PWR512" H 8500 2550 60  0001 C CNN
+F 0 "#PWR091" H 8500 2550 60  0001 C CNN
 F 1 "GNDD" H 8500 2650 60  0000 C CNN
 F 2 "" H 8500 2800 60  0000 C CNN
@@
 F 0 "P502" H 1500 7150 50  0000 C CNN
 F 1 "CONN_02X05" H 1500 6550 50  0000 C CNN
-F 2 "OHDSP-Footprints-Pretty:CONN_DIL_2X5" H 1500 5650 60  0001 C CNN
+F 2 "OHDSP-Footprints-Pretty:CONN_DIL_2X5_BOX" H 1500 5650 60  0001 C CNN
 F 3 "" H 1500 5650 60  0000 C CNN
 	1    1500 6850
@@
 F 0 "P503" H 1500 8200 50  0000 C CNN
 F 1 "CONN_02X05" H 1500 7600 50  0000 C CNN
-F 2 "OHDSP-Footprints-Pretty:CONN_DIL_2X5" H 1500 6700 60  0001 C CNN
+F 2 "OHDSP-Footprints-Pretty:CONN_DIL_2X5_BOX" H 1500 6700 60  0001 C CNN
 F 3 "" H 1500 6700 60  0000 C CNN
 	1    1500 7900
@@
 PI_GP16
 $Comp
-L GNDD #PWR530
+L GNDD #PWR092
 U 1 1 54FFB4F8
 P 14650 3250
-F 0 "#PWR530" H 14650 3000 60  0001 C CNN
+F 0 "#PWR092" H 14650 3000 60  0001 C CNN
 F 1 "GNDD" H 14650 3100 60  0000 C CNN
 F 2 "" H 14650 3250 60  0000 C CNN
@@
 $EndComp
 $Comp
-L GNDD #PWR507
+L GNDD #PWR093
 U 1 1 55149DF3
 P 2550 3900
-F 0 "#PWR507" H 2550 3650 60  0001 C CNN
+F 0 "#PWR093" H 2550 3650 60  0001 C CNN
 F 1 "GNDD" H 2550 3750 60  0000 C CNN
 F 2 "" H 2550 3900 60  0000 C CNN
@@
 $EndComp
 $Comp
-L GNDD #PWR509
+L GNDD #PWR094
 U 1 1 55152108
 P 5350 3850
-F 0 "#PWR509" H 5350 3600 60  0001 C CNN
+F 0 "#PWR094" H 5350 3600 60  0001 C CNN
 F 1 "GNDD" H 5350 3700 60  0000 C CNN
 F 2 "" H 5350 3850 60  0000 C CNN
@@
 	9450 7250 9550 7250
 $Comp
-L GNDD #PWR513
+L GNDD #PWR095
 U 1 1 55157B54
 P 8900 7400
-F 0 "#PWR513" H 8900 7150 60  0001 C CNN
+F 0 "#PWR095" H 8900 7150 60  0001 C CNN
 F 1 "GNDD" H 8900 7250 60  0000 C CNN
 F 2 "" H 8900 7400 60  0000 C CNN
@@
 Connection ~ 10050 7250
 $Comp
-L GNDD #PWR515
+L GNDD #PWR096
 U 1 1 551582D5
 P 10050 7800
-F 0 "#PWR515" H 10050 7550 60  0001 C CNN
+F 0 "#PWR096" H 10050 7550 60  0001 C CNN
 F 1 "GNDD" H 10050 7650 60  0000 C CNN
 F 2 "" H 10050 7800 60  0000 C CNN
@@
 	10050 7800 10050 7750
 $Comp
-L VPP #PWR517
+L VPP #PWR097
 U 1 1 5515886B
 P 10150 6750
-F 0 "#PWR517" H 10150 6600 60  0001 C CNN
+F 0 "#PWR097" H 10150 6600 60  0001 C CNN
 F 1 "VPP" H 10150 6900 60  0000 C CNN
 F 2 "" H 10150 6750 60  0000 C CNN
@@
 	9450 8950 9550 8950
 $Comp
-L GNDD #PWR514
+L GNDD #PWR098
 U 1 1 55159842
 P 8900 9100
-F 0 "#PWR514" H 8900 8850 60  0001 C CNN
+F 0 "#PWR098" H 8900 8850 60  0001 C CNN
 F 1 "GNDD" H 8900 8950 60  0000 C CNN
 F 2 "" H 8900 9100 60  0000 C CNN
@@
 Connection ~ 10050 8950
 $Comp
-L GNDD #PWR516
+L GNDD #PWR099
 U 1 1 55159855
 P 10050 9500
-F 0 "#PWR516" H 10050 9250 60  0001 C CNN
+F 0 "#PWR099" H 10050 9250 60  0001 C CNN
 F 1 "GNDD" H 10050 9350 60  0000 C CNN
 F 2 "" H 10050 9500 60  0000 C CNN
@@
 	10050 9500 10050 9450
 $Comp
-L VPP #PWR518
+L VPP #PWR0100
 U 1 1 5515985C
 P 10150 8450
-F 0 "#PWR518" H 10150 8300 60  0001 C CNN
+F 0 "#PWR0100" H 10150 8300 60  0001 C CNN
 F 1 "VPP" H 10150 8600 60  0000 C CNN
 F 2 "" H 10150 8450 60  0000 C CNN
@@
 	13450 6450 13350 6450
 $Comp
-L GNDD #PWR526
+L GNDD #PWR0101
 U 1 1 5515A1E8
 P 14500 6600
-F 0 "#PWR526" H 14500 6350 60  0001 C CNN
+F 0 "#PWR0101" H 14500 6350 60  0001 C CNN
 F 1 "GNDD" H 14500 6450 60  0000 C CNN
 F 2 "" H 14500 6600 60  0000 C CNN
@@
 	14100 6550 14100 6450
 $Comp
-L GNDD #PWR522
+L GNDD #PWR0102
 U 1 1 5515DB03
 P 14100 7000
-F 0 "#PWR522" H 14100 6750 60  0001 C CNN
+F 0 "#PWR0102" H 14100 6750 60  0001 C CNN
 F 1 "GNDD" H 14100 6850 60  0000 C CNN
 F 2 "" H 14100 7000 60  0000 C CNN
@@
 	13450 7300 13350 7300
 $Comp
-L GNDD #PWR527
+L GNDD #PWR0103
 U 1 1 5515EC44
 P 14500 7450
-F 0 "#PWR527" H 14500 7200 60  0001 C CNN
+F 0 "#PWR0103" H 14500 7200 60  0001 C CNN
 F 1 "GNDD" H 14500 7300 60  0000 C CNN
 F 2 "" H 14500 7450 60  0000 C CNN
@@
 	14100 7400 14100 7300
 $Comp
-L GNDD #PWR523
+L GNDD #PWR0104
 U 1 1 5515EC5B
 P 14100 7850
-F 0 "#PWR523" H 14100 7600 60  0001 C CNN
+F 0 "#PWR0104" H 14100 7600 60  0001 C CNN
 F 1 "GNDD" H 14100 7700 60  0000 C CNN
 F 2 "" H 14100 7850 60  0000 C CNN
@@
 	13450 8100 13350 8100
 $Comp
-L GNDD #PWR528
+L GNDD #PWR0105
 U 1 1 5515F0C7
 P 14500 8250
-F 0 "#PWR528" H 14500 8000 60  0001 C CNN
+F 0 "#PWR0105" H 14500 8000 60  0001 C CNN
 F 1 "GNDD" H 14500 8100 60  0000 C CNN
 F 2 "" H 14500 8250 60  0000 C CNN
@@
 	14100 8200 14100 8100
 $Comp
-L GNDD #PWR524
+L GNDD #PWR0106
 U 1 1 5515F0DE
 P 14100 8650
-F 0 "#PWR524" H 14100 8400 60  0001 C CNN
+F 0 "#PWR0106" H 14100 8400 60  0001 C CNN
 F 1 "GNDD" H 14100 8500 60  0000 C CNN
 F 2 "" H 14100 8650 60  0000 C CNN
@@
 	13450 8950 13350 8950
 $Comp
-L GNDD #PWR529
+L GNDD #PWR0107
 U 1 1 5515F0F4
 P 14500 9100
-F 0 "#PWR529" H 14500 8850 60  0001 C CNN
+F 0 "#PWR0107" H 14500 8850 60  0001 C CNN
 F 1 "GNDD" H 14500 8950 60  0000 C CNN
 F 2 "" H 14500 9100 60  0000 C CNN
@@
 	14100 9050 14100 8950
 $Comp
-L GNDD #PWR525
+L GNDD #PWR0108
 U 1 1 5515F10B
 P 14100 9500
-F 0 "#PWR525" H 14100 9250 60  0001 C CNN
+F 0 "#PWR0108" H 14100 9250 60  0001 C CNN
 F 1 "GNDD" H 14100 9350 60  0000 C CNN
 F 2 "" H 14100 9500 60  0000 C CNN
@@
 F 0 "P501" H 1200 4050 50  0000 C CNN
 F 1 "CONN_02X10" V 1200 3550 50  0000 C CNN
-F 2 "OHDSP-Footprints-Pretty:CONN_DIL_2X10" H 400 2100 60  0001 C CNN
+F 2 "OHDSP-Footprints-Pretty:CONN_DIL_2X10_BOX" H 400 2100 60  0001 C CNN
 F 3 "" H 400 2100 60  0000 C CNN
 	1    1200 3000
@@
 	3800 3100 3800 1600
 $Comp
-L GNDD #PWR508
+L GNDD #PWR0109
 U 1 1 55143B7B
 P 3800 3900
-F 0 "#PWR508" H 3800 3650 60  0001 C CNN
+F 0 "#PWR0109" H 3800 3650 60  0001 C CNN
 F 1 "GNDD" H 3800 3750 60  0000 C CNN
 F 2 "" H 3800 3900 60  0000 C CNN
@@
 F 0 "P505" H 8200 3850 50  0000 C CNN
 F 1 "CONN_02X10" V 8200 3350 50  0000 C CNN
-F 2 "OHDSP-Footprints-Pretty:CONN_DIL_2X10" H 7400 1900 60  0001 C CNN
+F 2 "OHDSP-Footprints-Pretty:CONN_DIL_2X10_BOX" H 7400 1900 60  0001 C CNN
 F 3 "" H 7400 1900 60  0000 C CNN
 	1    8200 2800
@@
 Connection ~ 1650 3000
 $Comp
-L GNDD #PWR502
+L GNDD #PWR0110
 U 1 1 551D386C
 P 1650 4150
-F 0 "#PWR502" H 1650 3900 60  0001 C CNN
+F 0 "#PWR0110" H 1650 3900 60  0001 C CNN
 F 1 "GNDD" H 1650 4000 60  0000 C CNN
 F 2 "" H 1650 4150 60  0000 C CNN
@@
 	7550 3700 7550 3600
 $Comp
-L GNDD #PWR511
+L GNDD #PWR0111
 U 1 1 551D45E4
 P 7550 4150
-F 0 "#PWR511" H 7550 3900 60  0001 C CNN
+F 0 "#PWR0111" H 7550 3900 60  0001 C CNN
 F 1 "GNDD" H 7550 4000 60  0000 C CNN
 F 2 "" H 7550 4150 60  0000 C CNN
@@
 	900  6650 1250 6650
 $Comp
-L GNDD #PWR504
+L GNDD #PWR0112
 U 1 1 551E8B52
 P 1850 8200
-F 0 "#PWR504" H 1850 7950 60  0001 C CNN
+F 0 "#PWR0112" H 1850 7950 60  0001 C CNN
 F 1 "GNDD" H 1850 8050 60  0000 C CNN
 F 2 "" H 1850 8200 60  0000 C CNN
@@
 	1850 8200 1850 8100
 $Comp
-L GNDD #PWR503
+L GNDD #PWR0113
 U 1 1 551E8BB2
 P 1850 7150
-F 0 "#PWR503" H 1850 6900 60  0001 C CNN
+F 0 "#PWR0113" H 1850 6900 60  0001 C CNN
 F 1 "GNDD" H 1850 7000 60  0000 C CNN
 F 2 "" H 1850 7150 60  0000 C CNN
