File: Schematics/ADAU1701 PSU.sch (KiCad schematic (older format))
At the start: 59 parts, among them P301 CONN_2x1, P302 CONN_2x1, P303 PIN, P304 PIN, P305 PIN, P306 PIN, U301 IC-REG-XRP7659ISTR-F, U302 IC-REG-XRP7659ISTR-F, U304 IC-REG-XC6210B332MR, U305 IC-REG-XC6210B332MR

Commit message: WIP
Parts:
- removed C301, C314: 220u, OHDSP-Footprints-Pretty:CAP-TH-D6.3mmP2.5mm, symbol CP1
- removed C303: 22u, OHDSP-Footprints-Pretty:SMD-0805, symbol C
- removed C305: 100n, OHDSP-Footprints-Pretty:SMD-0805, symbol C
- removed C309: 10n, OHDSP-Footprints-Pretty:SMD-0805, symbol C
- removed D303: SS24T3G, OHDSP-Footprints-Pretty:DIODE-SMB, symbol SCHOTTKY_DIODE
- removed L302: 744772047, OHDSP-Footprints-Pretty:PASSIVE-TH-IND-WURTH-5mm, symbol INDUCTOR
- removed R301: 100k, OHDSP-Footprints-Pretty:SMD-0805, symbol R
- removed R304: 47k, OHDSP-Footprints-Pretty:SMD-0805, symbol R
- removed R305: 97k6, OHDSP-Footprints-Pretty:SMD-0805, symbol R
- removed U301: IC-REG-XRP7659ISTR-F, OHDSP-Footprints-Pretty:IC-SOT23-6, symbol IC-REG-XRP7659ISTR-F
- removed U304, U305: IC-REG-XC6210B332MR, OHDSP-Footprints-Pretty:IC-SOT25, symbol IC-REG-XC6210B332MR
- added C319: 10n, symbol C
- added C320, C322, C325: 100n, symbol C
- added C328: 22u, symbol C
- added C331: 100u, symbol CP1
- added R309: 10k, symbol R
- added U302, U303: NCP700BSN33T1G, symbol IC-REG-NCP700B
- added U304: NCP700BSN18T1G, symbol IC-REG-NCP700B
- C301: renamed from C304; footprint OHDSP-Footprints-Pretty:SMD-0805 -> (none)
- C302: renamed from C306; footprint OHDSP-Footprints-Pretty:SMD-0805 -> (none)
- C303: renamed from C307; footprint OHDSP-Footprints-Pretty:SMD-0805 -> (none)
- C304: renamed from C308; footprint OHDSP-Footprints-Pretty:CAP-TH-D6.3mmP2.5mm -> (none)
- C305: renamed from C310; footprint OHDSP-Footprints-Pretty:SMD-0805 -> (none)
- C306: renamed from C311; footprint OHDSP-Footprints-Pretty:SMD-0805 -> (none)
- C307: renamed from C312; footprint OHDSP-Footprints-Pretty:SMD-0805 -> (none)
- C308: renamed from C315; footprint OHDSP-Footprints-Pretty:SMD-0805 -> (none)
- C309: renamed from C317; footprint OHDSP-Footprints-Pretty:CAP-TH-D6.3mmP2.5mm -> (none)
- C310: renamed from C319; footprint OHDSP-Footprints-Pretty:SMD-0805 -> (none)
- C311: renamed from C325; footprint OHDSP-Footprints-Pretty:SMD-0805 -> (none)
- C312: renamed from C326; footprint OHDSP-Footprints-Pretty:SMD-0805 -> (none)
- C313, C316, L301: footprint OHDSP-Footprints-Pretty:SMD-0805 -> (none)
- C314: renamed from C328; footprint OHDSP-Footprints-Pretty:SMD-0805 -> (none)
- C315: renamed from C329; footprint OHDSP-Footprints-Pretty:SMD-0805 -> (none)
- C317: renamed from C330; value 1u -> 10n; footprint OHDSP-Footprints-Pretty:SMD-0805 -> (none)
- C318: renamed from C331; footprint OHDSP-Footprints-Pretty:SMD-0805 -> (none)
- C321: value 1u -> 100n; footprint OHDSP-Footprints-Pretty:SMD-0805 -> (none)
- C323: renamed from C334; footprint OHDSP-Footprints-Pretty:SMD-0805 -> (none)
- C324: renamed from C335; footprint OHDSP-Footprints-Pretty:SMD-0805 -> (none)
- C326: renamed from C337; footprint OHDSP-Footprints-Pretty:SMD-0805 -> (none)
- C327: renamed from C338; footprint OHDSP-Footprints-Pretty:SMD-0805 -> (none)
- C329: renamed from C340; footprint OHDSP-Footprints-Pretty:CAP-TH-D6.3mmP2.5mm -> (none)
- C330: renamed from C341; footprint OHDSP-Footprints-Pretty:CAP-TH-D6.3mmP2.5mm -> (none)
- D301, D302: footprint OHDSP-Footprints-Pretty:DIODE-SMB -> (none)
- D303: renamed from D304; footprint OHDSP-Footprints-Pretty:DIODE-SMB -> (none)
- D304: renamed from D306; footprint OHDSP-Footprints-Pretty:SMD-1206 -> (none)
- L302: renamed from L303; footprint OHDSP-Footprints-Pretty:PASSIVE-TH-IND-WURTH-5mm -> (none)
- P301: renamed from P303; footprint OHDSP-Footprints-Pretty:MNT_HOLE_2.5mm -> (none)
- P302: renamed from P304; footprint OHDSP-Footprints-Pretty:MNT_HOLE_2.5mm -> (none)
- P303: renamed from P305; footprint OHDSP-Footprints-Pretty:MNT_HOLE_2.5mm -> (none)
- P304: renamed from P301; footprint OHDSP-Footprints-Pretty:CONN-SCREW-2WAY-5mm-5.08mm -> (none)
- P305: renamed from P302; footprint OHDSP-Footprints-Pretty:CONN-SCREW-2WAY-5mm-5.08mm -> (none)
- P306: footprint OHDSP-Footprints-Pretty:MNT_HOLE_2.5mm -> (none)
- R301: renamed from R302; footprint OHDSP-Footprints-Pretty:SMD-0805 -> (none)
- R302: renamed from R303; footprint OHDSP-Footprints-Pretty:SMD-0805 -> (none)
- R303: renamed from R306; footprint OHDSP-Footprints-Pretty:SMD-0805 -> (none)
- R304: renamed from R307; footprint OHDSP-Footprints-Pretty:SMD-0805 -> (none)
- R305: renamed from R308; footprint OHDSP-Footprints-Pretty:SMD-0805 -> (none)
- R306: renamed from R310; footprint OHDSP-Footprints-Pretty:SMD-0805 -> (none)
- R307: renamed from R313; value 100k -> 10k; footprint OHDSP-Footprints-Pretty:SMD-0805 -> (none)
- R308: renamed from R314; footprint OHDSP-Footprints-Pretty:SMD-0805 -> (none)
- U301: renamed from U302; footprint OHDSP-Footprints-Pretty:IC-SOT23-6 -> (none)
Connections:
- net GNDD: now also C319.2, C320.2, C322.2, C325.2, C328.2, C331.2, U302.2 (GND), U303.2 (GND), U304.2 (GND); no longer C323.2, C326.2, C329.2
- net VAA: now also U302.5 (OUT); no longer R306.1
- net VCOM: now also C313.1, C316.1, R306.1, R309.1, U302.1 (IN), U303.1 (IN), U304.1 (IN)
- net VDD: now also C325.1, C328.1, C331.1, U304.5 (OUT); no longer C313.1, C316.1
- net VPP: now also U303.5 (OUT)
- net at C321.1: now also U303.4 (BYP)
- net at C317.1, R307.2: now also U302.3 (EN)
- net at C318.1, R308.2: now also U303.3 (EN)
- new net: C320.1, U302.4 (BYP)
- new net: C319.1, R309.2, U304.3 (EN)
- new net: C322.1, U304.4 (BYP)
- no-connect marks 2 -> 0
Other:
- note added: "3v3 For ADAU1701 AVDD PVDD"
- note removed: "1v2 Supply"
- note removed: "3v3 Supplies"
- note removed: "Add small diode\nfor quick discharge"
- note removed: "Can use 1% resistors for\nR305 and R304 although\n0.1% would be better."
- note removed: "VAA - delayed 3v3\nFor ADAU1452 AVDD PVDD"
- note removed: "Wait for 3v3 supply before bringing\nup ADAU1452 DVDD supply. IOVDD\nmust always be first, order is not\nimportant on the other supplies."
- moved on the sheet: C301, C302, C303, C304, C305, C306, C307, C308, C309, C310, C311, C312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

Commit message: WIP
Parts:
- C301, C302, C303, C305, C306, C307, C308, C310, C311, C312, C313, C314, C315, C316, C317, C318, C319, C320, C321, C322, C323, C324, C325, C326, C327, C328, D304, L301, R301, R302, R303, R304, R305, R306, R307, R308, R309: footprint (none) -> OHDSP-Footprints-Pretty:SMD-0805
- C304, C309: footprint (none) -> OHDSP-Footprints-Pretty:CAP-TH-D6.3mmP2.5mm
- C329, C330, C331: value 100u -> 220u; footprint (none) -> OHDSP-Footprints-Pretty:CAP-TH-D6.3mmP2.5mm
- D301, D302, D303: footprint (none) -> OHDSP-Footprints-Pretty:DIODE-SMB
- L302: footprint (none) -> OHDSP-Footprints-Pretty:PASSIVE-TH-IND-WURTH-5mm
- P304, P305: footprint (none) -> OHDSP-Footprints-Pretty:CONN_SIL_2
- U301: footprint (none) -> OHDSP-Footprints-Pretty:IC-SOT23-6
- U302, U303, U304: footprint (none) -> OHDSP-Footprints-Pretty:IC-SOT23-5

Commit message: WIP
Parts:
- P301, P302, P303, P306: footprint (none) -> OHDSP-Footprints-Pretty:MNT_HOLE_2.5mm

Commit message: WIP
Connections:
- net GNDD: now also C323.2, C326.2, C329.2

Commit message: WIP PSU changes
Parts:
- removed D301: SS24T3G, OHDSP-Footprints-Pretty:DIODE-SMB, symbol DIODE
- removed P304: CONN_2x1, OHDSP-Footprints-Pretty:CONN_SIL_2, symbol CONN_2x1
Connections:
- net +5V: now also C308.1, C309.1, C310.1, C311.1, C312.1, C313.1, C314.1, C315.1, C316.1, R306.1, R307.1, R308.1, R309.1, U302.1 (IN), U303.1 (IN), U304.1 (IN)
- removed net VCOM: C308.1, C309.1, C310.1, C311.1, C312.1, C313.1, C314.1, C315.1, C316.1, L302.2, R303.1, R306.1, R307.1, R308.1, R309.1, U302.1 (IN), U303.1 (IN), U304.1 (IN)
Other:
- note added: "Screw terminals for 9V-18V input\nWill also power the Pi"
- note removed: "Two sets of screw terminals\nOne for 5V-16V self power\nOne set for 5V - will power the Pi as well\nDo not put 16V up the Pi!"
- moved on the sheet: C301, C302, C303, C304, C305, C306, C307, D302, D303, L301, L302, P301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
