File: Schematics/ADAU1701 PSU.sch (KiCad schematic (older format))
At the start: 54 parts, among them P301 PIN, P302 PIN, P303 PIN, P305 CONN_2x1, P306 PIN, U301 IC-REG-XRP7659ISTR-F, U302 NCP700BSN33T1G, U303 NCP700BSN33T1G, U304 NCP700BSN18T1G

Commit message: WIP
Parts:
- removed C308, C311, C312, C313: 22u, OHDSP-Footprints-Pretty:SMD-0805, symbol C
- removed C309: 220u, OHDSP-Footprints-Pretty:CAP-TH-D6.3mmP2.5mm, symbol CP1
- removed C310: 100n, OHDSP-Footprints-Pretty:SMD-0805, symbol C
- removed U301: IC-REG-XRP7659ISTR-F, OHDSP-Footprints-Pretty:IC-SOT23-6, symbol IC-REG-XRP7659ISTR-F
- added C308: 35ZL470MEFC10X20, OHDSP-Footprints-Pretty:CAP-TH-D10mmP5mm, symbol CP1
- added C309: 1n5, OHDSP-Footprints-Pretty:SMD-0805, symbol C
- added C310: 10ZL470MEFC8X11.5, OHDSP-Footprints-Pretty:CAP-TH-D8mmP3.5mm, symbol CP1
- added C311, C312, C313: 220u, OHDSP-Footprints-Pretty:CAP-TH-D6.3mmP2.5mm, symbol CP1
- added D301: 1N914, OHDSP-Footprints-Pretty:DIODE-DO-35, symbol DIODE
- added D305, D306: LED, OHDSP-Footprints-Pretty:SMD-0805, symbol LED
- added R310: 4k7, OHDSP-Footprints-Pretty:SMD-0805, symbol R
- added U301: LT1374CS8-5#PBF, OHDSP-Footprints-Pretty:IC_SOIC_8, symbol IC-REG-LT1374/6
- C305: value 10n -> 270n; Voltage (none) -> 100v
- D302, D303: value SS24T3G -> MBRS330T3; footprint OHDSP-Footprints-Pretty:DIODE-SMB -> OHDSP-Footprints-Pretty:DIODE-SMC
- L302: value 744772220 -> CDRH125NP-100MC; footprint OHDSP-Footprints-Pretty:PASSIVE-TH-IND-WURTH-5mm -> OHDSP-Footprints-Pretty:IND_SMD_CDRH125
- R301: value 100k -> 1R
- R303: value 39k -> 1R
- R304: value 10k -> 1R
- R305: value 0R -> 4k7
Connections:
- net labels removed: VCOM
- wire segments 122 -> 132
Other:
- note added: "External Power LEDs\n"
- note added: "External Supply Step Down"
- note added: "SHDN pin has max 7V. Could use as UVLO,\nbut easier to add a couple of useful "external"\npower LEDs, use the junction volage to create\nthe shutdown voltage."
- note added: "Screw terminals for 9V-25V input\n"
- note removed: "Power Supply"
- note removed: "Screw terminals for 9V-18V input\nWill also power the Pi"
- moved on the sheet: C301, C302, C303, C304, C305, C306, C307, D302, D303, D304, L301, L302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
