File: Schematics/ClockFanout.sch (KiCad schematic (older format))
At the start: 20 parts, among them CN401 COAX, CN402 COAX, CN405 COAX, CN406 COAX, U401 NB3L553

Commit message: WIP
Parts:
- removed CN402, CN405: COAX, OHDSP-Footprints-Pretty:CONN-RF-UFL, symbol COAX
- added C401, C403: 33p, symbol C
- added R401, R404: N/F, symbol R
- added R402: 100R, symbol R
- added X401: 24M576, symbol CRYSTAL
- C402: renamed from C401; footprint OHDSP-Footprints-Pretty:SMD-0805 -> (none)
- C404: renamed from C403; footprint OHDSP-Footprints-Pretty:SMD-0805 -> (none)
- C405: renamed from C404; footprint OHDSP-Footprints-Pretty:SMD-0805 -> (none)
- CN401: footprint OHDSP-Footprints-Pretty:CONN-RF-UFL -> (none)
- CN402: renamed from CN406; footprint OHDSP-Footprints-Pretty:CONN-RF-UFL -> (none)
- L401: footprint OHDSP-Footprints-Pretty:SMD-0805 -> (none)
- R403: renamed from R401; footprint OHDSP-Footprints-Pretty:SMD-0805 -> (none)
- R405: renamed from R402; footprint OHDSP-Footprints-Pretty:TH-RES-0W25 -> (none)
- R406: renamed from R404; footprint OHDSP-Footprints-Pretty:SMD-0805 -> (none)
- R407: renamed from R406; value 27R -> 75R; footprint OHDSP-Footprints-Pretty:SMD-0805 -> (none)
- R408: renamed from R407; value 27R -> 75R; footprint OHDSP-Footprints-Pretty:SMD-0805 -> (none)
- R409: renamed from R408; value 27R -> 75R; footprint OHDSP-Footprints-Pretty:SMD-0805 -> (none)
- R410: renamed from R409; footprint OHDSP-Footprints-Pretty:SMD-0805 -> (none)
- R411: renamed from R414; footprint OHDSP-Footprints-Pretty:SMD-0805 -> (none)
- R412: renamed from R418; footprint OHDSP-Footprints-Pretty:SMD-0805 -> (none)
- R413: renamed from R415; footprint OHDSP-Footprints-Pretty:SMD-0805 -> (none)
- R414: renamed from R419; footprint OHDSP-Footprints-Pretty:SMD-0805 -> (none)
- U401: footprint OHDSP-Footprints-Pretty:IC_SOIC_8 -> (none)
Connections:
- net MCLKC2 is gone; now on net GNDD: R408.1, R412.2
- net MCLKC3 is gone; now on net GNDD: R409.1, R413.2
- net GNDD: now also R407.1, R411.2, C401.2, C403.2, R401.2
- net MCLKA1: no longer R405.1, U401.5 (ICLK)
- net at C404.1, C405.1, L401.2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: no longer R406.2, U401.1 (Vdd)
- removed net MCLKC1: CN401.1, R407.1, R411.2
- net MCLK_IN: no longer names the net of R405.2
- new net: R406.2, U401.1 (Vdd)
- new net: C401.1, X401.1
- new net: C403.1, R402.2, X401.2
- new net: CN401.1, R404.2
Other:
- note added: "External Clock"
- note added: "Master Audio Clock"
- note added: "Master Clock - Two Options"
- note added: "Standard Crystal"
- note removed: "ADAU1452 Master Audio Clock Fanout"
- note removed: "Four clock outputs, suggest using external\nclock for more"
- moved on the sheet: C402, C404, C405, CN402, L401, R403, R405, R406, R407, R408, R409, R410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

Commit message: WIP
Parts:
- added C404: 220u, OHDSP-Footprints-Pretty:SMD-0805, symbol CP1
- added C407, C409: 100n, symbol C
- added C408, C410: 22u, symbol C
- added C411: 100p, symbol C
- added L402: 600R@100MHz, symbol INDUCTOR
- added R402: 1Meg, OHDSP-Footprints-Pretty:SMD-0805, symbol R
- added R406, R407: 0R, OHDSP-Footprints-Pretty:SMD-0805, symbol R
- added R410: 100R, OHDSP-Footprints-Pretty:SMD-0805, symbol R
- added R411: 47R, OHDSP-Footprints-Pretty:SMD-0805, symbol R
- added U401: NC7SZU04M5X, OHDSP-Footprints-Pretty:IC_SOIC_8, symbol IC-LOGIC-NC7SZU04M5X
- added U402: NC7SZU04M5X, symbol IC-LOGIC-NC7SZU04M5X
- C401, L401: footprint (none) -> OHDSP-Footprints-Pretty:SMD-0805
- C402: renamed from C403; footprint (none) -> OHDSP-Footprints-Pretty:SMD-0805
- C403: renamed from C402; footprint (none) -> OHDSP-Footprints-Pretty:SMD-0805
- C405: renamed from C404; footprint (none) -> OHDSP-Footprints-Pretty:SMD-0805
- CN401, CN402: footprint (none) -> OHDSP-Footprints-Pretty:CONN-RF-UFL
- R401: renamed from R404; footprint (none) -> OHDSP-Footprints-Pretty:SMD-0805
- R403: renamed from R401; footprint (none) -> OHDSP-Footprints-Pretty:SMD-0805
- R404: renamed from R402; footprint (none) -> OHDSP-Footprints-Pretty:SMD-0805
- R405: renamed from R403; footprint (none) -> OHDSP-Footprints-Pretty:SMD-0805
- R408: renamed from R405; value 75R -> 0R; footprint (none) -> OHDSP-Footprints-Pretty:SMD-0805
- R409: renamed from R406; footprint (none) -> OHDSP-Footprints-Pretty:SMD-0805
- R412: renamed from R407; footprint (none) -> OHDSP-Footprints-Pretty:SMD-0805
- R413: renamed from R408; footprint (none) -> OHDSP-Footprints-Pretty:SMD-0805
- R414: renamed from R409; footprint (none) -> OHDSP-Footprints-Pretty:SMD-0805
- X401: footprint (none) -> OHDSP-Footprints-Pretty:XTAL_HC49_TH
- renumbered C405 to C406, R410 to R415, R411 to R416, R412 to R417, R413 to R418, R414 to R419, U401 to U403
Connections:
- net GNDD: now also C404.2, C407.2, C408.2, C409.2, C410.2, C411.2, R410.1, U401.3 (GND), U402.3 (GND)
- net VPP: now also L402.1
- net at U403.1 (Vdd): now also C405.1, C406.1, L401.2, R405.1, C404.1; no longer R409.2
- net at U403.5 (ICLK): now also R408.1, R410.2
- net CLK: now reaches R408.2
- net at C401.1, X401.1: now also R402.1, U401.2 (A)
- net at C402.1, X401.2: now also R404.1; no longer R404.2
- net at R401.1: now also R403.1, R406.1
- new net: R402.2, R404.2, U401.4 (Y), U402.2 (A)
- new net: C407.1, C408.1, C409.1, C410.1, L402.2, R411.1, U401.5 (Vcc), U402.5 (Vcc)
- new net: R407.2, U402.4 (Y)
- new net: C411.1, R411.2
- new net: R406.2, R407.1
- no-connect marks 0 -> 1
Other:
- moved on the sheet: C401, C402, C403, C405, C406, CN401, CN402, L401, R401, R403, R404, R405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

Commit message: WIP
Parts:
- C406, C407, C408, C409, C410, C411, L402, R415, R416, R417, R418, R419: footprint (none) -> OHDSP-Footprints-Pretty:SMD-0805
- U401: footprint OHDSP-Footprints-Pretty:IC_SOIC_8 -> OHDSP-Footprints-Pretty:IC-SOT23-5
- U402: footprint (none) -> OHDSP-Footprints-Pretty:IC-SOT23-5
- U403: footprint (none) -> OHDSP-Footprints-Pretty:IC_SOIC_8
Connections:
- net GNDD: no longer R412.1, R413.1, R414.1, R416.2, R417.2, R418.2
- new net MCLK_OUT1: R412.1, R416.2
- new net MCLK_OUT2: R413.1, R417.2
- new net MCLK_OUT3: R414.1, R418.2
- no-connect marks 1 -> 2
Changed lines of the file:
@@
 F 0 "U403" H 5500 2100 60  0000 C CNN
 F 1 "NB3L553" H 5650 2000 60  0000 C CNN
-F 2 "" H 5250 1850 60  0001 C CNN
+F 2 "OHDSP-Footprints-Pretty:IC_SOIC_8" H 5250 1850 60  0001 C CNN
 F 3 "" H 5250 1850 60  0000 C CNN
 	1    5250 1850
@@
 F 0 "R415" V 6730 2300 40  0000 C CNN
 F 1 "27R" V 6657 2301 40  0000 C CNN
-F 2 "" V 6580 2300 30  0001 C CNN
+F 2 "OHDSP-Footprints-Pretty:SMD-0805" V 6580 2300 30  0001 C CNN
 F 3 "" H 6650 2300 30  0000 C CNN
 	1    6650 2300
@@
 $EndComp
 $Comp
-L GNDD #PWR409
+L GNDD #PWR081
 U 1 1 54E21AA5
 P 4350 2350
-F 0 "#PWR409" H 4350 2100 60  0001 C CNN
+F 0 "#PWR081" H 4350 2100 60  0001 C CNN
 F 1 "GNDD" H 4350 2200 60  0000 C CNN
 F 2 "" H 4350 2350 60  0000 C CNN
@@
 F 0 "R416" V 7630 1350 40  0000 C CNN
 F 1 "N/F" V 7557 1351 40  0000 C CNN
-F 2 "" V 7480 1350 30  0001 C CNN
+F 2 "OHDSP-Footprints-Pretty:SMD-0805" V 7480 1350 30  0001 C CNN
 F 3 "" H 7550 1350 30  0000 C CNN
 	1    7550 1350
@@
 $EndComp
 $Comp
-L GNDD #PWR413
+L GNDD #PWR082
 U 1 1 54E223FC
 P 7900 1400
-F 0 "#PWR413" H 7900 1150 60  0001 C CNN
+F 0 "#PWR082" H 7900 1150 60  0001 C CNN
 F 1 "GNDD" H 7900 1250 60  0000 C CNN
 F 2 "" H 7900 1400 60  0000 C CNN
@@
 F 0 "R417" V 7630 1900 40  0000 C CNN
 F 1 "N/F" V 7557 1901 40  0000 C CNN
-F 2 "" V 7480 1900 30  0001 C CNN
+F 2 "OHDSP-Footprints-Pretty:SMD-0805" V 7480 1900 30  0001 C CNN
 F 3 "" H 7550 1900 30  0000 C CNN
 	1    7550 1900
@@
 $EndComp
 $Comp
-L GNDD #PWR414
+L GNDD #PWR083
 U 1 1 54E228B4
 P 7900 1950
-F 0 "#PWR414" H 7900 1700 60  0001 C CNN
+F 0 "#PWR083" H 7900 1700 60  0001 C CNN
 F 1 "GNDD" H 7900 1800 60  0000 C CNN
 F 2 "" H 7900 1950 60  0000 C CNN
@@
 F 0 "R418" V 7630 2500 40  0000 C CNN
 F 1 "N/F" V 7557 2501 40  0000 C CNN
-F 2 "" V 7480 2500 30  0001 C CNN
+F 2 "OHDSP-Footprints-Pretty:SMD-0805" V 7480 2500 30  0001 C CNN
 F 3 "" H 7550 2500 30  0000 C CNN
 	1    7550 2500
@@
 $EndComp
 $Comp
-L GNDD #PWR415
+L GNDD #PWR084
 U 1 1 54E22C88
 P 7900 2550
-F 0 "#PWR415" H 7900 2300 60  0001 C CNN
+F 0 "#PWR084" H 7900 2300 60  0001 C CNN
 F 1 "GNDD" H 7900 2400 60  0000 C CNN
 F 2 "" H 7900 2550 60  0000 C CNN
@@
 F 0 "R419" V 7630 3100 40  0000 C CNN
 F 1 "N/F" V 7557 3101 40  0000 C CNN
-F 2 "" V 7480 3100 30  0001 C CNN
+F 2 "OHDSP-Footprints-Pretty:SMD-0805" V 7480 3100 30  0001 C CNN
 F 3 "" H 7550 3100 30  0000 C CNN
 	1    7550 3100
@@
 $EndComp
 $Comp
-L GNDD #PWR416
+L GNDD #PWR085
 U 1 1 54E22D69
 P 7900 3150
-F 0 "#PWR416" H 7900 2900 60  0001 C CNN
+F 0 "#PWR085" H 7900 2900 60  0001 C CNN
 F 1 "GNDD" H 7900 3000 60  0000 C CNN
 F 2 "" H 7900 3150 60  0000 C CNN
@@
 $EndComp
 $Comp
-L GNDD #PWR408
+L GNDD #PWR086
 U 1 1 54E607CE
 P 2900 3000
-F 0 "#PWR408" H 2900 2750 60  0001 C CNN
+F 0 "#PWR086" H 2900 2750 60  0001 C CNN
 F 1 "GNDD" H 2900 2850 60  0000 C CNN
 F 2 "" H 2900 3000 60  0000 C CNN
@@
 F 0 "C406" H 3900 2550 40  0000 L CNN
 F 1 "100n" H 3906 2365 40  0000 L CNN
-F 2 "" H 3938 2300 30  0000 C CNN
+F 2 "OHDSP-Footprints-Pretty:SMD-0805" H 3938 2300 30  0001 C CNN
 F 3 "~" H 3900 2450 60  0000 C CNN
 	1    3900 2450
@@
 $EndComp
 $Comp
-L VPP #PWR404
+L VPP #PWR087
 U 1 1 54E24C37
 P 2050 1700
-F 0 "#PWR404" H 2050 1550 60  0001 C CNN
+F 0 "#PWR087" H 2050 1550 60  0001 C CNN
 F 1 "VPP" H 2050 1850 60  0000 C CNN
 F 2 "" H 2050 1700 60  0000 C CNN
@@
 $EndComp
 $Comp
-L GNDD #PWR403
+L GNDD #PWR088
 U 1 1 5514C512
 P 1250 6200
-F 0 "#PWR403" H 1250 5950 60  0001 C CNN
+F 0 "#PWR088" H 1250 5950 60  0001 C CNN
 F 1 "GNDD" H 1250 6050 60  0000 C CNN
 F 2 "" H 1250 6200 60  0000 C CNN
@@
 $EndComp
 $Comp
-L GNDD #PWR406
+L GNDD #PWR089
 U 1 1 5514C518
 P 2450 6200
-F 0 "#PWR406" H 2450 5950 60  0001 C CNN
+F 0 "#PWR089" H 2450 5950 60  0001 C CNN
 F 1 "GNDD" H 2450 6050 60  0000 C CNN
 F 2 "" H 2450 6200 60  0000 C CNN
@@
 $EndComp
 $Comp
-L GNDD #PWR402
+L GNDD #PWR090
 U 1 1 5514C525
 P 1150 7000
-F 0 "#PWR402" H 1150 6750 60  0001 C CNN
+F 0 "#PWR090" H 1150 6750 60  0001 C CNN
 F 1 "GNDD" H 1150 6850 60  0000 C CNN
 F 2 "" H 1150 7000 60  0000 C CNN
@@
 $EndComp
 $Comp
-L GNDD #PWR405
+L GNDD #PWR091
 U 1 1 5514C53E
 P 2250 7450
-F 0 "#PWR405" H 2250 7200 60  0001 C CNN
+F 0 "#PWR091" H 2250 7200 60  0001 C CNN
 F 1 "GNDD" H 2250 7300 60  0000 C CNN
 F 2 "" H 2250 7450 60  0000 C CNN
@@
 	7200 1150 8150 1150
 Wire Wire Line
-	7900 1150 7900 1400
-Wire Wire Line
 	7800 1350 7900 1350
-Connection ~ 7900 1350
 Wire Wire Line
 	6950 1350 7300 1350
@@
 	7200 1350 7200 1150
 Wire Wire Line
-	7900 1700 7900 1950
-Wire Wire Line
-	7800 1900 7900 1900
-Connection ~ 7900 1900
-Wire Wire Line
 	7200 1900 7300 1900
 Wire Wire Line
 	7200 1700 7200 2000
 Wire Wire Line
-	7900 2300 7900 2550
-Wire Wire Line
 	7800 2500 7900 2500
-Connection ~ 7900 2500
 Wire Wire Line
 	7200 2500 7300 2500
@@
 Text HLabel 8150 2300 2    60   Output ~ 0
 MCLK_OUT3
-Connection ~ 7900 1150
-Connection ~ 7900 1700
-Connection ~ 7900 2300
 $Comp
 L IC-LOGIC-NC7SZU04M5X U401
@@
 F 0 "U401" H 1600 4700 60  0000 C CNN
 F 1 "NC7SZU04M5X" H 1800 4600 60  0000 C CNN
-F 2 "OHDSP-Footprints-Pretty:IC_SOIC_8" H 1350 4600 60  0001 C CNN
+F 2 "OHDSP-Footprints-Pretty:IC-SOT23-5" H 1350 4600 60  0001 C CNN
 F 3 "" H 1350 4600 60  0000 C CNN
 	1    1350 4450
@@
 Connection ~ 1250 4900
 $Comp
-L GNDD #PWR401
+L GNDD #PWR092
 U 1 1 55159F7A
 P 1100 4900
-F 0 "#PWR401" H 1100 4650 60  0001 C CNN
+F 0 "#PWR092" H 1100 4650 60  0001 C CNN
 F 1 "GNDD" H 1100 4750 60  0000 C CNN
 F 2 "" H 1100 4900 60  0000 C CNN
@@
 F 0 "U402" H 3050 4800 60  0000 C CNN
 F 1 "NC7SZU04M5X" H 3250 4700 60  0000 C CNN
-F 2 "" H 2800 4700 60  0000 C CNN
+F 2 "OHDSP-Footprints-Pretty:IC-SOT23-5" H 2800 4700 60  0001 C CNN
 F 3 "" H 2800 4700 60  0000 C CNN
 	1    2800 4550
@@
 Connection ~ 2450 4650
 $Comp
-L GNDD #PWR407
+L GNDD #PWR093
 U 1 1 5515ACFE
 P 2700 4800
-F 0 "#PWR407" H 2700 4550 60  0001 C CNN
+F 0 "#PWR093" H 2700 4550 60  0001 C CNN
 F 1 "GNDD" H 2700 4650 60  0000 C CNN
 F 2 "" H 2700 4800 60  0000 C CNN
@@
 F 0 "L402" V 5900 4350 40  0000 C CNN
 F 1 "600R@100MHz" V 6050 4350 40  0000 C CNN
-F 2 "" H 5950 4350 60  0001 C CNN
+F 2 "OHDSP-Footprints-Pretty:SMD-0805" H 5950 4350 60  0001 C CNN
 F 3 "~" H 5950 4350 60  0000 C CNN
 	1    5950 4350
@@
 F 0 "C411" H 5500 5300 40  0000 L CNN
 F 1 "100p" H 5506 5115 40  0000 L CNN
-F 2 "" H 5538 5050 30  0000 C CNN
+F 2 "OHDSP-Footprints-Pretty:SMD-0805" H 5538 5050 30  0001 C CNN
 F 3 "~" H 5500 5200 60  0000 C CNN
 	1    5500 5200
@@
 $EndComp
 $Comp
-L GNDD #PWR411
+L GNDD #PWR094
 U 1 1 5515C3B2
 P 5500 5500
-F 0 "#PWR411" H 5500 5250 60  0001 C CNN
+F 0 "#PWR094" H 5500 5250 60  0001 C CNN
 F 1 "GNDD" H 5500 5350 60  0000 C CNN
 F 2 "" H 5500 5500 60  0000 C CNN
@@
 F 0 "C409" H 4900 5050 40  0000 L CNN
 F 1 "100n" H 4906 4865 40  0000 L CNN
-F 2 "" H 4938 4800 30  0000 C CNN
+F 2 "OHDSP-Footprints-Pretty:SMD-0805" H 4938 4800 30  0001 C CNN
 F 3 "~" H 4900 4950 60  0000 C CNN
 	1    4900 4950
@@
 F 0 "C410" H 5200 5050 40  0000 L CNN
 F 1 "22u" H 5206 4865 40  0000 L CNN
-F 2 "" H 5238 4800 30  0000 C CNN
+F 2 "OHDSP-Footprints-Pretty:SMD-0805" H 5238 4800 30  0001 C CNN
 F 3 "~" H 5200 4950 60  0000 C CNN
 	1    5200 4950
@@
 $EndComp
 $Comp
-L VPP #PWR412
+L VPP #PWR095
 U 1 1 5515C3C4
 P 6350 4200
-F 0 "#PWR412" H 6350 4050 60  0001 C CNN
+F 0 "#PWR095" H 6350 4050 60  0001 C CNN
 F 1 "VPP" H 6350 4350 60  0000 C CNN
 F 2 "" H 6350 4200 60  0000 C CNN
@@
 F 0 "C407" H 4300 5050 40  0000 L CNN
 F 1 "100n" H 4306 4865 40  0000 L CNN
-F 2 "" H 4338 4800 30  0000 C CNN
+F 2 "OHDSP-Footprints-Pretty:SMD-0805" H 4338 4800 30  0001 C CNN
 F 3 "~" H 4300 4950 60  0000 C CNN
 	1    4300 4950
@@
 Connection ~ 5100 2000
 $Comp
-L GNDD #PWR410
+L GNDD #PWR096
 U 1 1 55160014
 P 5100 3000
-F 0 "#PWR410" H 5100 2750 60  0001 C CNN
+F 0 "#PWR096" H 5100 2750 60  0001 C CNN
 F 1 "GNDD" H 5100 2850 60  0000 C CNN
 F 2 "" H 5100 3000 60  0000 C CNN
@@
 F 0 "C408" H 4600 5050 40  0000 L CNN
 F 1 "22u" H 4606 4865 40  0000 L CNN
-F 2 "" H 4638 4800 30  0000 C CNN
+F 2 "OHDSP-Footprints-Pretty:SMD-0805" H 4638 4800 30  0001 C CNN
 F 3 "~" H 4600 4950 60  0000 C CNN
 	1    4600 4950
@@
 	4600 5150 4600 5450
 Connection ~ 4600 5450
+NoConn ~ 2800 4550
+Wire Wire Line
+	7900 1350 7900 1400
+Wire Wire Line
+	7800 1900 7900 1900
+Wire Wire Line
+	7900 1900 7900 1950
+Wire Wire Line
+	7900 2500 7900 2550
 $EndSCHEMATC

Commit message: WIP
Connections:
- net CLK: now also R406.2, R407.1
- net at C404.1, C405.1, C406.1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: now also R409.2
Changed lines of the file:
@@
 $EndComp
 $Comp
-L GNDD #PWR081
+L GNDD #PWR080
 U 1 1 54E21AA5
 P 4350 2350
-F 0 "#PWR081" H 4350 2100 60  0001 C CNN
+F 0 "#PWR080" H 4350 2100 60  0001 C CNN
 F 1 "GNDD" H 4350 2200 60  0000 C CNN
 F 2 "" H 4350 2350 60  0000 C CNN
@@
 $EndComp
 $Comp
-L GNDD #PWR082
+L GNDD #PWR081
 U 1 1 54E223FC
 P 7900 1400
-F 0 "#PWR082" H 7900 1150 60  0001 C CNN
+F 0 "#PWR081" H 7900 1150 60  0001 C CNN
 F 1 "GNDD" H 7900 1250 60  0000 C CNN
 F 2 "" H 7900 1400 60  0000 C CNN
@@
 $EndComp
 $Comp
-L GNDD #PWR083
+L GNDD #PWR082
 U 1 1 54E228B4
 P 7900 1950
-F 0 "#PWR083" H 7900 1700 60  0001 C CNN
+F 0 "#PWR082" H 7900 1700 60  0001 C CNN
 F 1 "GNDD" H 7900 1800 60  0000 C CNN
 F 2 "" H 7900 1950 60  0000 C CNN
@@
 $EndComp
 $Comp
-L GNDD #PWR084
+L GNDD #PWR083
 U 1 1 54E22C88
 P 7900 2550
-F 0 "#PWR084" H 7900 2300 60  0001 C CNN
+F 0 "#PWR083" H 7900 2300 60  0001 C CNN
 F 1 "GNDD" H 7900 2400 60  0000 C CNN
 F 2 "" H 7900 2550 60  0000 C CNN
@@
 $EndComp
 $Comp
-L GNDD #PWR085
+L GNDD #PWR084
 U 1 1 54E22D69
 P 7900 3150
-F 0 "#PWR085" H 7900 2900 60  0001 C CNN
+F 0 "#PWR084" H 7900 2900 60  0001 C CNN
 F 1 "GNDD" H 7900 3000 60  0000 C CNN
 F 2 "" H 7900 3150 60  0000 C CNN
@@
 $EndComp
 $Comp
-L GNDD #PWR086
+L GNDD #PWR085
 U 1 1 54E607CE
 P 2900 3000
-F 0 "#PWR086" H 2900 2750 60  0001 C CNN
+F 0 "#PWR085" H 2900 2750 60  0001 C CNN
 F 1 "GNDD" H 2900 2850 60  0000 C CNN
 F 2 "" H 2900 3000 60  0000 C CNN
@@
 $EndComp
 $Comp
-L VPP #PWR087
+L VPP #PWR086
 U 1 1 54E24C37
 P 2050 1700
-F 0 "#PWR087" H 2050 1550 60  0001 C CNN
+F 0 "#PWR086" H 2050 1550 60  0001 C CNN
 F 1 "VPP" H 2050 1850 60  0000 C CNN
 F 2 "" H 2050 1700 60  0000 C CNN
@@
 $EndComp
 $Comp
-L GNDD #PWR088
+L GNDD #PWR087
 U 1 1 5514C512
 P 1250 6200
-F 0 "#PWR088" H 1250 5950 60  0001 C CNN
+F 0 "#PWR087" H 1250 5950 60  0001 C CNN
 F 1 "GNDD" H 1250 6050 60  0000 C CNN
 F 2 "" H 1250 6200 60  0000 C CNN
@@
 $EndComp
 $Comp
-L GNDD #PWR089
+L GNDD #PWR088
 U 1 1 5514C518
 P 2450 6200
-F 0 "#PWR089" H 2450 5950 60  0001 C CNN
+F 0 "#PWR088" H 2450 5950 60  0001 C CNN
 F 1 "GNDD" H 2450 6050 60  0000 C CNN
 F 2 "" H 2450 6200 60  0000 C CNN
@@
 $EndComp
 $Comp
-L GNDD #PWR090
+L GNDD #PWR089
 U 1 1 5514C525
 P 1150 7000
-F 0 "#PWR090" H 1150 6750 60  0001 C CNN
+F 0 "#PWR089" H 1150 6750 60  0001 C CNN
 F 1 "GNDD" H 1150 6850 60  0000 C CNN
 F 2 "" H 1150 7000 60  0000 C CNN
@@
 $EndComp
 $Comp
-L GNDD #PWR091
+L GNDD #PWR090
 U 1 1 5514C53E
 P 2250 7450
-F 0 "#PWR091" H 2250 7200 60  0001 C CNN
+F 0 "#PWR090" H 2250 7200 60  0001 C CNN
 F 1 "GNDD" H 2250 7300 60  0000 C CNN
 F 2 "" H 2250 7450 60  0000 C CNN
@@
 Connection ~ 1250 4900
 $Comp
-L GNDD #PWR092
+L GNDD #PWR091
 U 1 1 55159F7A
 P 1100 4900
-F 0 "#PWR092" H 1100 4650 60  0001 C CNN
+F 0 "#PWR091" H 1100 4650 60  0001 C CNN
 F 1 "GNDD" H 1100 4750 60  0000 C CNN
 F 2 "" H 1100 4900 60  0000 C CNN
@@
 Wire Wire Line
 	5000 2000 5250 2000
-Wire Wire Line
-	4500 2000 4050 2000
 Text Label 4050 2000 0    60   ~ 0
 CLK
-Text Label 4150 6700 2    60   ~ 0
+Text Label 4150 6750 2    60   ~ 0
 CLK
 $Comp
@@
 Connection ~ 2450 4650
 $Comp
-L GNDD #PWR093
+L GNDD #PWR092
 U 1 1 5515ACFE
 P 2700 4800
-F 0 "#PWR093" H 2700 4550 60  0001 C CNN
+F 0 "#PWR092" H 2700 4550 60  0001 C CNN
 F 1 "GNDD" H 2700 4650 60  0000 C CNN
 F 2 "" H 2700 4800 60  0000 C CNN
@@
 $EndComp
 $Comp
-L GNDD #PWR094
+L GNDD #PWR093
 U 1 1 5515C3B2
 P 5500 5500
-F 0 "#PWR094" H 5500 5250 60  0001 C CNN
+F 0 "#PWR093" H 5500 5250 60  0001 C CNN
 F 1 "GNDD" H 5500 5350 60  0000 C CNN
 F 2 "" H 5500 5500 60  0000 C CNN
@@
 $EndComp
 $Comp
-L VPP #PWR095
+L VPP #PWR094
 U 1 1 5515C3C4
 P 6350 4200
-F 0 "#PWR095" H 6350 4050 60  0001 C CNN
+F 0 "#PWR094" H 6350 4050 60  0001 C CNN
 F 1 "VPP" H 6350 4350 60  0000 C CNN
 F 2 "" H 6350 4200 60  0000 C CNN
@@
 Connection ~ 5100 2000
 $Comp
-L GNDD #PWR096
+L GNDD #PWR095
 U 1 1 55160014
 P 5100 3000
-F 0 "#PWR096" H 5100 2750 60  0001 C CNN
+F 0 "#PWR095" H 5100 2750 60  0001 C CNN
 F 1 "GNDD" H 5100 2850 60  0000 C CNN
 F 2 "" H 5100 3000 60  0000 C CNN
@@
 Wire Wire Line
 	7900 2500 7900 2550
+Connection ~ 4400 1850
+Wire Wire Line
+	4050 2000 4500 2000
 $EndSCHEMATC
