File: Schematics/ClockFanout.sch (KiCad schematic (older format))
At the start: 38 parts, among them CN401 COAX, CN402 COAX, U401 NC7SZU04M5X, U402 NC7SZU04M5X, U403 NB3L553, X401 24M576

Commit message: WIP
Parts:
- C404: footprint OHDSP-Footprints-Pretty:SMD-0805 -> OHDSP-Footprints-Pretty:CAP-TH-D6.3mmP2.5mm
Changed lines of the file:
@@
 Wire Wire Line
 	4400 2150 4400 1850
+Text HLabel 8150 1700 2    60   Output ~ 0
+MCLK_OUT1
 Text HLabel 8150 1150 2    60   Output ~ 0
-MCLK_OUT1
-Text HLabel 8150 1700 2    60   Output ~ 0
 MCLK_OUT2
 Text HLabel 8150 2300 2    60   Output ~ 0
@@
 F 0 "C404" H 3300 2550 50  0000 L CNN
 F 1 "220u" H 3300 2350 50  0000 L CNN
-F 2 "OHDSP-Footprints-Pretty:SMD-0805" H 3250 2450 60  0001 C CNN
+F 2 "OHDSP-Footprints-Pretty:CAP-TH-D6.3mmP2.5mm" H 3250 2450 60  0001 C CNN
 F 3 "~" H 3250 2450 60  0000 C CNN
 	1    3250 2450

Commit message: WIP
Parts:
- removed C401: 33p, OHDSP-Footprints-Pretty:SMD-0805, symbol C
- removed C403, C411: 100p, OHDSP-Footprints-Pretty:SMD-0805, symbol C
- removed C409: 100n, OHDSP-Footprints-Pretty:SMD-0805, symbol C
- removed C410: 22u, OHDSP-Footprints-Pretty:SMD-0805, symbol C
- removed R401, R416, R417, R418: N/F, OHDSP-Footprints-Pretty:SMD-0805, symbol R
- removed R402: 1Meg, OHDSP-Footprints-Pretty:SMD-0805, symbol R
- removed R405, R411: 47R, OHDSP-Footprints-Pretty:SMD-0805, symbol R
- removed R408: 0R, OHDSP-Footprints-Pretty:SMD-0805, symbol R
- removed R410: 100R, OHDSP-Footprints-Pretty:SMD-0805, symbol R
- removed U401, U402: NC7SZU04M5X, OHDSP-Footprints-Pretty:IC-SOT23-5, symbol IC-LOGIC-NC7SZU04M5X
- removed X401: 24M576, OHDSP-Footprints-Pretty:XTAL_HC49_TH, symbol CRYSTAL
- added XTAL401: XTAL-OSC-4PIN, OHDSP-Footprints-Pretty:XTAL_8_DIL, symbol XTAL-OSC-4PIN
- C402: value 33p -> 100n
- R404: value 100R -> 1k
- R406: value 0R -> N/F
- R407: value 0R -> 27R
Connections:
- wire segments 96 -> 53
- no-connect marks 2 -> 0
Other:
- moved on the sheet: C402, C407, C408, CN401, L402, R403, R404, R406, R407
