File: Schematics/OHDSP-ADAU1701.kicad_pcb (KiCad board)
At the start: 4 copper layers, 100 x 100 mm, 382 parts, among them CN201 COAX, CN401 COAX, CN402 COAX, CN405 COAX, CN406 COAX, CN701 COAX, CN702 COAX, P201 CONN_2x1, P203 CONN_6X2, P204 CONN_6x1, P301 CONN_2x1, P302 CONN_2x1, P303 PIN, P304 PIN, P305 PIN, P306 PIN, P601 CONN_02X05, P602 CONN_02X05, P603 CONN_02X05, P604 CONN_02X05, P605 CONN_02X05, P606 CONN_6X2, P607 CONN_02X05, P608 CONN_02X05, P609 CONN_02X20, P610 CONN_02X05, P611 CONN_02X05, P612 CONN_02X05, P613 CONN_02X05, P614 CONN_02X05, P615 CONN_02X05, P616 CONN_02X05, P701 CONN_02X05, P702 CONN_2x1, P703 CONN_02X05, P704 CONN_3x1, P705 CONN_3x1, SW202 SWITCH, U201 ADAU1452WBCPZ, U202 ADM13307-5ARZ, U203 25AA1024, U301 IC-REG-XRP7659ISTR-F, U302 IC-REG-XRP7659ISTR-F, U304 IC-REG-XC6210B332MR, U305 IC-REG-XC6210B332MR, U401 NB3L553, U501 IC-SPDIF-RX-OPTO, U502 IC-SPDIF-TX-OPTO, U701 IC-REG-LM317-TO220, U702 IC-DAC-WM8501, U703 IC-ADC-WM8783, U704 IC-REG-XC6210B332MR, X201 24M576

Commit message: WIP
Parts:
- removed the C205 at (266.2, 77.5)
- removed the C212 at (265.2, 96.8)
- removed the C213 at (281.4, 98.6)
- removed the C215 at (280.5, 99.3)
- removed the C217 at (278.6, 99.2)
- removed the C220 at (281.4, 86.5)
- removed the C221 at (267.2, 81.8)
- removed the C222 at (267.2, 80.4)
- removed the C223 at (279.9, 86.5)
- removed the C226 at (259.2, 105.0)
- removed the C230 at (269.5, 86.0)
- removed the C232 at (267.0, 84.6)
- removed the C233 at (266.6, 98.9)
- removed the C234 at (266.6, 98.9)
- removed the C238 at (258.1, 89.0)
- removed C241, C711, C713, C714, C723, C724, C725, C727: 22u, OHDSP-Footprints-Pretty:SMD-0805
- removed the C315 at (213.9, 95.0)
- removed the C321 at (206.6, 82.2)
- removed the C328 at (223.3, 84.1)
- removed C340, C341, C731, C736, C737: 100u, OHDSP-Footprints-Pretty:CAP-TH-D6.3mmP2.5mm
- removed the C404 at (253.1, 116.5)
- removed C601, C707, C710, C720, C721, C722, C726, C735: 100n, OHDSP-Footprints-Pretty:SMD-0805
- removed C605: 220u, OHDSP-Footprints-Pretty:CAP-TH-D6.3mmP2.5mm
- removed C701, C703, C705: 220u, OHDSP-Footprints-Pretty:CAP-TH-D8mmP3.5mm
- removed C702, C704, C706, C716: 10n, OHDSP-Footprints-Pretty:CAP_TH_5mm
- removed C708, C709, C712, C715: 100u, OHDSP-Footprints-Pretty:CAP-TH-D10mmP5mm
- removed C717, C718: 1n, OHDSP-Footprints-Pretty:SMD-0805
- removed C719: 10n, OHDSP-Footprints-Pretty:SMD-0805
- removed C732, C733, C734: 100p, OHDSP-Footprints-Pretty:SMD-0805
- removed CN201, CN405, CN701, CN702: COAX, OHDSP-Footprints-Pretty:CONN-RF-UFL
- removed the CN402 at (246.4, 121.4)
- removed the D303 at (213.6, 76.5)
- removed D306: LED, OHDSP-Footprints-Pretty:SMD-1206
- removed D601, D602, D603, D604, D605, D606, D607, D608, D609, D610, D611, D612: 1N5818, OHDSP-Footprints-Pretty:DIODE-DO-41
- removed D701: SS24T3G, OHDSP-Footprints-Pretty:DIODE-SMB
- removed the L302 at (217.2, 81.8)
- removed the L501 at (277.6, 64.0)
- removed L701, L702, L703, L704: 600R@100MHz, OHDSP-Footprints-Pretty:SMD-0805
- removed P203, P606: CONN_6X2, OHDSP-Footprints-Pretty:CONN_DIL_2X6
- removed P204: CONN_6x1, OHDSP-Footprints-Pretty:CONN_SIL_6
- removed the P303 at (223.5, 120.5)
- removed P601, P602, P603, P604, P613, P614, P615, P616, P701, P703: CONN_02X05, OHDSP-Footprints-Pretty:CONN_DIL_2X5
- removed P702: CONN_2x1, OHDSP-Footprints-Pretty:CONN-SCREW-2WAY-5mm-5.08mm
- removed P704, P705: CONN_3x1, OHDSP-Footprints-Pretty:CONN_SIL_3
- removed the R230 at (247.5, 88.3)
- removed the R231 at (213.9, 116.3)
- removed the R232 at (213.9, 112.0)
- removed R233: 1k, OHDSP-Footprints-Pretty:SMD-0805
- removed the R304 at (209.7, 87.0)
- removed the R305 at (207.5, 85.1)
- removed the R502 at (295.1, 60.6)
- removed the R503 at (277.9, 80.3)
- removed the R504 at (286.0, 73.9)
- removed R607, R608, R609, R610, R611, R612, R613, R614, R615: 0R, OHDSP-Footprints-Pretty:SMD-0603
- removed R617, R618, R619, R621, R622, R623, R624, R625, R626, R627, R663, R664, R665, R667, R668, R669, R671, R672, R673: N/F, OHDSP-Footprints-Pretty:SMD-0603
- removed R631, R632, R633, R642, R644, R701, R703, R707, R709: 0R, OHDSP-Footprints-Pretty:SMD-0805
- removed R635, R636, R637, R638, R639, R640: 4k7, OHDSP-Footprints-Pretty:SMD-0805
- removed R648, R726, R727, R728: 47R, OHDSP-Footprints-Pretty:SMD-0805
- removed R650, R651, R652, R653, R654, R655, R656, R657, R658, R659, R660, R661: 27R, OHDSP-Footprints-Pretty:SMD-0603
- removed R674, R702, R704, R705, R706, R713, R714, R716, R730, R732, R734: N/F, OHDSP-Footprints-Pretty:SMD-0805
- removed R710, R711, R712: 27R, OHDSP-Footprints-Pretty:SMD-0805
- removed R715, R719, R720, R723, R724, R725, R729, R731, R733: 10k, OHDSP-Footprints-Pretty:SMD-0805
- removed R717: 360R, OHDSP-Footprints-Pretty:SMD-0805
- removed R718: 120R, OHDSP-Footprints-Pretty:SMD-0805
- removed R721, R722: 2k2, OHDSP-Footprints-Pretty:SMD-0805
- removed U305, U704: IC-REG-XC6210B332MR, OHDSP-Footprints-Pretty:IC-SOT25
- removed U501: IC-SPDIF-RX-OPTO, OHDSP-Footprints-Pretty:IC_SPDIF_OPTO
- removed U502: IC-SPDIF-TX-OPTO, OHDSP-Footprints-Pretty:IC_SPDIF_OPTO
- removed U701: IC-REG-LM317-TO220, Power_Integrations:TO-220
- removed U702: IC-DAC-WM8501, OHDSP-Footprints-Pretty:IC_SOIC_14
- removed U703: IC-ADC-WM8783, OHDSP-Footprints-Pretty:IC_SOIC_8
- removed X201: 24M576, OHDSP-Footprints-Pretty:XTAL_HC49_TH
- added C202: 100p, OHDSP-Footprints-Pretty:CAP-TH-D6.3mmP2.5mm, B.Cu at (265.0, 74.8)
- added C206: 1u, OHDSP-Footprints-Pretty:SMD-0805, B.Cu at (265.0, 85.9)
- added C219: 22u, OHDSP-Footprints-Pretty:SMD-0603, B.Cu at (259.2, 105.0)
- added C228: 22u, OHDSP-Footprints-Pretty:SMD-0603, F.Cu at (269.7, 79.0)
- added C239: 5n6, OHDSP-Footprints-Pretty:SMD-0805, F.Cu at (267.2, 81.8)
- added C240: 150p, OHDSP-Footprints-Pretty:SMD-0805, F.Cu at (267.2, 80.4)
- added C309: 220u, OHDSP-Footprints-Pretty:SMD-0805, F.Cu at (215.1, 90.7)
- added C313: 22u, OHDSP-Footprints-Pretty:SMD-0805, F.Cu at (208.5, 89.4)
- added C316: 100n, OHDSP-Footprints-Pretty:SMD-0805, F.Cu at (255.0, 134.1)
- added C318: 10n, OHDSP-Footprints-Pretty:CAP-TH-D6.3mmP2.5mm, B.Cu at (227.3, 87.0)
- added C325: 100n, OHDSP-Footprints-Pretty:SMD-0805, F.Cu at (215.6, 73.9)
- added C329: 100u, OHDSP-Footprints-Pretty:SMD-0805, F.Cu at (229.6, 80.8)
- added C402: 100p, OHDSP-Footprints-Pretty:SMD-0603, F.Cu at (258.1, 107.2)
- added C403: 33p, OHDSP-Footprints-Pretty:SMD-0805, F.Cu at (255.0, 134.1)
- added C405: 100n, OHDSP-Footprints-Pretty:SMD-0603, F.Cu at (253.1, 116.5)
- added C502: 100n, OHDSP-Footprints-Pretty:CAP-TH-D6.3mmP2.5mm, B.Cu at (230.6, 110.4)
- added C504: 220u, OHDSP-Footprints-Pretty:SMD-0805, F.Cu at (230.5, 102.7)
- added C507: 47u, OHDSP-Footprints-Pretty:SMD-0805, F.Cu at (255.0, 134.1)
- added C515: 5n6, OHDSP-Footprints-Pretty:SMD-0805, F.Cu at (255.0, 134.1)
- added D304: LED, OHDSP-Footprints-Pretty:DIODE-SMB, F.Cu at (233.2, 85.0)
- added D501, D502, D503, D504: 1N5818, OHDSP-Footprints-Pretty:DIODE-DO-41, F.Cu at (255.0, 134.1)
- added P305: CONN_2x1, OHDSP-Footprints-Pretty:MNT_HOLE_2.5mm, F.Cu at (208.0, 63.0)
- added R217: 1k, OHDSP-Footprints-Pretty:SMD-0603, B.Cu at (259.0, 115.0)
- added R401, R404, R528: N/F, OHDSP-Footprints-Pretty:SMD-0805, F.Cu at (255.0, 134.1)
- added R405: 75R, OHDSP-Footprints-Pretty:SMD-0805, F.Cu at (256.0, 93.3)
- added R505: 0R, OHDSP-Footprints-Pretty:SMD-0603, B.Cu at (295.1, 60.6)
- added R509: 0R, OHDSP-Footprints-Pretty:SMD-0603, F.Cu at (277.9, 80.3)
- added R510: 0R, OHDSP-Footprints-Pretty:SMD-0603, F.Cu at (286.0, 73.9)
- added R511, R512, R527: 0R, OHDSP-Footprints-Pretty:SMD-0603, F.Cu at (255.0, 134.1)
- added R515: N/F, OHDSP-Footprints-Pretty:SMD-0805, F.Cu at (303.4, 103.8)
- added R516, R517, R519, R529, R530, R531, R535: N/F, OHDSP-Footprints-Pretty:SMD-0603, F.Cu at (255.0, 134.1)
- added R518: 47R, OHDSP-Footprints-Pretty:SMD-0603, B.Cu at (230.6, 106.6)
- added R520, R524, R525: 27R, OHDSP-Footprints-Pretty:SMD-0805, F.Cu at (255.0, 134.1)
- added R521: 27R, OHDSP-Footprints-Pretty:SMD-0805, F.Cu at (261.1, 105.4)
- added R522: 27R, OHDSP-Footprints-Pretty:SMD-0805, F.Cu at (263.1, 105.4)
- added R523: 27R, OHDSP-Footprints-Pretty:SMD-0805, F.Cu at (264.9, 105.4)
- added R526: 27R, OHDSP-Footprints-Pretty:SMD-0603, F.Cu at (255.0, 134.1)
- added R536, R537: 18k, OHDSP-Footprints-Pretty:SMD-0805, F.Cu at (255.0, 134.1)
- added R546, R547, R548, R549: 560R, OHDSP-Footprints-Pretty:SMD-0805, F.Cu at (255.0, 134.1)
- added X401: 24M576, OHDSP-Footprints-Pretty:XTAL_HC49_TH, F.Cu at (255.0, 134.1)
- C203: value 100p -> 220u; moved to F.Cu
- C204, C301: value 220u -> 22u; moved to B.Cu
- C207, C210: value 1u -> 100n; footprint OHDSP-Footprints-Pretty:SMD-0603 -> OHDSP-Footprints-Pretty:SMD-0805; moved to F.Cu
- C208, C211: value 100n -> 10n; footprint OHDSP-Footprints-Pretty:SMD-0603 -> OHDSP-Footprints-Pretty:SMD-0805
- C209: value 10n -> 1u; footprint OHDSP-Footprints-Pretty:SMD-0603 -> OHDSP-Footprints-Pretty:SMD-0805; moved to B.Cu
- C235, C236: footprint OHDSP-Footprints-Pretty:SMD-0603 -> OHDSP-Footprints-Pretty:SMD-0805
- C237: value 33p -> 1u; footprint OHDSP-Footprints-Pretty:SMD-0603 -> OHDSP-Footprints-Pretty:SMD-0805
- C238: renamed from C219; value 1u -> 100n
- C304: value 22u -> 220u; moved to F.Cu
- C308: value 220u -> 22u
- C314: value 220u -> 100n; moved to B.Cu
- C317: value 220u -> 10n; moved to B.Cu
- C319: renamed from C303; value 22u -> 10n
- C321: renamed from C309; value 10n -> 100n
- C322: renamed from C313; value 22u -> 100n
- C328: renamed from C316; value 100n -> 22u
- C330: value 1u -> 100u; moved to F.Cu
- C331: value 10n -> 100u; moved to F.Cu
- C401: value 100p -> 33p
- C506: renamed from C501; value 100p -> 47u
- C508: renamed from C503; value 22u -> 220u
- C509: renamed from C504; value 100n -> 220u
- C510: renamed from C505; value 100n -> 220u
- C511: renamed from C506; value 100n -> 220u
- C512: renamed from C507; value 10n -> 5n6
- C513: renamed from C508; value 22u -> 5n6
- C514: renamed from C509; value 22u -> 5n6
- P301, P302: value CONN_2x1 -> PIN
- P304: value PIN -> CONN_2x1
- R211: renamed from R220; value 3k3 -> 8k2
- R214: renamed from R224; value 3k6 -> 4k7
- R215: renamed from R227; value 100R -> 7k5
- R216: renamed from R229; value N/F -> 0R
- R307: renamed from R313; value 100k -> 10k
- R309: renamed from R301; value 100k -> 10k
- R402: value 75R -> 100R
- R407: renamed from R406; value 27R -> 75R
- R408: renamed from R407; value 27R -> 75R
- R409: renamed from R408; value 27R -> 75R
- R504: renamed from R501; value 47R -> N/F
- U201: value ADAU1452WBCPZ -> IC-EEPROM-I2C
- U203: value 25AA1024 -> IC-DSP-ADAU1701JSTZ
- U302: renamed from U301; value IC-REG-XRP7659ISTR-F -> NCP700BSN33T1G
- U304: value IC-REG-XC6210B332MR -> NCP700BSN18T1G
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- renumbered C206 to C205, C214 to C212, C216 to C213, C252 to C214, C218 to C215, C254 to C216, C224 to C217, C225 to C218, C227 to C220, C228 to C221, C229 to C222, C231 to C223, C246 to C224, C239 to C225, C240 to C226, C244 to C227, C242 to C229, C202 to C230, C245 to C231, C243 to C232, C250 to C233, C251 to C234, C306 to C302, C307 to C303, C310 to C305, C311 to C306, C312 to C307, C319 to C310, C325 to C311, C326 to C312, C329 to C315, C305 to C320, C334 to C323, C335 to C324, C337 to C326, C338 to C327, C403 to C404, C609 to C501, C603 to C503, C607 to C505, CN406 to CN402, D304 to D303, L303 to L302, L601 to L501, P305 to P303, P607 to P502, P608 to P503, P610 to P504, P609 to P508, P605 to P509, P612 to P510, P611 to P511, R235 to R206, R206 to R207, R225 to R208, R218 to R209, R219 to R210, R222 to R212, R223 to R213, R228 to R218, R226 to R219, R221 to R220, R234 to R221, R207 to R222, R208 to R223, R209 to R224, R210 to R225, R211 to R226, R212 to R227, R213 to R228, R214 to R229, R215 to R230, R216 to R231, R217 to R232, R302 to R301, R303 to R302, R306 to R303, R307 to R304, R308 to R305, R310 to R306, R314 to R308, R401 to R403, R404 to R406, R409 to R410, R414 to R411, R418 to R412, R415 to R413, R419 to R414, R601 to R501, R602 to R502, R603 to R503, R604 to R506, R605 to R507, R606 to R508, R616 to R513, R620 to R514, R662 to R532, R666 to R533, R670 to R534, R629 to R538, R630 to R539, R628 to R540, R634 to R541, R641 to R542, R643 to R543, R646 to R544, R647 to R545, SW202 to SW201, U302 to U301
Connections:
- net /ADAU1452/MRST renamed /ADAU1701/MRST
- C203 pad 1: Net-(C203-Pad1) -> /ADAU1701/DVDD
- C204 pad 1: /ADAU1452/DVDD -> /ADAU1701/DVDD
- C205 pad 1: /ADAU1452/DVDD -> /ADAU1701/DVDD
- C207 pad 1: /ADAU1452/DVDD -> /ADAU1701/DVDD
- C208 pad 1: /ADAU1452/DVDD -> /ADAU1701/DVDD
- C209 pad 1: /ADAU1452/DVDD -> /ADAU1701/DVDD
- C210 pad 1: /ADAU1452/DVDD -> /ADAU1701/DVDD
- C211 pad 1: /ADAU1452/DVDD -> /ADAU1701/DVDD
- C214 pad 1: Net-(C252-Pad1) -> Net-(C214-Pad1)
- C216 pad 1: Net-(C252-Pad1) -> Net-(C214-Pad1)
- C218 pad 1: /ADAU1452/IOVDD -> /ADAU1701/IOVDD
- C218 pad 2: GNDD -> Net-(C218-Pad2)
- C220 pad 1: /ADAU1452/IOVDD -> /ADAU1701/IOVDD
- C220 pad 2: GNDD -> Net-(C218-Pad2)
- C221 pad 1: /ADAU1452/IOVDD -> /ADAU1701/IOVDD
- C221 pad 2: GNDD -> Net-(C218-Pad2)
- C222 pad 1: /ADAU1452/IOVDD -> /ADAU1701/IOVDD
- C222 pad 2: GNDD -> Net-(C218-Pad2)
- C224 pad 1: /ADAU1452/RESET -> /ADAU1701/RESET
- C226 pad 1: /ADAU1452/PVDD -> /ADAU1701/PVDD
- C229 pad 1: /ADAU1452/PVDD -> /ADAU1701/PVDD
- C232 pad 1: /ADAU1452/AVDD -> /ADAU1701/AVDD
- C233 pad 1: /ADAU1452/AVDD -> /ADAU1701/AVDD
- C234 pad 1: /ADAU1452/AVDD -> /ADAU1701/AVDD
- C235 pad 1: /ADAU1452/IOVDD -> /ADAU1701/AVDD
- C236 pad 1: /ADAU1452/IOVDD -> /ADAU1701/AVDD
- C237 pad 1: /ADAU1452/XTALIN -> /ADAU1701/AVDD
- C238 pad 1: /ADAU1452/DVDD -> /ADAU1701/AVDD
- C301 pad 1: VCC -> GNDD
- C301 pad 2: GNDD -> VCC
- C304 pad 1: GNDD -> VCC
- C304 pad 2: VCC -> GNDD
- C308 pad 1: VCC -> VCOM
- C314 pad 1: VDD -> VCOM
- C317 pad 1: VCOM -> Net-(C317-Pad1)
- C319 pad 1: GNDD -> Net-(C319-Pad1)
- C319 pad 2: VCC -> GNDD
- C320 pad 1: GNDD -> Net-(C320-Pad1)
- C320 pad 2: VCC -> GNDD
- C321 pad 1: Net-(C309-Pad1) -> Net-(C321-Pad1)
- C321 pad 2: Net-(C309-Pad2) -> GNDD
- C322 pad 1: VDD -> Net-(C322-Pad1)
- C323 pad 2: GNDD -> Net-(C323-Pad2)
- C326 pad 2: GNDD -> Net-(C326-Pad2)
- C330 pad 1: Net-(C330-Pad1) -> VPP
- C331 pad 1: Net-(C331-Pad1) -> VDD
- C404 pad 1: Net-(C403-Pad1) -> Net-(C404-Pad1)
- C506 pad 1: Net-(C501-Pad1) (its old number) -> /Connectors/ANAIN1
- C506 pad 2: GNDD -> Net-(C506-Pad2)
- C508 pad 1: Net-(C503-Pad1) -> /Connectors/ANAOUT1
- C508 pad 2: GNDD -> Net-(C508-Pad2)
- C509 pad 1: Net-(C503-Pad1) -> /Connectors/ANAOUT2
- C509 pad 2: GNDD -> Net-(C509-Pad2)
- C510 pad 1: Net-(C503-Pad1) -> /Connectors/ANAOUT3
- C510 pad 2: GNDD -> Net-(C510-Pad2)
- C511 pad 1: Net-(C503-Pad1) -> /Connectors/ANAOUT4
- C511 pad 2: GNDD -> Net-(C511-Pad2)
- C512 pad 2: Net-(C507-Pad2) -> GNDD
- C513 pad 1: Net-(C503-Pad1) -> Net-(C513-Pad1)
- C514 pad 1: Net-(C503-Pad1) -> Net-(C514-Pad1)
- CN401 pad 1: /ClockFanout/MCLKC1 -> Net-(CN401-Pad1)
- L201 pad 2: /ADAU1452/DVDD -> Net-(L201-Pad2)
- L203 pad 2: /ADAU1452/IOVDD -> /ADAU1701/IOVDD
- L204 pad 2: /ADAU1452/PVDD -> /ADAU1701/PVDD
- L205 pad 2: /ADAU1452/AVDD -> /ADAU1701/AVDD
- L401 pad 2: Net-(C403-Pad1) -> Net-(C404-Pad1)
- P201 pad 1: /ADAU1452/SELFBOOT -> /ADAU1701/SELFBOOT
- P301 pad 1: +5V -> GNDD
- P301 pad 2: GNDD -> (no net)
- P302 pad 1: Net-(D302-Pad1) -> GNDD
- P302 pad 2: GNDD -> (no net)
- P304 pad 1: GNDD -> +5V
- P502 pad 5: /ADAU1452/I2C_SCL -> /Connectors/I2C_SCL
- P502 pad 7: Net-(P607-Pad7) -> /ADAU1701/I2C_SCL
- P503 pad 5: /ADAU1452/I2C_SCL -> /Connectors/I2C_SCL
- P503 pad 7: Net-(P607-Pad7) -> /ADAU1701/I2C_SCL
- P504 pad 1: /ADAU1452/I2C_SCL -> /Connectors/I2C_SCL
- P504 pad 3: /ADAU1452/I2C_SDA -> /ADAU1701/I2C_SCL
- P504 pad 5: /ADAU1452/SPI_MISO -> /Connectors/SL_MISO
- P504 pad 7: /ADAU1452/SPI_SCLK -> /Connectors/SL_SCLK
- P504 pad 8: /ADAU1452/SPI_MOSI -> /Connectors/SL_MOSI
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Routing:
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
Commit message: WIP
Parts:
- removed the C219 at (259.2, 105.0)
- removed the C220 at (256.5, 101.9)
- removed the C221 at (275.8, 85.0)
- removed the C222 at (278.5, 84.5)
- removed the C228 at (269.7, 79.0)
- removed the C234 at (274.6, 82.5)
- removed the C239 at (267.2, 81.8)
- removed the C240 at (267.2, 80.4)
- removed the C402 at (258.1, 107.2)
- removed the C405 at (253.1, 116.5)
- removed the R205 at (246.9, 90.9)
- removed the R217 at (259.0, 115.0)
- removed the R224 at (248.5, 102.0)
- removed the R225 at (248.5, 104.0)
- removed the R516 at (255.0, 134.1)
- removed the R526 at (255.0, 134.1)
- removed the R529 at (255.0, 134.1)
- added C201: 220u, OHDSP-Footprints-Pretty:CAP-TH-D6.3mmP2.5mm, F.Cu at (225.3, 169.1)
- added C205: 10u, OHDSP-Footprints-Pretty:SMD-0805, F.Cu at (279.2, 144.9)
- added C206: 10u, OHDSP-Footprints-Pretty:SMD-0805, F.Cu at (274.2, 150.7)
- added C207: 10u, OHDSP-Footprints-Pretty:SMD-0805, F.Cu at (285.6, 162.2)
- added C208: 220u, OHDSP-Footprints-Pretty:CAP-TH-D6.3mmP2.5mm, F.Cu at (212.7, 181.1)
- added C210: 100n, OHDSP-Footprints-Pretty:SMD-0805, F.Cu at (270.2, 180.8)
- added C211: 100n, OHDSP-Footprints-Pretty:SMD-0805, F.Cu at (252.5, 167.1)
- added C212: 100n, OHDSP-Footprints-Pretty:SMD-0805, F.Cu at (280.6, 167.9)
- added C214: 22u, OHDSP-Footprints-Pretty:SMD-0805, B.Cu at (262.0, 144.0)
- added C223: 56n, OHDSP-Footprints-Pretty:SMD-0805, F.Cu at (232.2, 187.1)
- added C224: 3n3, OHDSP-Footprints-Pretty:SMD-0805, F.Cu at (265.2, 186.5)
- added C231: 1u, OHDSP-Footprints-Pretty:SMD-0805, B.Cu at (255.3, 152.2)
- added C233: 100n, OHDSP-Footprints-Pretty:SMD-0805, F.Cu at (233.0, 165.8)
- added C236: 22u, OHDSP-Footprints-Pretty:SMD-0805, F.Cu at (241.0, 165.2)
- added C237: 100n, OHDSP-Footprints-Pretty:SMD-0805, F.Cu at (211.2, 187.5)
- added C242: 100n, OHDSP-Footprints-Pretty:SMD-0805, F.Cu at (216.1, 163.4)
- added C246: 100n, OHDSP-Footprints-Pretty:SMD-0805, B.Cu at (274.2, 144.9)
- added C403: 100p, OHDSP-Footprints-Pretty:SMD-0805, F.Cu at (320.9, 208.7)
- added C404: 220u, OHDSP-Footprints-Pretty:SMD-0805, F.Cu at (343.3, 220.0)
- added C406: 100n, OHDSP-Footprints-Pretty:SMD-0805, F.Cu at (309.5, 218.1)
- added C407: 100n, OHDSP-Footprints-Pretty:SMD-0805, F.Cu at (344.8, 208.5)
- added C408: 22u, OHDSP-Footprints-Pretty:SMD-0805, F.Cu at (330.6, 225.7)
- added C409: 100n, OHDSP-Footprints-Pretty:SMD-0805, F.Cu at (343.3, 214.3)
- added C410: 22u, OHDSP-Footprints-Pretty:SMD-0805, F.Cu at (338.3, 220.0)
- added C411: 100p, OHDSP-Footprints-Pretty:SMD-0805, F.Cu at (335.6, 225.7)
- added L402: 600R@100MHz, OHDSP-Footprints-Pretty:SMD-0805, F.Cu at (299.5, 202.8)
- added P501: CONN_02X10, OHDSP-Footprints-Pretty:CONN_DIL_2X10, F.Cu at (277.0, 119.4)
- added P505: CONN_02X10, OHDSP-Footprints-Pretty:CONN_DIL_2X10, F.Cu at (299.7, 121.9)
- added P506: CONN_2x1, OHDSP-Footprints-Pretty:CONN_SIL_2, F.Cu at (221.5, 234.7)
- added P507: CONN_2x1, OHDSP-Footprints-Pretty:CONN_SIL_2, F.Cu at (208.9, 240.3)
- added P512: CONN_2x1, OHDSP-Footprints-Pretty:CONN_SIL_2, F.Cu at (208.9, 234.7)
- added P513: CONN_2x1, OHDSP-Footprints-Pretty:CONN_SIL_2, F.Cu at (208.9, 246.0)
- added P514: CONN_2x1, OHDSP-Footprints-Pretty:CONN_SIL_2, F.Cu at (221.5, 240.3)
- added P515: CONN_2x1, OHDSP-Footprints-Pretty:CONN_SIL_2, F.Cu at (240.2, 219.4)
- added R209: 475R, OHDSP-Footprints-Pretty:SMD-0805, F.Cu at (265.2, 180.8)
- added R210: 0R, OHDSP-Footprints-Pretty:SMD-0805, F.Cu at (280.6, 162.2)
- added R214: 1k, OHDSP-Footprints-Pretty:SMD-0805, B.Cu at (285.6, 156.4)
- added R216: 1k, OHDSP-Footprints-Pretty:SMD-0805, F.Cu at (270.2, 175.0)
- added R218: 0R, OHDSP-Footprints-Pretty:SMD-0805, F.Cu at (284.2, 144.9)
- added R219: 100k, OHDSP-Footprints-Pretty:SMD-0805, F.Cu at (280.6, 156.4)
- added R221: 100k, OHDSP-Footprints-Pretty:SMD-0805, F.Cu at (242.2, 188.8)
- added R234: N/F, OHDSP-Footprints-Pretty:SMD-0805, F.Cu at (237.2, 187.1)
- added R235: 1k, OHDSP-Footprints-Pretty:SMD-0805, F.Cu at (234.2, 181.3)
- added R238: 1k, OHDSP-Footprints-Pretty:SMD-0805, F.Cu at (257.2, 192.2)
- added R239: N/F, OHDSP-Footprints-Pretty:SMD-0805, F.Cu at (265.6, 157.8)
- added R404: 100R, OHDSP-Footprints-Pretty:SMD-0805, F.Cu at (328.3, 219.4)
- added R406: 0R, OHDSP-Footprints-Pretty:SMD-0805, F.Cu at (339.8, 208.5)
- added R407: 0R, OHDSP-Footprints-Pretty:SMD-0805, F.Cu at (333.3, 220.0)
- added R410: 100R, OHDSP-Footprints-Pretty:SMD-0805, F.Cu at (325.6, 225.1)
- added R411: 47R, OHDSP-Footprints-Pretty:SMD-0805, F.Cu at (338.3, 214.3)
- added R515: N/F, OHDSP-Footprints-Pretty:SMD-0805, F.Cu at (253.0, 223.2)
- added R520: N/F, OHDSP-Footprints-Pretty:SMD-0805, F.Cu at (272.7, 235.0)
- added R528: 0R, OHDSP-Footprints-Pretty:SMD-0805, F.Cu at (293.4, 118.1)
- added R536: N/F, OHDSP-Footprints-Pretty:SMD-0805, F.Cu at (265.4, 245.6)
- added TP201: TP, OHDSP-Footprints-Pretty:TP-2mm, F.Cu at (247.6, 167.1)
- added TP202: TP, OHDSP-Footprints-Pretty:TP-2mm, F.Cu at (261.4, 153.4)
- added TR201: BC847, OHDSP-Footprints-Pretty:IC-SOT23, F.Cu at (227.0, 185.8)
- added TR202: BC857, OHDSP-Footprints-Pretty:IC-SOT23, F.Cu at (269.0, 146.1)
- added TR203: BC857, OHDSP-Footprints-Pretty:IC-SOT23, F.Cu at (235.0, 176.1)
- added U303: NCP700BSN33T1G, OHDSP-Footprints-Pretty:IC-SOT23-5, F.Cu at (303.4, 166.3)
- added U401: NC7SZU04M5X, OHDSP-Footprints-Pretty:IC-SOT23-5, F.Cu at (311.9, 204.0)
- added U402: NC7SZU04M5X, OHDSP-Footprints-Pretty:IC-SOT23-5, F.Cu at (299.7, 213.8)
- C202: value 100p -> 220u; moved to F.Cu
- C203, C304, C309, C504: footprint OHDSP-Footprints-Pretty:SMD-0805 -> OHDSP-Footprints-Pretty:CAP-TH-D6.3mmP2.5mm
- C204: value 22u -> 100p; footprint OHDSP-Footprints-Pretty:CAP-TH-D6.3mmP2.5mm -> OHDSP-Footprints-Pretty:SMD-0805
- C229: value 100n -> 22u; footprint OHDSP-Footprints-Pretty:SMD-0603 -> OHDSP-Footprints-Pretty:SMD-0805; moved to B.Cu
- C230: value 220u -> 100n; footprint OHDSP-Footprints-Pretty:CAP-TH-D6.3mmP2.5mm -> OHDSP-Footprints-Pretty:SMD-0805; moved to B.Cu
- C238: value 100n -> 220u; footprint OHDSP-Footprints-Pretty:SMD-0603 -> OHDSP-Footprints-Pretty:CAP-TH-D6.3mmP2.5mm; moved to F.Cu
- C301, C308, C314, C317, C318, C502: footprint OHDSP-Footprints-Pretty:CAP-TH-D6.3mmP2.5mm -> OHDSP-Footprints-Pretty:SMD-0805
- C329, C330, C331: value 100u -> 220u; footprint OHDSP-Footprints-Pretty:SMD-0805 -> OHDSP-Footprints-Pretty:CAP-TH-D6.3mmP2.5mm
- C506, C507, C508, C509, C510, C511: footprint OHDSP-Footprints-Pretty:SMD-0805 -> OHDSP-Footprints-Pretty:CAP-TH-D8mmP3.5mm
- D304: footprint OHDSP-Footprints-Pretty:DIODE-SMB -> OHDSP-Footprints-Pretty:SMD-0805
- P301, P302: footprint OHDSP-Footprints-Pretty:CONN-SCREW-2WAY-5mm-5.08mm -> OHDSP-Footprints-Pretty:MNT_HOLE_2.5mm
- P304, P305: footprint OHDSP-Footprints-Pretty:MNT_HOLE_2.5mm -> OHDSP-Footprints-Pretty:CONN_SIL_2
- R222, R223: value 0R -> 10k; moved to F.Cu
- R226, R227: value N/F -> 0R; moved to F.Cu
- R228, R231: moved to F.Cu
- R229: value 0R -> N/F; moved to F.Cu
- R230: value N/F -> 1k; moved to F.Cu
- R232: value 4k3 -> 1k; footprint OHDSP-Footprints-Pretty:SMD-0603 -> OHDSP-Footprints-Pretty:SMD-0805
- R402: value 100R -> 1Meg; footprint OHDSP-Footprints-Pretty:TH-RES-0W25 -> OHDSP-Footprints-Pretty:SMD-0805
- R408: renamed from R405; value 75R -> 0R
- R505, R532: footprint OHDSP-Footprints-Pretty:SMD-0603 -> OHDSP-Footprints-Pretty:SMD-0805; moved to F.Cu
- R506, R507, R508, R509, R510, R511, R512, R514, R517, R530, R531, R533, R534: footprint OHDSP-Footprints-Pretty:SMD-0603 -> OHDSP-Footprints-Pretty:SMD-0805
- R513: value N/F -> 1k; footprint OHDSP-Footprints-Pretty:SMD-0603 -> OHDSP-Footprints-Pretty:SMD-0805
- R518: value 47R -> N/F; footprint OHDSP-Footprints-Pretty:SMD-0603 -> OHDSP-Footprints-Pretty:SMD-0805; moved to F.Cu
- R519: value N/F -> 47R; footprint OHDSP-Footprints-Pretty:SMD-0603 -> OHDSP-Footprints-Pretty:SMD-0805; moved to B.Cu
- R527: value 0R -> 27R; footprint OHDSP-Footprints-Pretty:SMD-0603 -> OHDSP-Footprints-Pretty:SMD-0805
- R535: footprint OHDSP-Footprints-Pretty:SMD-0603 -> OHDSP-Footprints-Pretty:SMD-0805; moved to B.Cu
- U201: value IC-EEPROM-I2C -> ADM13307-5ARZ; footprint OHDSP-Footprints-Pretty:IC-LFCSP72-HANDFIT -> OHDSP-Footprints-Pretty:IC_DIP_8; moved to B.Cu
- U202: value ADM13307-5ARZ -> ADAU1701JSTZ; footprint OHDSP-Footprints-Pretty:IC_SOIC_8 -> OHDSP-Footprints-Pretty:IC-LQFP48_7x7; moved to F.Cu
- U203: value IC-DSP-ADAU1701JSTZ -> IC-EEPROM-I2C
- U302: footprint OHDSP-Footprints-Pretty:IC-SOT23-6 -> OHDSP-Footprints-Pretty:IC-SOT23-5
- U304: footprint OHDSP-Footprints-Pretty:IC-SOT25 -> OHDSP-Footprints-Pretty:IC-SOT23-5
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- renumbered C212 to C209, C205 to C216, C206 to C217, C207 to C218, C208 to C219, C209 to C220, C210 to C221, C211 to C222, C217 to C225, C223 to C226, C218 to C227, C224 to C228, C227 to C232, C225 to C234, C226 to C235, C231 to C239, C232 to C240, C233 to C241, C235 to C243, C236 to C244, C237 to C245, C214 to C247, C216 to C248, C201 to C249, C403 to C402, C404 to C405, R204 to R201, R207 to R202, R209 to R203, R210 to R204, R211 to R205, R212 to R206, R213 to R207, R214 to R208, R215 to R211, R208 to R212, R216 to R213, R219 to R215, R220 to R217, R218 to R220, R201 to R224, R221 to R225, R206 to R233, R203 to R236, R202 to R237, R404 to R401, R401 to R403, R403 to R405, R406 to R409, R407 to R412, R408 to R413, R409 to R414, R410 to R415, R411 to R416, R412 to R417, R413 to R418, R414 to R419, R515 to R516, R520 to R521, R521 to R522, R522 to R523, R523 to R524, R524 to R525, R525 to R526, R528 to R529, R536 to R537, R537 to R538, R538 to R539, R539 to R540, R540 to R541, R541 to R542, R542 to R543, R543 to R544, R544 to R545, R545 to R546, R546 to R547, R547 to R548, R548 to R549, R549 to R550, U401 to U403
Connections:
- C202 pad 1: Net-(C202-Pad1) -> /ADAU1701/FILTD
- C203 pad 1: /ADAU1701/DVDD -> /ADAU1701/CM
- C204 pad 1: /ADAU1701/DVDD -> Net-(C204-Pad1)
- C226 pad 1: Net-(C223-Pad1) -> Net-(C226-Pad1)
- C227 pad 2: Net-(C218-Pad2) -> Net-(C227-Pad2)
- C228 pad 1: /ADAU1701/RESET -> /Connectors/ADC_RESET
- C229 pad 1: /ADAU1701/PVDD -> /ADAU1701/IOVDD
- C229 pad 2: GNDD -> Net-(C227-Pad2)
- C230 pad 1: VAA -> /ADAU1701/IOVDD
- C230 pad 2: GNDD -> Net-(C227-Pad2)
- C232 pad 1: /ADAU1701/MRST -> Net-(C232-Pad1)
- C238 pad 1: /ADAU1701/AVDD -> VAA
- C247 pad 1: Net-(C214-Pad1) -> /ADAU1701/IOVDD
- C248 pad 1: Net-(C214-Pad1) -> (no net)
- C323 pad 2: Net-(C323-Pad2) -> (no net)
- C326 pad 2: Net-(C326-Pad2) -> (no net)
- C329 pad 2: Net-(C329-Pad2) -> (no net)
- C402 pad 1: Net-(C403-Pad1) (its old number) -> Net-(C402-Pad1)
- C506 pad 1: /Connectors/ANAIN1 -> /ADAU1701/ADC_IN0
- C507 pad 1: /Connectors/ANAIN2 -> /ADAU1701/ADC_IN1
- C508 pad 1: /Connectors/ANAOUT1 -> /Connectors/ANA_OUT1
- C509 pad 1: /Connectors/ANAOUT2 -> /Connectors/ANA_OUT2
- C510 pad 1: /Connectors/ANAOUT3 -> /Connectors/ANA_OUT3
- C511 pad 1: /Connectors/ANAOUT4 -> /Connectors/ANA_OUT4
- D501 pad 2: /Connectors/ANAIN1 -> /ADAU1701/ADC_IN0
- D502 pad 2: /Connectors/ANAIN2 -> /ADAU1701/ADC_IN1
- D503 pad 1: /Connectors/ANAIN1 -> /ADAU1701/ADC_IN0
- D504 pad 1: /Connectors/ANAIN2 -> /ADAU1701/ADC_IN1
- L201 pad 2: Net-(L201-Pad2) -> (no net)
- P502 pad 5: /Connectors/I2C_SCL -> /ADAU1701/I2C_SCL
- P502 pad 7: /ADAU1701/I2C_SCL -> /ADAU1701/I2C_SDA
- P503 pad 5: /Connectors/I2C_SCL -> /ADAU1701/I2C_SCL
- P503 pad 7: /ADAU1701/I2C_SCL -> /ADAU1701/I2C_SDA
- P504 pad 1: /Connectors/I2C_SCL -> /ADAU1701/I2C_SCL
- P504 pad 2: Net-(P504-Pad2) -> (no net)
- P504 pad 3: /ADAU1701/I2C_SCL -> /ADAU1701/I2C_SDA
- P504 pad 4: Net-(P504-Pad4) -> (no net)
- P504 pad 5: /Connectors/SL_MISO -> (no net)
- P504 pad 7: /Connectors/SL_SCLK -> (no net)
- P504 pad 8: /Connectors/SL_MOSI -> (no net)
- P504 pad 9: /Connectors/SL_~SS -> (no net)
- P508 pad 1: Net-(P508-Pad1) -> (no net)
- P508 pad 17: Net-(P508-Pad17) -> (no net)
- R201 pad 2: Net-(C202-Pad1) -> Net-(C204-Pad1)
- R203 pad 2: Net-(R209-Pad2) -> Net-(R203-Pad2)
- R204 pad 2: Net-(R210-Pad2) -> Net-(R204-Pad2)
- R205 pad 2: Net-(R211-Pad2) -> Net-(R205-Pad2)
- R206 pad 2: Net-(R209-Pad2) -> Net-(R203-Pad2)
- R207 pad 2: Net-(R210-Pad2) -> Net-(R204-Pad2)
- R208 pad 2: Net-(R211-Pad2) -> Net-(R205-Pad2)
- R211 pad 1: Net-(R215-Pad1) -> Net-(R211-Pad1)
- R213 pad 1: Net-(R216-Pad1) -> Net-(R213-Pad1)
- R213 pad 2: /ADAU1701/RESET -> /Connectors/ADC_RESET
- R215 pad 2: /ADAU1701/RESET -> /Connectors/ADC_RESET
- R217 pad 2: Net-(R220-Pad2) -> Net-(R217-Pad2)
- R222 pad 1: /ADAU1701/SL_MISO -> Net-(R221-Pad2)
- R222 pad 2: Net-(R222-Pad2) -> /Connectors/ADI_RST
- R223 pad 1: /Connectors/I2C_SCL -> Net-(R219-Pad2)
- R223 pad 2: Net-(R222-Pad2) -> /Connectors/PI_RST
- R228 pad 1: /ADAU1701/SL_MOSI -> /ADAU1701/IOVDD
- R228 pad 2: Net-(R227-Pad2) -> Net-(R228-Pad2)
- R229 pad 1: /ADAU1701/SL_~SS -> /ADAU1701/ADDR0
- R229 pad 2: Net-(R226-Pad2) -> /ADAU1701/IOVDD
- R230 pad 1: GNDD -> /ADAU1701/ADDR0
- R230 pad 2: Net-(R227-Pad2) -> GNDD
- R231 pad 1: GNDD -> /ADAU1701/ADDR1
- R231 pad 2: Net-(R226-Pad2) -> /ADAU1701/IOVDD
- R232 pad 1: Net-(C239-Pad2) -> /ADAU1701/ADDR1
- R232 pad 2: Net-(C240-Pad2) -> GNDD
- R233 pad 1: Net-(R206-Pad1) -> /ADAU1701/IOVDD
- R233 pad 2: Net-(R206-Pad2) -> Net-(R233-Pad2)
- R236 pad 2: /Connectors/I2C_SCL -> /ADAU1701/I2C_SDA
- R401 pad 1: Net-(R404-Pad1) -> Net-(R401-Pad1)
- R402 pad 1: Net-(R402-Pad1) -> Net-(C401-Pad1)
- R402 pad 2: Net-(C403-Pad1) (its old number) -> Net-(R402-Pad2)
- R408 pad 1: Net-(R405-Pad1) -> Net-(R408-Pad1)
- R408 pad 2: Net-(R405-Pad2) -> (no net)
- R409 pad 2: Net-(R406-Pad2) -> (no net)
- R412 pad 1: GNDD -> /ADAU1701/MCLK
- R413 pad 1: GNDD -> /Connectors/ADC_MCLK
- R414 pad 1: GNDD -> /Connectors/DAC_MCLK
- R416 pad 2: GNDD -> /ADAU1701/MCLK
- R417 pad 2: GNDD -> /Connectors/ADC_MCLK
- R418 pad 2: GNDD -> /Connectors/DAC_MCLK
- R513 pad 1: GNDD -> /Connectors/ADI_RST
- R513 pad 2: /ADAU1701/ADCIN_SDATA0 -> Net-(P504-Pad6)
- R514 pad 2: /ADAU1701/ADCIN_BCLK0 -> /ADAU1701/ADCIN_SDATA0
- R517 pad 2: /ADAU1701/ADCIN_SDATA2 -> /ADAU1701/ADCIN_SDATA3
- R518 pad 1: Net-(C505-Pad1) -> GNDD
- R518 pad 2: Net-(C501-Pad1) -> /ADAU1701/ADCIN_SDATA2
- R519 pad 1: GNDD -> Net-(C505-Pad1)
- R519 pad 2: /ADAU1701/ADCIN_SDATA1 -> Net-(C501-Pad1)
- R527 pad 1: /Connectors/DAC_RESET -> /ADAU1701/DACOUT_SDATA3
- R527 pad 2: Net-(P505-Pad17) -> Net-(P505-Pad13)
- R530 pad 2: Net-(P505-Pad11) -> Net-(P505-Pad13)
- R531 pad 2: Net-(P505-Pad9) -> Net-(P505-Pad11)
- R532 pad 2: Net-(P505-Pad7) -> Net-(P505-Pad9)
- R533 pad 2: Net-(P505-Pad5) -> Net-(P505-Pad7)
- R534 pad 2: Net-(P505-Pad3) -> Net-(P505-Pad5)
- R535 pad 2: Net-(P505-Pad1) -> Net-(P505-Pad3)
- R539 pad 1: /ADAU1701/I2C_SCL -> /ADAU1701/I2C_SDA
- R540 pad 1: /Connectors/I2C_SCL -> /ADAU1701/I2C_SCL
- R541 pad 1: /ADAU1701/MRST -> /Connectors/PI_RST
- R545 pad 2: /Connectors/RPI_SDATA_IN -> (no net)
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Routing:
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- removed copper zone on In2.Cu, net GNDD

Commit message: WIP
Parts:
- removed P304: CONN_2x1, OHDSP-Footprints-Pretty:CONN_SIL_2
- added C250, R240: N/F, OHDSP-Footprints-Pretty:SMD-0805, F.Cu at (255.0, 134.1)
- added D305, D306: LED, OHDSP-Footprints-Pretty:SMD-0805, F.Cu at (255.0, 134.1)
- added R241: 0R, OHDSP-Footprints-Pretty:SMD-0805, F.Cu at (255.0, 134.1)
- added R310: 4k7, OHDSP-Footprints-Pretty:SMD-0805, F.Cu at (255.0, 134.1)
- added TR204: N/F, OHDSP-Footprints-Pretty:IC-SOT23, F.Cu at (255.0, 134.1)
- C305: value 10n -> 270n
- C308: value 22u -> 35ZL470MEFC10X20; footprint OHDSP-Footprints-Pretty:SMD-0805 -> OHDSP-Footprints-Pretty:CAP-TH-D10mmP5mm
- C309: value 220u -> 1n5; footprint OHDSP-Footprints-Pretty:CAP-TH-D6.3mmP2.5mm -> OHDSP-Footprints-Pretty:SMD-0805
- C310: value 100n -> 10ZL470MEFC8X11.5; footprint OHDSP-Footprints-Pretty:SMD-0805 -> OHDSP-Footprints-Pretty:CAP-TH-D8mmP3.5mm
- C311, C312, C313: value 22u -> 220u; footprint OHDSP-Footprints-Pretty:SMD-0805 -> OHDSP-Footprints-Pretty:CAP-TH-D6.3mmP2.5mm
- D301: value SS24T3G -> 1N914; footprint OHDSP-Footprints-Pretty:DIODE-SMB -> OHDSP-Footprints-Pretty:DIODE-DO-35
- D302, D303: value SS24T3G -> MBRS330T3; footprint OHDSP-Footprints-Pretty:DIODE-SMB -> OHDSP-Footprints-Pretty:DIODE-SMC
- L302: value 744772220 -> CDRH125NP-100MC; footprint OHDSP-Footprints-Pretty:PASSIVE-TH-IND-WURTH-5mm -> OHDSP-Footprints-Pretty:IND_SMD_CDRH125
- R230: value 1k -> 10k
- R231: value N/F -> 10k
- R232: value 1k -> N/F
- R301: value 100k -> 1R
- R303: value 39k -> 1R
- R304: value 10k -> 1R
- R305: value 0R -> 4k7
- R543: value 0R -> N/F
- U301: value IC-REG-XRP7659ISTR-F -> LT1374CS8-5#PBF; footprint OHDSP-Footprints-Pretty:IC-SOT23-6 -> OHDSP-Footprints-Pretty:IC_SOIC_8
- moved CN401 201.4 mm to (337.1, 27.9), turned to 270 degrees
- moved X401 199.6 mm to (320.5, 22.1)
- moved R402 197.5 mm to (320.3, 29.6)
- moved C402 196.2 mm to (324.1, 25.3)
- moved R404 193.0 mm to (321.3, 26.6), turned to 270 degrees
- moved R405 191.4 mm to (350.3, 24.1), turned to 270 degrees
- moved C411 189.4 mm to (310.1, 38.1), turned to 270 degrees
- moved C408 189.1 mm to (317.8, 37.1), turned to 180 degrees
- moved C403 188.3 mm to (353.1, 23.1)
- moved C410 187.5 mm to (314.5, 34.0), turned to 270 degrees
- moved L401 184.2 mm to (351.8, 30.5)
- moved C409 182.2 mm to (316.7, 34.0), turned to 270 degrees
- moved R411 182.2 mm to (310.1, 34.3), turned to 270 degrees
- moved R407 180.5 mm to (322.3, 39.9), turned to 90 degrees
- moved U402 180.2 mm to (324.4, 35.3), turned to 180 degrees
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Connections:
- C238 pad 1: VAA -> /ADAU1701/AVDD
- C248 pad 1: (no net) -> /ADAU1701/IOVDD
- C308 pad 1: VCOM -> VCC
- C309 pad 1: VCOM -> GNDD
- C309 pad 2: GNDD -> Net-(C309-Pad2)
- C310 pad 1: VCOM -> +5V
- C311 pad 1: VCOM -> Net-(C311-Pad1)
- C312 pad 1: VCOM -> Net-(C312-Pad1)
- C313 pad 1: VCOM -> Net-(C313-Pad1)
- C314 pad 1: VCOM -> Net-(C311-Pad1)
- C315 pad 1: VCOM -> Net-(C312-Pad1)
- C316 pad 1: VCOM -> Net-(C313-Pad1)
- C323 pad 2: (no net) -> GNDD
- C326 pad 2: (no net) -> GNDD
- C329 pad 2: (no net) -> GNDD
- D301 pad 2: Net-(D301-Pad2) -> Net-(C305-Pad2)
- D302 pad 2: Net-(D301-Pad2) -> Net-(D302-Pad2)
- D303 pad 2: Net-(C305-Pad2) -> Net-(C305-Pad1)
- L201 pad 2: (no net) -> /ADAU1701/DVDD
- L301 pad 1: Net-(D301-Pad2) -> Net-(D302-Pad2)
- L302 pad 1: Net-(C305-Pad2) -> Net-(C305-Pad1)
- L302 pad 2: VCOM -> +5V
- R301 pad 1: Net-(R301-Pad1) -> Net-(C311-Pad1)
- R301 pad 2: VCC -> +5V
- R303 pad 1: VCOM -> Net-(C312-Pad1)
- R303 pad 2: Net-(R303-Pad2) -> +5V
- R304 pad 1: Net-(R303-Pad2) -> Net-(C313-Pad1)
- R304 pad 2: Net-(R304-Pad2) -> +5V
- R305 pad 1: Net-(R304-Pad2) -> VCC
- R305 pad 2: GNDD -> Net-(D305-Pad1)
- R306 pad 1: VCOM -> +5V
- R307 pad 1: VCOM -> Net-(C311-Pad1)
- R308 pad 1: VCOM -> Net-(C312-Pad1)
- R309 pad 1: VCOM -> Net-(C313-Pad1)
- R406 pad 2: Net-(R406-Pad2) -> /ClockFanout/CLK
- R407 pad 1: Net-(R406-Pad2) -> /ClockFanout/CLK
- R408 pad 2: (no net) -> /ClockFanout/CLK
- R409 pad 2: (no net) -> Net-(C404-Pad1)
- R529 pad 1: /Connectors/RPI_SDATA_OUT -> /Connectors/RPI_SDATA_IN
- R545 pad 2: (no net) -> /Connectors/RPI_SDATA_IN
- U202 pad 21: (no net) -> /ADAU1701/WP
- U301 pad 1: Net-(C305-Pad1) -> VCC
- U301 pad 2: GNDD -> Net-(C305-Pad2)
- U301 pad 3: Net-(R303-Pad2) -> +5V
- U301 pad 4: Net-(R301-Pad1) -> GNDD
- U301 pad 5: VCC -> +5V
- U301 pad 6: Net-(C305-Pad2) -> Net-(C309-Pad2)
- U302 pad 1: VCOM -> Net-(C311-Pad1)
- U303 pad 1: VCOM -> Net-(C312-Pad1)
- U304 pad 1: VCOM -> Net-(C313-Pad1)
Routing:
- net /ADAU1701/ADCIN_LRCLK0: track 0.00 -> 22.5 mm
- net /ADAU1701/ADCIN_BCLK0: track 0.00 -> 20.1 mm
- net /ADAU1701/DACOUT_SDATA1: track 0.00 -> 20.0 mm
- net /ADAU1701/DACOUT_LRCLK0: track 0.00 -> 18.7 mm
- net /ADAU1701/DACOUT_SDATA0: track 0.00 -> 18.2 mm
- net /ADAU1701/ADCIN_SDATA0: track 0.00 -> 17.8 mm
- net /ADAU1701/DACOUT_BCLK0: track 0.00 -> 17.7 mm
- net /ADAU1701/ADCIN_SDATA1: track 0.00 -> 14.5 mm
- net Net-(C401-Pad1): track 0.00 -> 12.5 mm
- net Net-(P505-Pad5): track 0.00 -> 9.81 mm
- net Net-(R402-Pad2): track 0.00 -> 5.17 mm
- net Net-(P505-Pad3): track 0.00 -> 5.03 mm
- net Net-(C402-Pad1): track 0.00 -> 4.98 mm
- net GNDD: track 0.00 -> 3.65 mm

Commit message: WIP
Parts:
- added C516: 100p, OHDSP-Footprints-Pretty:SMD-0805, F.Cu at (276.2, 120.1)
- added C517: 100p, OHDSP-Footprints-Pretty:SMD-0805, F.Cu at (290.6, 126.2)
- added R242: 0R, OHDSP-Footprints-Pretty:SMD-0805, F.Cu at (284.5, 98.4)
- added R243: 0R, OHDSP-Footprints-Pretty:SMD-0805, F.Cu at (284.5, 100.7)
- added R551: 0R, OHDSP-Footprints-Pretty:SMD-1206, F.Cu at (259.1, 100.3)
- added R552: 0R, OHDSP-Footprints-Pretty:SMD-1206, F.Cu at (259.1, 97.8)
- added R553: 0R, OHDSP-Footprints-Pretty:SMD-1206, F.Cu at (259.1, 95.2)
- added R554: 0R, OHDSP-Footprints-Pretty:SMD-1206, F.Cu at (259.1, 92.7)
- added R555: 0R, OHDSP-Footprints-Pretty:SMD-1206, F.Cu at (259.1, 102.9)
- added R556: 0R, OHDSP-Footprints-Pretty:SMD-1206, F.Cu at (259.1, 105.4)
- added R557: 47R, OHDSP-Footprints-Pretty:SMD-0805, F.Cu at (275.5, 116.8)
- added R558: 47R, OHDSP-Footprints-Pretty:SMD-0805, F.Cu at (296.4, 125.9)
- added R559: 1k, OHDSP-Footprints-Pretty:SMD-0805, F.Cu at (317.5, 88.9)
- C209, C213, C215, C226, C228, C232, C502, C503, C505, C506, C508, C509, C510, C511, C513, C514, L202, L501, R202, R203, R204, R205, R206, R207, R208, R214, R215, R501, R502, R503, R504, R533, R534, R535, R540, R541, R542, R543, R545, R546: moved to F.Cu
- C404: footprint OHDSP-Footprints-Pretty:SMD-0805 -> OHDSP-Footprints-Pretty:CAP-TH-D6.3mmP2.5mm
- R211, R537, R538, R547, R548, R549, R550: footprint OHDSP-Footprints-Pretty:SMD-0805 -> OHDSP-Footprints-Pretty:SMD-1206
- R519: value 47R -> 1k; moved to F.Cu
- U201: footprint OHDSP-Footprints-Pretty:IC_DIP_8 -> OHDSP-Footprints-Pretty:IC_SOIC_8; moved to F.Cu
- moved C232 179.4 mm to (97.5, 138.6), turned to 0 degrees
- moved C512 176.6 mm to (209.6, 120.7), turned to 270 degrees
- moved R519 169.7 mm to (317.5, 77.5), turned to 0 degrees
- moved P502 163.6 mm to (318.8, 81.3)
- moved R550 160.4 mm to (214.6, 91.4)
- moved R549 159.3 mm to (212.1, 96.5)
- moved C515 155.5 mm to (209.6, 90.2), turned to 270 degrees
- moved P503 144.8 mm to (318.8, 92.7)
- moved R226 144.2 mm to (359.4, 90.2)
- moved C506 142.7 mm to (242.6, 106.7)
- moved P514 142.0 mm to (207.0, 99.1), turned to 270 degrees
- moved R548 142.0 mm to (213.4, 109.2)
- moved R416 138.1 mm to (249.6, 115.6), turned to 90 degrees
- moved P513 136.8 mm to (207.0, 109.2), turned to 270 degrees
- moved C513 136.5 mm to (209.6, 110.5), turned to 270 degrees
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Connections:
- C505 pad 1: Net-(C505-Pad1) -> (no net)
- C506 pad 1: /ADAU1701/ADC_IN0 -> Net-(C506-Pad1)
- C507 pad 1: /ADAU1701/ADC_IN1 -> Net-(C507-Pad1)
- C508 pad 1: /Connectors/ANA_OUT1 -> Net-(C508-Pad1)
- C509 pad 1: /Connectors/ANA_OUT2 -> Net-(C509-Pad1)
- C510 pad 1: /Connectors/ANA_OUT3 -> Net-(C510-Pad1)
- C511 pad 1: /Connectors/ANA_OUT4 -> Net-(C511-Pad1)
- D501 pad 2: /ADAU1701/ADC_IN0 -> Net-(C506-Pad1)
- D502 pad 2: /ADAU1701/ADC_IN1 -> Net-(C507-Pad1)
- D503 pad 1: /ADAU1701/ADC_IN0 -> Net-(C506-Pad1)
- D504 pad 1: /ADAU1701/ADC_IN1 -> Net-(C507-Pad1)
- P502 pad 1: GNDD -> /ADAU1701/I2C_SCL
- P502 pad 2: Net-(C501-Pad1) -> (no net)
- P502 pad 3: GNDD -> /ADAU1701/I2C_SDA
- P502 pad 4: Net-(C501-Pad1) -> (no net)
- P502 pad 5: /ADAU1701/I2C_SCL -> (no net)
- P502 pad 6: GNDD -> Net-(P502-Pad6)
- P502 pad 7: /ADAU1701/I2C_SDA -> (no net)
- P502 pad 8: GNDD -> (no net)
- P502 pad 9: GNDD -> (no net)
- P503 pad 1: GNDD -> /ADAU1701/I2C_SCL
- P503 pad 2: Net-(C501-Pad1) -> (no net)
- P503 pad 3: GNDD -> /ADAU1701/I2C_SDA
- P503 pad 4: Net-(C501-Pad1) -> (no net)
- P503 pad 5: /ADAU1701/I2C_SCL -> (no net)
- P503 pad 6: GNDD -> Net-(P503-Pad6)
- P503 pad 7: /ADAU1701/I2C_SDA -> (no net)
- P503 pad 8: GNDD -> (no net)
- P503 pad 9: GNDD -> (no net)
- R219 pad 1: Net-(R219-Pad1) -> VPP
- R221 pad 1: Net-(R219-Pad1) -> VPP
- R412 pad 1: /ADAU1701/MCLK -> /Connectors/ADC_MCLK
- R413 pad 1: /Connectors/ADC_MCLK -> /ADAU1701/MCLK
- R416 pad 2: /ADAU1701/MCLK -> /Connectors/ADC_MCLK
- R417 pad 2: /Connectors/ADC_MCLK -> /ADAU1701/MCLK
- R519 pad 1: Net-(C505-Pad1) -> /Connectors/ADC_RESET
- R519 pad 2: Net-(C501-Pad1) -> Net-(P502-Pad6)
- U202 pad 22: /ADAU1701/I2C_SDA -> Net-(R242-Pad2)
- U202 pad 23: /ADAU1701/I2C_SCL -> Net-(R243-Pad2)
Routing:
- net Net-(C506-Pad1): track 0.00 -> 15.7 mm
- net /Connectors/ANA_OUT4: track 0.00 -> 12.8 mm
- net /Connectors/ANA_OUT3: track 0.00 -> 11.5 mm
- net /Connectors/ANA_OUT1: track 0.00 -> 10.6 mm
- net /ADAU1701/ADC_IN1: track 0.00 -> 10.3 mm
- net /Connectors/ANA_OUT2: track 0.00 -> 10.3 mm
- net /ADAU1701/ADC_IN0: track 0.00 -> 9.94 mm
- net /ClockFanout/CLK: track 0.00 -> 9.60 mm
- net Net-(C401-Pad1): track 12.5 -> 3.20 mm
- net Net-(C507-Pad2): track 0.00 -> 8.34 mm
- net Net-(C404-Pad1): track 0.00 -> 7.56 mm
- net Net-(C507-Pad1): track 0.00 -> 6.12 mm
- net Net-(C506-Pad2): track 0.00 -> 5.86 mm
- net Net-(R402-Pad2): track 5.17 -> 0.00 mm
- net Net-(R408-Pad1): track 0.00 -> 3.79 mm
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