File: Schematics/OHDSP-ADAU1701.kicad_pcb (KiCad board)
At the start: 4 copper layers, 100 x 100 mm, 301 parts, among them CN401 COAX, CN402 COAX, P201 CONN_2x1, P301 PIN, P302 PIN, P303 PIN, P305 CONN_2x1, P306 PIN, P501 CONN_02X10, P502 CONN_02X05, P503 CONN_02X05, P504 CONN_02X05, P505 CONN_02X10, P506 CONN_2x1, P507 CONN_2x1, P508 CONN_02X20, P509 CONN_02X05, P510 CONN_02X05, P511 CONN_02X05, P512 CONN_2x1, P513 CONN_2x1, P514 CONN_2x1, P515 CONN_2x1, SW201 SWITCH, U201 ADM13307-5ARZ, U202 ADAU1701JSTZ, U203 IC-EEPROM-I2C, U301 LT1374CS8-5#PBF, U302 NCP700BSN33T1G, U303 NCP700BSN33T1G, U304 NCP700BSN18T1G, U401 NC7SZU04M5X, U402 NC7SZU04M5X, U403 NB3L553, X401 24M576

Commit message: WIP
Parts:
- C305, D303, R305, U301: moved to F.Cu
- U203: footprint OHDSP-Footprints-Pretty:IC_DIP_8 -> OHDSP-Footprints-Pretty:IC_SOIC_8
- moved R310 208.5 mm to (462.8, 113.3)
- moved D305 202.0 mm to (466.6, 113.3)
- moved D306 194.0 mm to (466.6, 115.3), turned to 180 degrees
- moved L302 181.2 mm to (473.7, 104.1), turned to 0 degrees
- moved C309 160.7 mm to (460.2, 110.5), turned to 0 degrees
- moved P504 156.1 mm to (318.8, 72.4), turned to 90 degrees
- moved C305 150.8 mm to (462.3, 99.1), turned to 180 degrees
- moved U301 146.8 mm to (458.5, 104.1), turned to 0 degrees
- moved D303 136.2 mm to (462.3, 91.4)
- moved C310 134.1 mm to (480.1, 91.4)
- moved D301 134.1 mm to (457.5, 116.1)
- moved C308 128.8 mm to (452.1, 97.8), turned to 90 degrees
- moved C301 110.3 mm to (449.6, 97.8), turned to 270 degrees
- moved C302 105.2 mm to (454.7, 97.8), turned to 270 degrees
- moved R305 104.4 mm to (455.9, 110.5)
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Routing:
- net /ADAU1701/SELFBOOT: track 0.00 -> 30.5 mm
- net /ADAU1701/DACOUT_SDATA1: track 20.0 -> 0.00 mm
- net /ADAU1701/DACOUT_LRCLK0: track 18.7 -> 0.08 mm
- net /ADAU1701/DACOUT_SDATA0: track 18.2 -> 0.00 mm
- net /ADAU1701/DACOUT_BCLK0: track 17.7 -> 0.00 mm
- net /Connectors/ANA_OUT4: track 12.8 -> 0.00 mm
- net /Connectors/ANA_OUT3: track 11.5 -> 0.00 mm
- net /Connectors/ANA_OUT1: track 10.6 -> 0.00 mm
- net /Connectors/ANA_OUT2: track 10.3 -> 0.00 mm
- net Net-(C507-Pad1): track 6.12 -> 0.00 mm
- net Net-(C309-Pad2): track 0.00 -> 5.59 mm
- net Net-(P501-Pad2): track 0.00 -> 3.85 mm
- net /ADAU1701/ADC_IN1: track 10.3 -> 12.9 mm
- net /ADAU1701/ADCIN_LRCLK0: track 21.5 -> 19.2 mm
- net /ADAU1701/ADCIN_SDATA1: track 14.5 -> 16.5 mm
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
Commit message: WIP
Parts:
- C309: moved to B.Cu
- C311, C317, C320, R301, R307, U302: moved to F.Cu
- moved U304 180.5 mm to (467.5, 248.0)
- moved C331 175.0 mm to (481.5, 245.5)
- moved C330 169.6 mm to (487.0, 208.0)
- moved U303 164.8 mm to (462.0, 211.0)
- moved C328 156.1 mm to (474.0, 244.5)
- moved C319 143.9 mm to (456.0, 250.0)
- moved C329 140.9 mm to (455.5, 154.5), turned to 180 degrees
- moved R309 138.4 mm to (465.5, 255.0)
- moved C325 137.2 mm to (469.0, 238.5)
- moved C321 136.6 mm to (469.0, 207.0)
- moved C322 136.2 mm to (457.0, 242.0)
- moved C320 136.0 mm to (463.5, 157.5), turned to 270 degrees
- moved U302 134.4 mm to (460.5, 157.5), turned to 0 degrees
- moved C313 133.5 mm to (456.5, 238.0)
- moved C327 126.5 mm to (476.5, 210.0)
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Routing:
- net Net-(C309-Pad2): track 5.59 -> 0.00 mm

Commit message: WIP
Parts:
- removed C204, C225, C234, C403, C411, C505: 100p, OHDSP-Footprints-Pretty:SMD-0805
- removed C401: 33p, OHDSP-Footprints-Pretty:SMD-0805
- removed C409, C501, C502: 100n, OHDSP-Footprints-Pretty:SMD-0805
- removed C410, C503: 22u, OHDSP-Footprints-Pretty:SMD-0805
- removed C504: 220u, OHDSP-Footprints-Pretty:CAP-TH-D6.3mmP2.5mm
- removed L501: 600R@100MHz, OHDSP-Footprints-Pretty:SMD-0805
- removed R201, R212, R220, R405, R411: 47R, OHDSP-Footprints-Pretty:SMD-0805
- removed R210, R408: 0R, OHDSP-Footprints-Pretty:SMD-0805
- removed R401, R416, R417, R418: N/F, OHDSP-Footprints-Pretty:SMD-0805
- removed R402: 1Meg, OHDSP-Footprints-Pretty:SMD-0805
- removed R410: 100R, OHDSP-Footprints-Pretty:SMD-0805
- removed U401, U402: NC7SZU04M5X, OHDSP-Footprints-Pretty:IC-SOT23-5
- removed X401: 24M576, OHDSP-Footprints-Pretty:XTAL_HC49_TH
- added R560: 0R, OHDSP-Footprints-Pretty:SMD-1206, F.Cu at (286.6, 95.5)
- added R561: 0R, OHDSP-Footprints-Pretty:SMD-1206, F.Cu at (284.2, 95.5)
- added XTAL401: XTAL-OSC-4PIN, OHDSP-Footprints-Pretty:XTAL_8_DIL, F.Cu at (283.2, 81.9)
- C205, C206, C207, C210, C211, C212, C223, C224, C316, C325, C328, C405, C406, C516, C517, R209, R211, R217, R218, R514, R515, R516, R517, R518, R520, R530, R531, R532, R533, R534, R535, R536, R551, R552, R553, R554, R555, R556, R557, R558: moved to B.Cu
- C312, C318, C319, C321, R233, R303, R304, R308, R544, U304: moved to F.Cu
- C402: value 33p -> 100n
- R404: value 100R -> 1k
- R406: value 0R -> N/F
- R407: value 0R -> 27R
- moved R502 195.4 mm to (270.3, 53.3)
- moved R545 190.8 mm to (267.3, 60.3)
- moved R503 177.0 mm to (264.7, 51.3)
- moved R546 173.9 mm to (273.7, 62.9)
- moved R501 172.9 mm to (266.2, 45.7)
- moved R539 171.6 mm to (231.8, 78.7)
- moved R542 169.7 mm to (279.4, 54.6)
- moved R544 165.3 mm to (241.9, 66.7)
- moved R529 161.9 mm to (287.0, 62.2)
- moved R540 158.5 mm to (228.0, 78.7), turned to 90 degrees
- moved R536 152.0 mm to (297.0, 97.0), turned to 90 degrees
- moved R532 140.1 mm to (294.6, 111.8), turned to 180 degrees
- moved R514 135.8 mm to (258.1, 115.8)
- moved R535 129.6 mm to (294.6, 101.6), turned to 180 degrees
- moved R533 129.2 mm to (294.6, 107.7)
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Connections:
- C227 pad 2: Net-(C227-Pad2) -> GNDD
- C229 pad 2: Net-(C227-Pad2) -> GNDD
- C230 pad 2: Net-(C227-Pad2) -> GNDD
- C231 pad 2: Net-(C227-Pad2) -> GNDD
- C233 pad 2: Net-(C227-Pad2) -> GNDD
- P502 pad 1: /ADAU1701/I2C_SCL -> /Connectors/SL_SCL
- P502 pad 3: /ADAU1701/I2C_SDA -> /Connectors/SL_SDA
- P503 pad 1: /ADAU1701/I2C_SCL -> /Connectors/SL_SCL
- P503 pad 3: /ADAU1701/I2C_SDA -> /Connectors/SL_SDA
- P504 pad 1: /ADAU1701/I2C_SCL -> /Connectors/SL_SCL
- P504 pad 3: /ADAU1701/I2C_SDA -> /Connectors/SL_SDA
- R403 pad 1: Net-(R401-Pad1) -> Net-(CN401-Pad1)
- R404 pad 1: Net-(C402-Pad1) -> Net-(C407-Pad1)
- R404 pad 2: Net-(R402-Pad2) -> Net-(C402-Pad1)
- R406 pad 1: Net-(R401-Pad1) -> Net-(CN401-Pad1)
- R504 pad 2: Net-(P501-Pad2) -> /Connectors/ADC_MCLK
- R514 pad 2: /ADAU1701/ADCIN_SDATA0 -> Net-(P501-Pad8)
- R515 pad 2: /ADAU1701/ADCIN_BCLK0 -> Net-(P501-Pad6)
- R516 pad 2: /ADAU1701/ADCIN_LRCLK0 -> Net-(P501-Pad4)
- R517 pad 2: /ADAU1701/ADCIN_SDATA3 -> Net-(P501-Pad14)
- R518 pad 2: /ADAU1701/ADCIN_SDATA2 -> Net-(P501-Pad12)
- R520 pad 2: /ADAU1701/ADCIN_SDATA1 -> Net-(P501-Pad10)
- R522 pad 1: /ADAU1701/DACOUT_LRCLK0 -> /ADAU1701/DACOUT_SDATA2
- R523 pad 1: /ADAU1701/DACOUT_BCLK0 -> /ADAU1701/DACOUT_SDATA3
- R524 pad 1: /ADAU1701/DACOUT_SDATA0 -> /ADAU1701/DACOUT_BCLK0
- R525 pad 1: /ADAU1701/DACOUT_SDATA1 -> /ADAU1701/DACOUT_LRCLK0
- R526 pad 1: /ADAU1701/DACOUT_SDATA2 -> /ADAU1701/DACOUT_SDATA0
- R527 pad 1: /ADAU1701/DACOUT_SDATA3 -> /ADAU1701/DACOUT_SDATA1
- R530 pad 2: Net-(P505-Pad13) -> /ADAU1701/DACOUT_SDATA1
- R531 pad 2: Net-(P505-Pad11) -> /ADAU1701/DACOUT_SDATA0
- R532 pad 2: Net-(P505-Pad9) -> /ADAU1701/DACOUT_LRCLK0
- R533 pad 2: Net-(P505-Pad7) -> /ADAU1701/DACOUT_BCLK0
- R534 pad 2: Net-(P505-Pad5) -> /ADAU1701/DACOUT_SDATA3
- R535 pad 2: Net-(P505-Pad3) -> /ADAU1701/DACOUT_SDATA2
- R536 pad 2: Net-(P505-Pad1) -> /Connectors/DAC_MCLK
- R539 pad 1: /ADAU1701/I2C_SDA -> /Connectors/SL_SDA
- R540 pad 1: /ADAU1701/I2C_SCL -> /Connectors/SL_SCL
- U202 pad 32: Net-(R210-Pad1) -> /ADAU1701/MCLK
- U403 pad 5: Net-(R408-Pad1) -> /ClockFanout/CLK
Routing:
- net /Connectors/ADC_MCLK: track 2.03 -> 34.7 mm
- net /ADAU1701/SELFBOOT: track 30.5 -> 0.00 mm
- net /Connectors/SL_SDA: track 0.00 -> 29.5 mm
- net /Connectors/SL_SCL: track 0.00 -> 28.9 mm
- net /ADAU1701/DACOUT_SDATA3: track 0.00 -> 23.3 mm
- net /ADAU1701/DACOUT_SDATA2: track 0.00 -> 22.9 mm
- net /ADAU1701/DACOUT_SDATA1: track 0.00 -> 22.1 mm
- net /ADAU1701/ADCIN_SDATA2: track 0.00 -> 22.1 mm, vias 0 -> 2
- net /Connectors/DAC_MCLK: track 0.00 -> 22.0 mm
- net /ADAU1701/DACOUT_SDATA0: track 0.00 -> 21.2 mm
- net /ADAU1701/ADCIN_SDATA3: track 0.00 -> 21.1 mm, vias 0 -> 2
- net (no net): track 0.00 -> 21.0 mm
- net /ADAU1701/DACOUT_LRCLK0: track 0.08 -> 19.3 mm
- net /ADAU1701/DACOUT_BCLK0: track 0.00 -> 18.3 mm
- net Net-(CN401-Pad1): track 0.00 -> 17.2 mm
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Other:
- board text added: "Seeed Studio/Fusion PCB do a 1mm stackup that would give reasonable trace widths For 50ohm on top use inner top layer as ground (5mil thick) Trace width is 0.24mm, ground clearance anything <1mm For 75ohm on top use inner bottom layer as ground (29mil thick) Trace width is 0.5mm with ground on 0.4mm clearance OR Trace width is 0.45mm with ground on 0.3mm clearance For 90ohm on top use inner botto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"
- board text removed: "Seeed Studio/Fusion PCB do a 1mm stackup that would give reasonable trace widths For 50ohm on top use inner top layer as ground (5mil thick) Trace width is 0.24mm, ground clearance anything <1mm For 75ohm on top use inner bottom layer as ground (29mil thick) Trace width is 0.5mm with ground on 0.4mm clearance OR Trace width is 0.45mm with ground on 0.3mm clearance For 100ohm on top use inner bott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"

Commit message: WIP
Parts:
- removed C219, C222: 10n, OHDSP-Footprints-Pretty:SMD-0805
- C246: moved to F.Cu
- moved C218 94.0 mm to (277.2, 108.8), turned to 270 degrees
- moved D503 70.8 mm to (222.1, 153.2)
- moved C221 51.3 mm to (278.5, 98.7), turned to 180 degrees
- moved C246 47.6 mm to (268.5, 97.7), turned to 270 degrees
- moved C244 43.0 mm to (268.0, 107.3), turned to 0 degrees
- moved C207 31.3 mm to (268.2, 94.9), turned to 90 degrees
- moved C212 30.0 mm to (266.2, 94.9), turned to 90 degrees
- moved C203 27.4 mm to (264.2, 95.0), turned to 90 degrees
- moved C405 11.4 mm to (263.5, 86.4), turned to 180 degrees
- moved C404 8.84 mm to (263.5, 88.3), turned to 180 degrees
- moved C406 6.37 mm to (263.5, 90.2), turned to 180 degrees
- moved C210 3.87 mm to (263.1, 108.2), turned to 180 degrees
- moved C211 3.51 mm to (259.5, 96.4), turned to 135 degrees
- moved R505 3.03 mm to (252.7, 116.1)
- moved C206 2.70 mm to (260.2, 94.2), turned to 135 degrees
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Connections:
- R522 pad 1: /ADAU1701/DACOUT_SDATA2 -> /ADAU1701/DACOUT_SDATA3
- R523 pad 1: /ADAU1701/DACOUT_SDATA3 -> /ADAU1701/DACOUT_SDATA2
- R534 pad 2: /ADAU1701/DACOUT_SDATA3 -> /ADAU1701/DACOUT_SDATA2
- R535 pad 2: /ADAU1701/DACOUT_SDATA2 -> /ADAU1701/DACOUT_SDATA3
Routing:
- net /ADAU1701/DACOUT_SDATA2: track 22.9 -> 43.5 mm
- net /ADAU1701/DACOUT_SDATA3: track 23.3 -> 3.12 mm
- net /Connectors/ANA_OUT4: track 0.00 -> 13.5 mm, vias 0 -> 1
- net /Connectors/ANA_OUT1: track 0.00 -> 13.0 mm, vias 0 -> 1
- net /Connectors/ANA_OUT3: track 0.00 -> 12.6 mm, vias 0 -> 1
- net /Connectors/ANA_OUT2: track 0.00 -> 12.4 mm, vias 0 -> 1
- net /ADAU1701/FILTD: track 0.00 -> 10.8 mm
- net /ADAU1701/CM: track 0.00 -> 7.09 mm
- net /ADAU1701/ADC_IN1: track 19.3 -> 16.2 mm
- net Net-(R211-Pad1): track 0.61 -> 3.52 mm, vias 0 -> 1
- net Net-(P501-Pad2): track 3.85 -> 2.20 mm
- net /ADAU1701/ADCIN_SDATA0: track 20.9 -> 19.7 mm
- net /ADAU1701/ADCIN_LRCLK0: track 24.2 -> 23.1 mm
- net /ADAU1701/ADCIN_BCLK0: track 22.4 -> 21.3 mm
- net /ADAU1701/ADC_IN0: track 14.5 -> 13.5 mm
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