File: Schematics/SPDIF.sch (KiCad schematic (older format))
At the start: 15 parts, among them U501 IC-SPDIF-RX-OPTO, U502 IC-SPDIF-TX-OPTO

Commit message: WIP
Add master audio clock to I2S headers.
Parts:
- renumbered C501 to C401, C503 to C402, C504 to C403, C508 to C404, C509 to C405, C505 to C406, C506 to C407, C507 to C408, L501 to L401, R501 to R401, R502 to R402, R503 to R403, R504 to R404, U501 to U401, U502 to U402
Changed lines of the file:
@@
 $Descr A4 11693 8268
 encoding utf-8
-Sheet 5 7
+Sheet 5 6
 Title ""
 Date ""
@@
 $EndDescr
 $Comp
-L C C505
+L C C406
 U 1 1 54E21C5D
 P 6350 3100
-F 0 "C505" H 6350 3200 40  0000 L CNN
+F 0 "C406" H 6350 3200 40  0000 L CNN
 F 1 "100n" H 6356 3015 40  0000 L CNN
 F 2 "OHDSP-Footprints-Pretty:SMD-0805" H 6388 2950 30  0001 C CNN
@@
 $EndComp
 $Comp
-L GNDD #PWR096
+L GNDD #PWR089
 U 1 1 54E21D36
 P 6350 3350
-F 0 "#PWR096" H 6350 3100 60  0001 C CNN
+F 0 "#PWR089" H 6350 3100 60  0001 C CNN
 F 1 "GNDD" H 6350 3200 60  0000 C CNN
 F 2 "" H 6350 3350 60  0000 C CNN
@@
 $EndComp
 $Comp
-L C C506
+L C C407
 U 1 1 54E21F71
 P 6400 4550
-F 0 "C506" H 6400 4650 40  0000 L CNN
+F 0 "C407" H 6400 4650 40  0000 L CNN
 F 1 "100n" H 6406 4465 40  0000 L CNN
 F 2 "OHDSP-Footprints-Pretty:SMD-0805" H 6438 4400 30  0001 C CNN
@@
 $EndComp
 $Comp
-L GNDD #PWR097
+L GNDD #PWR090
 U 1 1 54E607CA
 P 6400 4800
-F 0 "#PWR097" H 6400 4550 60  0001 C CNN
+F 0 "#PWR090" H 6400 4550 60  0001 C CNN
 F 1 "GNDD" H 6400 4650 60  0000 C CNN
 F 2 "" H 6400 4800 60  0000 C CNN
@@
 $EndComp
 $Comp
-L INDUCTOR L501
+L INDUCTOR L401
 U 1 1 54E2473D
 P 3800 2100
-F 0 "L501" V 3750 2100 40  0000 C CNN
+F 0 "L401" V 3750 2100 40  0000 C CNN
 F 1 "600R@100MHz" V 3900 2100 40  0000 C CNN
 F 2 "OHDSP-Footprints-Pretty:SMD-0805" H 3800 2100 60  0001 C CNN
@@
 $EndComp
 $Comp
-L C C501
+L C C401
 U 1 1 54E24744
 P 4250 2950
-F 0 "C501" H 4250 3050 40  0000 L CNN
+F 0 "C401" H 4250 3050 40  0000 L CNN
 F 1 "100p" H 4256 2865 40  0000 L CNN
 F 2 "OHDSP-Footprints-Pretty:SMD-0805" H 4288 2800 30  0000 C CNN
@@
 $EndComp
 $Comp
-L R R501
+L R R401
 U 1 1 54E2474B
 P 4250 2400
-F 0 "R501" V 4330 2400 40  0000 C CNN
+F 0 "R401" V 4330 2400 40  0000 C CNN
 F 1 "47R" V 4257 2401 40  0000 C CNN
 F 2 "OHDSP-Footprints-Pretty:SMD-0805" V 4180 2400 30  0001 C CNN
@@
 $EndComp
 $Comp
-L GNDD #PWR098
+L GNDD #PWR091
 U 1 1 54E24752
 P 4250 3250
-F 0 "#PWR098" H 4250 3000 60  0001 C CNN
+F 0 "#PWR091" H 4250 3000 60  0001 C CNN
 F 1 "GNDD" H 4250 3100 60  0000 C CNN
 F 2 "" H 4250 3250 60  0000 C CNN
@@
 $EndComp
 $Comp
-L C C504
+L C C403
 U 1 1 54E2475F
 P 5250 2700
-F 0 "C504" H 5250 2800 40  0000 L CNN
+F 0 "C403" H 5250 2800 40  0000 L CNN
 F 1 "100n" H 5256 2615 40  0000 L CNN
 F 2 "OHDSP-Footprints-Pretty:SMD-0805" H 5288 2550 30  0000 C CNN
@@
 $EndComp
 $Comp
-L C C503
+L C C402
 U 1 1 54E24766
 P 4950 2700
-F 0 "C503" H 4950 2800 40  0000 L CNN
+F 0 "C402" H 4950 2800 40  0000 L CNN
 F 1 "22u" H 4956 2615 40  0000 L CNN
 F 2 "OHDSP-Footprints-Pretty:SMD-0805" H 4988 2550 30  0000 C CNN
@@
 $EndComp
 $Comp
-L VPP #PWR099
+L VPP #PWR092
 U 1 1 54E607D2
 P 3400 1950
-F 0 "#PWR099" H 3400 1800 60  0001 C CNN
+F 0 "#PWR092" H 3400 1800 60  0001 C CNN
 F 1 "VPP" H 3400 2100 60  0000 C CNN
 F 2 "" H 3400 1950 60  0000 C CNN
@@
 SPDIF Optical Input and Output
 $Comp
-L IC-SPDIF-RX-OPTO U501
+L IC-SPDIF-RX-OPTO U401
 U 1 1 54E30C44
 P 6750 3100
-F 0 "U501" V 6600 2450 59  0000 C CNN
+F 0 "U401" V 6600 2450 59  0000 C CNN
 F 1 "IC-SPDIF-RX-OPTO" V 6700 2850 59  0000 C CNN
 F 2 "OHDSP-Footprints-Pretty:IC_SPDIF_OPTO" H 6750 3100 118 0001 C CNN
@@
 $EndComp
 $Comp
-L IC-SPDIF-TX-OPTO U502
+L IC-SPDIF-TX-OPTO U402
 U 1 1 54E30C95
 P 6750 4500
-F 0 "U502" V 6650 3850 59  0000 C CNN
+F 0 "U402" V 6650 3850 59  0000 C CNN
 F 1 "IC-SPDIF-TX-OPTO" V 6750 4200 59  0000 C CNN
 F 2 "OHDSP-Footprints-Pretty:IC_SPDIF_OPTO" H 6750 4500 118 0001 C CNN
@@
 $EndComp
 $Comp
-L GNDD #PWR0100
+L GNDD #PWR093
 U 1 1 54E30F61
 P 6900 3800
-F 0 "#PWR0100" H 6900 3550 60  0001 C CNN
+F 0 "#PWR093" H 6900 3550 60  0001 C CNN
 F 1 "GNDD" H 6900 3650 60  0000 C CNN
 F 2 "" H 6900 3800 60  0000 C CNN
@@
 $EndComp
 $Comp
-L GNDD #PWR0101
+L GNDD #PWR094
 U 1 1 54E30F88
 P 6900 5250
-F 0 "#PWR0101" H 6900 5000 60  0001 C CNN
+F 0 "#PWR094" H 6900 5000 60  0001 C CNN
 F 1 "GNDD" H 6900 5100 60  0000 C CNN
 F 2 "" H 6900 5250 60  0000 C CNN
@@
 SPDIF_TX
 $Comp
-L R R503
+L R R403
 U 1 1 54E313A7
 P 7750 4800
-F 0 "R503" V 7830 4800 40  0000 C CNN
+F 0 "R403" V 7830 4800 40  0000 C CNN
 F 1 "0R" V 7757 4801 40  0000 C CNN
 F 2 "OHDSP-Footprints-Pretty:SMD-0805" V 7680 4800 30  0001 C CNN
@@
 $EndComp
 $Comp
-L R R502
+L R R402
 U 1 1 54E3151C
 P 7300 3000
-F 0 "R502" V 7380 3000 40  0000 C CNN
+F 0 "R402" V 7380 3000 40  0000 C CNN
 F 1 "10k" V 7307 3001 40  0000 C CNN
 F 2 "OHDSP-Footprints-Pretty:SMD-0805" V 7230 3000 30  0001 C CNN
@@
 Connection ~ 7300 3400
 $Comp
-L C C507
+L C C408
 U 1 1 54E31704
 P 7750 3400
-F 0 "C507" H 7750 3500 40  0000 L CNN
+F 0 "C408" H 7750 3500 40  0000 L CNN
 F 1 "10n" H 7756 3315 40  0000 L CNN
 F 2 "OHDSP-Footprints-Pretty:SMD-0805" H 7788 3250 30  0000 C CNN
@@
 Copyright Paul Janicki 2015\n\nLicensed under the TAPR Open Hardware License (www.tapr.org/OHL).\n\nThis documentation is distributed\nWITHOUT ANY EXPRESS OR IMPLIED WARRANTY, INCLUDING OF\nMERCHANTABILITY, SATISFACTORY QUALITY AND FITNESS FOR A\nPARTICULAR PURPOSE.\n
 $Comp
-L R R504
+L R R404
 U 1 1 55004FB3
 P 8350 3400
-F 0 "R504" V 8430 3400 40  0000 C CNN
+F 0 "R404" V 8430 3400 40  0000 C CNN
 F 1 "22R" V 8357 3401 40  0000 C CNN
 F 2 "OHDSP-Footprints-Pretty:SMD-0805" V 8280 3400 30  0001 C CNN
@@
 	8700 3400 8600 3400
 $Comp
-L C C508
+L C C404
 U 1 1 5500568E
 P 6050 3100
-F 0 "C508" H 6050 3200 40  0000 L CNN
+F 0 "C404" H 6050 3200 40  0000 L CNN
 F 1 "22u" H 6056 3015 40  0000 L CNN
 F 2 "OHDSP-Footprints-Pretty:SMD-0805" H 6088 2950 30  0000 C CNN
@@
 $EndComp
 $Comp
-L C C509
+L C C405
 U 1 1 550056ED
 P 6100 4550
-F 0 "C509" H 6100 4650 40  0000 L CNN
+F 0 "C405" H 6100 4650 40  0000 L CNN
 F 1 "22u" H 6106 4465 40  0000 L CNN
 F 2 "OHDSP-Footprints-Pretty:SMD-0805" H 6138 4400 30  0000 C CNN
@@
 $EndComp
 $Comp
-L GNDD #PWR0102
+L GNDD #PWR095
 U 1 1 5500577B
 P 6050 3350
-F 0 "#PWR0102" H 6050 3100 60  0001 C CNN
+F 0 "#PWR095" H 6050 3100 60  0001 C CNN
 F 1 "GNDD" H 6050 3200 60  0000 C CNN
 F 2 "" H 6050 3350 60  0000 C CNN
@@
 $EndComp
 $Comp
-L GNDD #PWR0103
+L GNDD #PWR096
 U 1 1 55005796
 P 6100 4800
-F 0 "#PWR0103" H 6100 4550 60  0001 C CNN
+F 0 "#PWR096" H 6100 4550 60  0001 C CNN
 F 1 "GNDD" H 6100 4650 60  0000 C CNN
 F 2 "" H 6100 4800 60  0000 C CNN
