File: Schematics/AD1937 CODEC.sch (KiCad schematic (older format))
At the start: 53 parts, among them P201 CONN_2x1

Commit message: WIP
Connections:
- net labels added: AD1937_CM
Changed lines of the file:
@@
 LIBS:power
 LIBS:OHDSP-Lib
+LIBS:OHDSP-XOVER-cache
 EELAYER 25 0
 EELAYER END
 $Descr A3 16535 11693
 encoding utf-8
-Sheet 6 7
+Sheet 6 9
 Title ""
 Date "10 feb 2015"
@@
 	15150 6150 15150 6200
 Wire Wire Line
-	13850 6150 15150 6150
+	13850 6150 15250 6150
 Wire Wire Line
 	14800 6150 14800 6200
@@
 Wire Wire Line
 	13350 3650 13250 3650
+Text HLabel 15250 6150 2    60   Output ~ 0
+AD1937_CM
+Connection ~ 15150 6150
 $EndSCHEMATC

Commit message: WIP
Parts:
- removed C208, C238: 220u, OHDSP-Footprints-Pretty:CAP-TH-D6.3mmP2.5mm, symbol CP1
- removed C211, C216, C218, C244, C246: 100n, OHDSP-Footprints-Pretty:SMD-0805, symbol C
- removed C217, C245: 1u, OHDSP-Footprints-Pretty:SMD-0805, symbol C
- removed C223: 5n6, OHDSP-Footprints-Pretty:SMD-0805, symbol C
- removed C239: 100p, OHDSP-Footprints-Pretty:SMD-0805, symbol C
- removed C240: 22u, OHDSP-Footprints-Pretty:SMD-0805, symbol C
- removed L205: 600R@100MHz, OHDSP-Footprints-Pretty:SMD-0805, symbol INDUCTOR
- removed R209: 562R, OHDSP-Footprints-Pretty:SMD-0805, symbol R
- removed R217: 0R, OHDSP-Footprints-Pretty:SMD-0805, symbol R
- removed R230, R231: 10k, OHDSP-Footprints-Pretty:SMD-0805, symbol R
- added C501: 220u, OHDSP-Footprints-Pretty:CAP-TH-D6.3mmP2.5mm, symbol CP1
- added C503, C505, C516, C518, C523: 100n, OHDSP-Footprints-Pretty:SMD-0805, symbol C
- added C504, C517: 1u, OHDSP-Footprints-Pretty:SMD-0805, symbol C
- added C508: 100p, OHDSP-Footprints-Pretty:SMD-0805, symbol C
- added C509: 5n6, OHDSP-Footprints-Pretty:SMD-0805, symbol C
- added C511: 220u, OHDSP-Footprints-Pretty:CAP-TH-D8mmP3.5mm, symbol CP1
- added C512: 22u, OHDSP-Footprints-Pretty:SMD-0805, symbol C
- added L502: 600R@100MHz, OHDSP-Footprints-Pretty:SMD-0805, symbol INDUCTOR
- added R503: 0R, OHDSP-Footprints-Pretty:SMD-0805, symbol R
- added R512: 562R, OHDSP-Footprints-Pretty:SMD-0805, symbol R
- added R514, R515: 10k, OHDSP-Footprints-Pretty:SMD-0805, symbol R
- U501: renamed from U?; footprint (none) -> OHDSP-Footprints-Pretty:IC-LQFP64
- gave numbers to parts that had none: 20
- renumbered C214 to C502, C220 to C506, C221 to C507, C224 to C510, C242 to C514, C243 to C515, C212 to C524, C206 to C525, C207 to C526, C202 to C527, C203 to C528, L201 to L501, P201 to P501, R225 to R504, R224 to R513
