File: Schematics/AD1937_AnaIn.sch (KiCad schematic (older format))
At the start: 149 parts

Commit message: WIP
Connections:
- net +12VA: now also U?.7; no longer U?.8
- net -12VA: now also U?.4; no longer U?.4
- net AD1937_ANAIN_1N: no longer C?.2, C?.2, C?.2, R?.2, R?.2, R?.2
- net AD1937_ANAIN_1P: no longer C?.2, C?.2, C?.2, R?.2, R?.2, R?.2
- new net AD1937_ANAIN_2N: C?.2, R?.2
- new net AD1937_ANAIN_2P: C?.2, R?.2
- new net AD1937_ANAIN_3N: C?.2, R?.2
- new net AD1937_ANAIN_3P: C?.2, R?.2
- new net AD1937_ANAIN_4N: C?.2, R?.2
- new net AD1937_ANAIN_4P: C?.2, R?.2
Other:
- note added: "Copyright Paul Janicki 2015\n\nLicensed under the TAPR Open Hardware License (www.tapr.org/OHL).\n\nThis documentation is distributed\nWITHOUT ANY EXPRESS OR IMPLIED WARRANTY, INCLUDING OF\nMERCHANTABILITY, SATISFACTORY QUALITY AND FITNESS FOR A\nPARTICULAR PURPOSE.\n"

Commit message: WIP
Parts:
- C701, C702, C704, C706, C707, C708, C712, C714, C719, C720, C721, C722, C723, C724, C725, C726, C727, C728, C729, C730, C735, C736, C738, C740, C741, C742, C744, C746, C751, C752, C753, C754, C755, C756, C757, C758, C759, C760, C761, C762: renamed from C?; footprint (none) -> OHDSP-Footprints-Pretty:CAP_TH_5mm
- C703, C705, C709, C711, C713, C715, C716, C717, C718, C731, C732, C737, C739, C743, C745, C747, C748, C749, C750, C763, C764, C765, C766, C767, C768, C769, C770: renamed from C?; footprint OHDSP-Footprints-Pretty:CAP-TH-D6.3mmP2.5mm -> OHDSP-Footprints-Pretty:CAP-TH-D10mmP5mm
- C710: renamed from C?; footprint OHDSP-Footprints-Pretty:SMD-0805 -> OHDSP-Footprints-Pretty:CAP_TH_5mm
- P701, P702, P703, P704: renamed from P?; footprint (none) -> OHDSP-Footprints-Pretty:CONN_SIL_3
- R701, R702, R703, R704, R705, R706, R707, R708, R709, R710, R711, R712, R713, R714, R715, R716, R717, R718, R719, R720, R721, R722, R723, R724, R725, R726, R727, R728, R729, R730, R731, R732, R733, R734, R735, R736, R737, R738, R739, R740, R741, R742, R743, R744, R745, R746, R747, R748, R749, R750, R751, R752, R753, R754, R755, R756, R757, R758: renamed from R?; footprint (none) -> OHDSP-Footprints-Pretty:TH-RES-0W25
- U701, U702, U703, U704, U705: renamed from U?; footprint (none) -> OHDSP-Footprints-Pretty:IC_DIP_8
- gave numbers to parts that had none: 10
Connections:
- net at C723.1, R722.2, R727.1: now also U702.1; no longer U702.7
- net at C723.2, R714.2, R722.1: now also U702.2 (-); no longer U702.6 (-)
- net at C715.1, C719.2, R713.2: now also U702.3 (+); no longer U702.5 (+)
- net at C726.1, R715.2, R725.2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: now also U703.7; no longer U703.1
- net at C726.2, R721.2, R725.1: now also U703.6 (-); no longer U703.2 (-)
- net at C718.1, C722.2, R720.2: now also U703.5 (+); no longer U703.3 (+)
- net at C724.1, R723.2, R728.1: now also U702.7; no longer U702.1
- net at C724.2, R717.2, R723.1: now also U702.6 (-); no longer U702.2 (-)
- net at C716.1, C720.2, R716.2: now also U702.5 (+); no longer U702.3 (+)
- net at C758.1, R744.2, R754.2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: now also U705.7; no longer U705.1
- net at C758.2, R750.2, R754.1: now also U705.6 (-); no longer U705.2 (-)
- net at C750.1, C754.2, R749.2: now also U705.5 (+); no longer U705.3 (+)
- net at C756.1, R752.2, R756.1: now also U704.7; no longer U704.1
- net at C756.2, R746.2, R752.1: now also U704.6 (-); no longer U704.2 (-)
- net at C748.1, C752.2, R745.2: now also U704.5 (+); no longer U704.3 (+)
