File: Schematics/AD1937_DigiOut_1To4.sch (KiCad schematic (older format))
At the start: 252 parts

Commit message: WIP
Parts:
- removed C? (x11): 1n, symbol C
- removed C? (x24): 100u, OHDSP-Footprints-Pretty:CAP-TH-D6.3mmP2.5mm, symbol CP1
- removed C? (x10): 100n, symbol C
- removed C? (x5): N/F, symbol C
- removed C?: 100p, symbol C
- removed C? (x14): 100n, OHDSP-Footprints-Pretty:SMD-0805, symbol C
- removed P? (x3): CONN_3x1, symbol CONN_3x1
- removed P?: CONN_2x1, symbol CONN_2x1
- removed R? (x29): 10k, symbol R
- removed R? (x10): 100R, symbol R
- removed R? (x4): 3k6, symbol R
- removed U? (x9): IC-OPAMP-DUAL-SOIC8, symbol IC-OPAMP-DUAL-SOIC8
- added C803, C807, C811, C821, C826, C829, C853, C855, C861, C863, C871, C872, C874, C881, C882, C901, C902, C903, C904, C917, C919, C923, C925, C927: 100u, OHDSP-Footprints-Pretty:CAP-TH-D10mmP5mm, symbol CP1
- added C806, C856, C864, C868, C873, C918, C920, C922, C924, C928: 100n, OHDSP-Footprints-Pretty:CAP_TH_5mm, symbol C
- added C816, C833, C834, C835, C836, C844, C878, C879, C880, C885, C886, C887, C888, C906: 100n, OHDSP-Footprints-Pretty:SMD-0805, symbol C
- added C817, C819, C820, C823, C889, C890, C891, C893, C895, C897, C899: 1n, OHDSP-Footprints-Pretty:CAP_TH_5mm, symbol C
- added C910: 100p, OHDSP-Footprints-Pretty:CAP_TH_5mm, symbol C
- added C912, C913, C914, C915, C916: N/F, OHDSP-Footprints-Pretty:CAP_TH_5mm, symbol C
- added P801, P805, P807: CONN_3x1, OHDSP-Footprints-Pretty:CONN_SIL_3, symbol CONN_3x1
- added P806: CONN_2x1, OHDSP-Footprints-Pretty:CONN_SIL_2, symbol CONN_2x1
- added R802, R849, R854, R855: 3k6, OHDSP-Footprints-Pretty:TH-RES-0W25, symbol R
- added R811, R837, R838, R839, R841, R857, R860, R885, R886, R889: 100R, OHDSP-Footprints-Pretty:TH-RES-0W25, symbol R
- added R818, R819, R820, R822, R823, R825, R827, R829, R830, R831, R832, R835, R836, R844, R848, R861, R863, R868, R871, R872, R873, R875, R879, R882, R883, R884, R892, R894, R896: 10k, OHDSP-Footprints-Pretty:TH-RES-0W25, symbol R
- added U801, U808: IC-OPAMP-DUAL-SOIC8, OHDSP-Footprints-Pretty:IC_DIP_8, symbol IC-OPAMP-DUAL-SOIC8
- added unit 2 of U802
- added unit 1 of U803
- added unit 1 of U807
- added unit 2 of U809
- added unit 2 of U810
- C801, C805, C809, C810, C812, C830, C837, C838, C839, C840, C857, C859, C865, C866, C867, C869, C876, C883, C884, C921: renamed from C?; footprint OHDSP-Footprints-Pretty:CAP-TH-D6.3mmP2.5mm -> OHDSP-Footprints-Pretty:CAP-TH-D10mmP5mm
- C802, C804, C808, C818, C822, C824, C825, C827, C828, C831, C832, C845, C846, C847, C848, C849, C850, C851, C852, C854, C858, C860, C862, C870, C875, C892, C894, C896, C898, C900, C909, C911, C926: renamed from C?; footprint (none) -> OHDSP-Footprints-Pretty:CAP_TH_5mm
- P802, P804, P808: renamed from P?; footprint (none) -> OHDSP-Footprints-Pretty:CONN_SIL_2
- P803: renamed from P?; footprint (none) -> OHDSP-Footprints-Pretty:CONN_SIL_3
- R801, R803, R804, R805, R806, R807, R808, R809, R810, R812, R813, R814, R815, R816, R817, R821, R824, R826, R828, R833, R834, R840, R842, R843, R845, R846, R847, R850, R851, R852, R853, R856, R858, R859, R862, R864, R865, R866, R867, R869, R870, R874, R876, R877, R878, R880, R881, R887, R888, R890, R891, R893, R895: renamed from R?; footprint (none) -> OHDSP-Footprints-Pretty:TH-RES-0W25
- U802, U803, U804, U805, U806, U807, U809, U810, U811, U812: renamed from U?; footprint (none) -> OHDSP-Footprints-Pretty:IC_DIP_8
- gave numbers to parts that had none: 10
Connections:
- net +12VA: now also C811.1, C816.2, C829.1, C835.2, C836.2, C844.2, C878.2, C880.2, C882.1, C886.2, C888.2, C902.1, C904.1, C906.2, U801.8, U801.8, U802.8, U803.8, U807.8, U808.8, U808.8, U809.8, U810.8
- net -12VA: now also C821.2, C826.2, C833.1, C834.1, C871.2, C879.1, C881.2, C885.1, C887.1, C901.2, C903.2, U801.4, U801.4, U802.4, U803.4, U807.4, U808.4, U808.4, U809.4, U810.4
- net DIGIOUT_1N: now also C803.2
- net DIGIOUT_2P: now also C868.2
- net DIGIOUT_3N: now also C807.2
- net DIGIOUT_3P: now also C806.2
- net DIGIOUT_4N: now also C874.2
- net DIGIOUT_4P: now also C872.2, C873.2
- net GNDD: now also C811.2, C816.1, C821.1, C826.1, C829.2, C833.2, C834.2, C835.1, C836.1, C844.1, C871.1, C878.1, C879.2, C880.1, C881.1, C882.2, C885.2, C886.1, C887.2, C888.1, C897.1, C899.1, C901.1, C902.2, C903.1, C904.2, C906.1, P801.3 (P3), P805.3 (P3), P806.2 (P2), P807.3 (P3), R818.2, R819.2, R820.2, R822.2, R823.2, R827.2, R844.2, R848.2, R868.2, R871.2, R875.2, R892.2, R894.2, R896.2
- net at C818.1, R810.1: now also C817.1, U801.1, U801.2 (-)
- net at C827.2, R805.2: now also U801.3 (+)
- net at C854.1, R843.1: now also C853.1, P801.2 (P2)
- net at C818.2, R801.2, R805.1: now also C817.2
- net at C848.2: now also U803.7, R832.2, R838.1; no longer U803.1
- net at C848.1: now also U803.6 (-), R822.1, R832.1; no longer U803.2 (-)
- net at R810.2, R813.1: now also U803.5 (+), R818.1; no longer U803.3 (+)
- net at R809.1: now also C819.1, C820.1, U801.6 (-), U801.7
- net at C828.2, R806.2: now also U801.5 (+)
- net at C804.1: now also C803.1, R802.1
- net at R806.1: now also C819.2, C820.2, R802.2
- net at C847.2: now also R831.2, R837.1, U803.1
- net at C847.1, R821.1: now also R831.1, U803.2 (-)
- net at R809.2, R814.2, R817.1: now also U803.3 (+)
- net at C854.2: now also C853.2, R837.2
- net at C851.1, U805.2 (-): now also R825.1, R835.1
- net at R824.1, U805.3 (+): now also R823.1
- net at C851.2, U805.6: now also R835.2, R841.1
- net at C845.1, R814.1: now also R825.2
- net at C862.2: now also C861.2, R841.2
- net at C862.1, P802.1 (P1), R847.1: now also C861.1
- net at R858.1: now also C889.1, C890.1, U807.1, U807.2 (-)
- net at R853.2: now also C897.2, U807.3 (+)
- net at C867.1: now also C868.1, R849.1
- net at R891.1: now also C917.1, C918.1, P805.2 (P2)
- net at R853.1: now also C889.2, C890.2, R849.2
- net at R880.2: now also C912.2, R886.1, U809.7
- net at R870.1, R880.1: now also C912.1, U809.6 (-)
- net at R858.2, R866.1: now also R861.1, U809.5 (+)
- net at C898.2: now also U807.5 (+), R854.2; no longer U807.3 (+)
- net at C892.2, R850.2: now also C891.2, R854.1
- net at C911.2, U809.1: now also R879.2, R885.1
- net at C911.1, R869.1, U809.2 (-): now also R879.1
- net at R862.2, R865.1, U809.3 (+): now also R857.2
- net at U811.2 (-): now also C915.1, R873.1, R883.1
- net at U811.3 (+): now also R871.1, R872.1
- net at U811.6: now also C915.2, R883.2, R889.1
- net at C909.2: now also R861.2, R872.2
- net at C909.1, R862.1: now also R873.2
- net at C926.2: now also C925.2, R889.2
- net at C926.1, R895.1: now also C925.1, P806.1 (P1)
- net at C822.1, R812.1, U802.1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: now also C823.1
- net at C805.1, R803.1: now also C806.1
- net at C822.2, R803.2, R807.1: now also C823.2
- net at C850.2, R834.2, R840.1: now also U804.7; no longer U804.1
- net at C850.1, R834.1: now also U804.6 (-), R827.1; no longer U804.2 (-)
- net at R812.2, R815.1: now also U804.5 (+), R820.1; no longer U804.3 (+)
- net at C824.1, C825.1: now also R811.1, U802.6 (-), U802.7
- net at C832.2, R808.2: now also U802.5 (+)
- net at C808.1, R804.1: now also C807.1
- net at C849.2, R833.2, U804.1: now also R839.1
- net at R816.2, U804.3 (+): now also R811.2, R819.1
- net at C857.2, C858.2: now also R839.2
- net at C852.1, U806.2 (-): now also R830.1, R836.1
- net at R828.1, U806.3 (+): now also R829.1
- net at C852.2, R842.1, U806.6: now also R836.2
- net at C846.2, R815.2: now also R829.2
- net at C846.1, R816.1: now also R830.2
- net at R842.2: now also C863.2, C864.2
- net at P804.1 (P1): now also C863.1, C864.1, R848.1
- net at C894.1: now also C893.1, R860.1, U808.1, U808.2 (-)
- net at R851.1: now also C872.1, C873.1
- net at C921.1, R893.1: now also C922.1, P807.2 (P2)
- net at C894.2, R851.2: now also C893.2, R855.1
- net at R888.1: now also C914.2, R882.2, U810.7
- net at R888.2: now also C923.2, C924.2
- net at C896.1, R859.1: now also C895.1, U808.6 (-), U808.7
- net at C900.2, R856.2: now also U808.5 (+)
- net at C875.1, R852.1: now also C874.1
- net at C896.2, R852.2, R856.1: now also C895.2
- net at R881.2, R887.1, U810.1: now also C913.2
- net at R874.1, R881.1, U810.2 (-): now also C913.1
- net at C921.2, R887.2: now also C922.2
- net at R878.1, U812.2 (-): now also C916.1, R884.1
- net at R890.1, U812.6: now also C916.2, R884.2
- net at R877.2: now also C910.2, R863.2
- net at R864.1, R878.2: now also C910.1
- net at R890.2: now also C927.2, C928.2
- net at P808.1 (P1): now also C927.1, C928.1, R896.1
- new net: C855.1, C856.1, P801.1 (P1), R844.1
- new net: C855.2, C856.2, R838.2
- new net: C919.1, C920.1, P805.1 (P1), R892.1
- new net: C919.2, C920.2, R886.2
- new net: C891.1, C892.1, R857.1, U807.6 (-), U807.7
- new net: C917.2, C918.2, R885.2
- new net: C899.2, R855.2, U808.3 (+)
- new net: C923.1, C924.1, P807.1 (P1), R894.1
- new net: R860.2, R863.1, R868.1, U810.5 (+)
- new net: C914.1, R875.1, R882.1, U810.6 (-)
