File: Schematics/AD1937_DigiOut_5To8.sch (KiCad schematic (older format))
At the start: 252 parts

Commit message: WIP
Connections:
- net DIGIOUT_1N renamed DIGIOUT_5N
- net DIGIOUT_1P renamed DIGIOUT_5P
- net DIGIOUT_2N renamed DIGIOUT_6N
- net DIGIOUT_2P renamed DIGIOUT_6P
- net DIGIOUT_3N renamed DIGIOUT_7N
- net DIGIOUT_3P renamed DIGIOUT_7P
- net DIGIOUT_4N renamed DIGIOUT_8N
- net DIGIOUT_4P renamed DIGIOUT_8P
Changed lines of the file:
@@
 $Descr A2 23386 16535
 encoding utf-8
-Sheet 9 10
+Sheet 10 10
 Title ""
 Date ""
@@
 Connection ~ 6500 3600
 Text HLabel 2200 1900 0    60   Input ~ 0
-DIGIOUT_1P
+DIGIOUT_5P
 Text HLabel 2200 3950 0    60   Input ~ 0
-DIGIOUT_1N
+DIGIOUT_5N
 $Comp
 L C C?
@@
 Connection ~ 16300 3700
 Text HLabel 12000 2000 0    60   Input ~ 0
-DIGIOUT_2P
+DIGIOUT_6P
 Text HLabel 12000 4050 0    60   Input ~ 0
-DIGIOUT_2N
+DIGIOUT_6N
 $Comp
 L C C?
@@
 Connection ~ 6550 9650
 Text HLabel 2250 7950 0    60   Input ~ 0
-DIGIOUT_3P
+DIGIOUT_7P
 Text HLabel 2250 10000 0    60   Input ~ 0
-DIGIOUT_3N
+DIGIOUT_7N
 $Comp
 L C C?
@@
 Connection ~ 16350 9750
 Text HLabel 12050 8050 0    60   Input ~ 0
-DIGIOUT_4P
+DIGIOUT_8P
 Text HLabel 12050 10100 0    60   Input ~ 0
-DIGIOUT_4N
+DIGIOUT_8N
 $Comp
 L C C?

Commit message: WIP
Parts:
- removed C? (x20): 100u, OHDSP-Footprints-Pretty:CAP-TH-D6.3mmP2.5mm, symbol CP1
- removed C? (x10): 100n, symbol C
- removed C? (x13): 1n, symbol C
- removed C? (x3): 100p, symbol C
- removed C? (x7): N/F, symbol C
- removed C? (x10): 100n, OHDSP-Footprints-Pretty:SMD-0805, symbol C
- removed P? (x3): CONN_2x1, symbol CONN_2x1
- removed P?: CONN_3x1, symbol CONN_3x1
- removed R? (x12): 3k6, symbol R
- removed R? (x10): 100R, symbol R
- removed R? (x31): 10k, symbol R
- removed U? (x7): IC-OPAMP-DUAL-SOIC8, symbol IC-OPAMP-DUAL-SOIC8
- removed U? (x4): IC-OPAMP-SINGLE-SOIC8, symbol IC-OPAMP-SINGLE-SOIC8
- added C1003, C1054, C930, C932, C936, C982, C986, C988, C990, C998: 100n, OHDSP-Footprints-Pretty:CAP_TH_5mm, symbol C
- added C1004, C1011, C1012, C1049, C929, C933, C937, C938, C940, C958, C965, C966, C967, C968, C985, C987, C993, C994, C995, C997: 100u, OHDSP-Footprints-Pretty:CAP-TH-D10mmP5mm, symbol CP1
- added C1005: 100n, OHDSP-Footprints-Pretty:CAP-TH-D10mmP5mm, symbol C
- added C1020, C1022, C1024, C1026, C1028, C946, C950, C952, C953, C955, C956, C959, C960: 1n, OHDSP-Footprints-Pretty:CAP_TH_5mm, symbol C
- added C1033, C1035, C1036, C941, C942, C943, C969, C970, C971: 100n, OHDSP-Footprints-Pretty:SMD-0805, symbol C
- added C1037, C973, C974: 100p, OHDSP-Footprints-Pretty:CAP_TH_5mm, symbol C
- added C1039, C975, C976, C977, C978, C979, C980: N/F, OHDSP-Footprints-Pretty:CAP_TH_5mm, symbol C
- added P902, P904, P908: CONN_2x1, OHDSP-Footprints-Pretty:CONN_SIL_2, symbol CONN_2x1
- added P903: CONN_3x1, OHDSP-Footprints-Pretty:CONN_SIL_3, symbol CONN_3x1
- added R901, R903, R904, R905, R906, R907, R908, R950, R951, R952, R953, R956: 3k6, OHDSP-Footprints-Pretty:TH-RES-0W25, symbol R
- added R909, R910, R912, R940, R942, R958, R959, R987, R988, R990: 100R, OHDSP-Footprints-Pretty:TH-RES-0W25, symbol R
- added R913, R914, R915, R916, R917, R921, R924, R926, R928, R933, R934, R943, R945, R946, R947, R962, R964, R965, R966, R967, R969, R970, R974, R976, R977, R978, R980, R981, R991, R993, R995: 10k, OHDSP-Footprints-Pretty:TH-RES-0W25, symbol R
- added unit 1 of U902
- added unit 2 of U903
- added U904: IC-OPAMP-DUAL-SOIC8, OHDSP-Footprints-Pretty:IC_DIP_8, symbol IC-OPAMP-DUAL-SOIC8
- added U905, U906, U911, U912: IC-OPAMP-SINGLE-SOIC8, OHDSP-Footprints-Pretty:IC_DIP_8, symbol IC-OPAMP-SINGLE-SOIC8
- added unit 2 of U907
- added unit 1 of U909
- added unit 1 of U910
- C1000, C1002, C1009, C1010, C1029, C1030, C1031, C1032, C1045, C1047, C1051, C1053, C1055, C931, C935, C939, C949, C954, C957, C981, C983, C989, C991, C999: renamed from C?; footprint OHDSP-Footprints-Pretty:CAP-TH-D6.3mmP2.5mm -> OHDSP-Footprints-Pretty:CAP-TH-D10mmP5mm
- C1001, C1017, C1018, C1019, C1021, C1023, C1025, C1027, C1038, C1040, C1041, C1042, C1043, C1044, C1046, C1048, C1050, C1052, C1056, C934, C945, C947, C948, C951, C984, C992, C996: renamed from C?; footprint (none) -> OHDSP-Footprints-Pretty:CAP_TH_5mm
- P901, P905, P907: renamed from P?; footprint (none) -> OHDSP-Footprints-Pretty:CONN_SIL_3
- P906: renamed from P?; footprint (none) -> OHDSP-Footprints-Pretty:CONN_SIL_2
- R902, R911, R918, R919, R920, R922, R923, R925, R927, R929, R930, R931, R932, R935, R936, R937, R938, R939, R941, R944, R948, R949, R954, R955, R957, R960, R961, R963, R968, R971, R972, R973, R975, R979, R982, R983, R984, R985, R986, R989, R992, R994, R996: renamed from R?; footprint (none) -> OHDSP-Footprints-Pretty:TH-RES-0W25
- U901, U902, U903, U907, U908, U909, U910: renamed from U?; footprint (none) -> OHDSP-Footprints-Pretty:IC_DIP_8
- gave numbers to parts that had none: 14
Connections:
- net +12VA: now also C1004.1, C1012.1, C1036.2, C940.1, C943.2, C958.1, C967.1, C968.1, C971.2, C994.1, U902.8, U903.8, U904.8, U904.8, U905.7, U906.7, U907.8, U909.8, U910.8, U911.7, U912.7
- net -12VA: now also C1005.1, C1011.2, C1033.1, C1035.1, C937.2, C938.2, C941.1, C942.1, C965.2, C966.2, C969.1, C970.1, C993.2, U902.4, U903.4, U904.4, U904.4, U905.4, U906.4, U907.4, U909.4, U910.4, U911.4, U912.4
- net DIGIOUT_5N: now also C932.2
- net DIGIOUT_5P: now also C929.2, C930.2
- net DIGIOUT_6N: now also C997.2, C998.2
- net DIGIOUT_6P: now also C995.2
- net DIGIOUT_7N: now also C936.2
- net DIGIOUT_7P: now also C933.2
- net DIGIOUT_8N: now also C1003.2
- net GNDD: now also C1004.2, C1005.2, C1011.1, C1012.2, C1026.1, C1028.1, C1033.2, C1035.2, C1036.1, C937.1, C938.1, C940.2, C941.2, C942.2, C943.1, C955.1, C956.1, C958.2, C959.1, C960.1, C965.1, C966.1, C967.2, C968.2, C969.2, C970.2, C971.1, C993.1, C994.2, P902.2 (P2), P903.3 (P3), P904.2 (P2), P908.2 (P2), R917.2, R921.2, R926.2, R928.2, R943.2, R945.2, R946.2, R947.2, R965.2, R966.2, R967.2, R969.2, R970.2, R974.2, R976.2, R991.2, R993.2, R995.2
- net at C945.1, U901.1, U901.2 (-): now also C946.1, R910.1
- net at U901.3 (+): now also C955.2, R905.2
- net at C981.1, P901.2 (P2): now also C982.1, R943.1
- net at C945.2: now also C946.2, R901.2, R905.1
- net at R932.2, R938.1: now also C976.2, U903.7
- net at R922.1, R932.1: now also C976.1, U903.6 (-)
- net at R918.1: now also R910.2, R913.1, U903.5 (+)
- net at C947.1, C948.1: now also U901.6 (-), U901.7, R909.1; no longer U901.1, U901.2 (-)
- net at C931.1, R902.1: now also C932.1
- net at C947.2, C948.2, R902.2: now also R906.1
- net at R931.2, R937.1, U903.1: now also C975.2
- net at R931.1, U903.2 (-): now also C975.1, R921.1
- net at U903.3 (+): now also R909.2, R914.2, R917.1
- net at C981.2, R937.2: now also C982.2
- net at R925.1, R935.1: now also C979.1, U905.2 (-)
- net at R923.1: now also R924.1, U905.3 (+)
- net at R935.2, R941.1: now also C979.2, U905.6
- net at R925.2: now also C973.1, R914.1
- net at C989.2, R941.2: now also C990.2
- net at C989.1: now also C990.1, P902.1 (P1), R947.1
- net at C1017.1, C1018.1, U907.1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: now also R958.1
- net at C1025.2, U907.3 (+): now also R953.2
- net at C996.1, R949.1: now also C995.1
- net at C1045.1, C1046.1, P905.2 (P2): now also R991.1
- net at C1017.2, C1018.2, R949.2: now also R953.1
- net at C1040.2, R986.1: now also U909.7, R980.2; no longer U909.1
- net at C1040.1: now also U909.6 (-), R970.1, R980.1; no longer U909.2 (-)
- net at R961.1: now also U909.5 (+), R958.2, R966.1; no longer U909.3 (+)
- net at C1019.1, R957.1: now also C1020.1, U907.6 (-), U907.7
- net at R954.2: now also C1026.2, U907.5 (+)
- net at C1019.2, R954.1: now also C1020.2, R950.2
- net at R979.2, R985.1: now also C1039.2, U909.1
- net at R979.1: now also C1039.1, R969.1, U909.2 (-)
- net at R957.2: now also R962.2, R965.1, U909.3 (+)
- net at C1043.1, R973.1, R983.1: now also U911.2 (-)
- net at R971.1, R972.1: now also U911.3 (+)
- net at C1043.2, R983.2, R989.1: now also U911.6
- net at R961.2, R972.2: now also C1037.2
- net at R973.2: now also C1037.1, R962.1
- net at C1053.2, R989.2: now also C1054.2
- net at C1053.1, P906.1 (P1): now also C1054.1, R995.1
- net at C951.1: now also C950.1, R912.1, U902.1, U902.2 (-)
- net at C934.1: now also C933.1, R903.1
- net at C951.2: now also C950.2, R903.2, R907.1
- net at R927.1: now also C978.1, R934.1, U904.6 (-)
- net at R920.1: now also R912.2, R915.1, U904.5 (+)
- net at C935.1: now also C936.1, R904.1
- net at R939.1: now also C977.2, R933.2, U904.1
- net at R911.2, R919.1: now also R916.2, U904.3 (+)
- net at R939.2: now also C985.2, C986.2
- net at R930.1, R936.1: now also C980.1, U906.2 (-)
- net at R929.1: now also R928.1, U906.3 (+)
- net at R936.2: now also C980.2, R942.1, U906.6
- net at R929.2: now also C974.2, R915.2
- net at R930.2: now also C974.1, R916.1
- net at C991.2, C992.2: now also R942.2
- net at C991.1, C992.1, R948.1: now also P904.1 (P1)
- net at C1021.1, R960.1, U908.1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: now also C1022.1
- net at C1000.1, C1001.1: now also R951.1
- net at C1050.1, P907.2 (P2): now also C1049.1, R993.1
- net at C1021.2, R955.1: now also C1022.2, R951.2
- net at C1042.2, R982.2: now also U910.7, R988.1; no longer U910.1
- net at C1042.1, R975.1, R982.1: now also U910.6 (-); no longer U910.2 (-)
- net at R960.2, R963.1, R968.1: now also U910.5 (+); no longer U910.3 (+)
- net at C1051.2, C1052.2: now also R988.2
- net at C1002.1: now also C1003.1, R952.1
- net at C1023.2: now also C1024.2, R952.2, R956.1
- net at C1041.2: now also R981.2, R987.1, U910.1
- net at C1041.1: now also R974.1, R981.1, U910.2 (-)
- net at C1050.2: now also C1049.2, R987.2
- net at C1044.1, R984.1: now also R978.1, U912.2 (-)
- net at C1044.2, R984.2: now also R990.1, U912.6
- net at C1038.2, R963.2: now also R977.2
- net at C1038.1: now also R964.1, R978.2
- net at C1055.2, C1056.2: now also R990.2
- net at C1055.1, C1056.1, R996.1: now also P908.1 (P1)
- new net: C956.2, R906.2, U901.5 (+)
- new net: C929.1, C930.1, R901.1
- new net: C973.2, R913.2, R924.2
- new net: C997.1, C998.1, R950.1
- new net: C959.2, R907.2, U902.3 (+)
- new net: C987.1, C988.1, P903.1 (P1), R946.1
- new net: C985.1, C986.1, P903.2 (P2), R945.1
- new net: C978.2, R934.2, R940.1, U904.7
- new net: C987.2, C988.2, R940.2
- new net: C952.2, C953.2, R904.2, R908.1
- new net: C952.1, C953.1, R911.1, U902.6 (-), U902.7
- new net: C960.2, R908.2, U902.5 (+)
- new net: C977.1, R926.1, R933.1, U904.2 (-)
- new net: C1023.1, C1024.1, R959.1, U908.6 (-), U908.7
- new net: C1028.2, R956.2, U908.5 (+)
- new net: R959.2, R964.2, R967.1, U910.3 (+)
- new net: R976.1, R977.1, U912.3 (+)
