File: Schematics/OHDSP-XOVER.kicad_pcb (KiCad board)
At the start: 4 copper layers, 100 x 100 mm, 265 parts, among them CN401 COAX, CN402 COAX, P201 CONN_2x1, P301 PIN, P302 PIN, P303 PIN, P305 CONN_2x1, P306 PIN, P501 CONN_02X10, P502 CONN_02X05, P503 CONN_02X05, P504 CONN_02X05, P505 CONN_02X10, P506 CONN_2x1, P507 CONN_2x1, P508 CONN_02X20, P509 CONN_02X05, P510 CONN_02X05, P511 CONN_02X05, P512 CONN_2x1, P513 CONN_2x1, P514 CONN_2x1, P515 CONN_2x1, SW201 SWITCH, U201 IC-RST-ADM811, U202 ADAU1701JSTZ, U203 IC-EEPROM-I2C, U301 LT1374CS8-5#PBF, U302 NCP700BSN33T1G, U303 NCP700BSN33T1G, U304 NCP700BSN18T1G, U403 NB3L553

Commit message: WIP
Parts:
- removed C246, C247, C249, C307, C314, C315, C316, C320, C321, C322, C323, C324, C325: 100n, OHDSP-Footprints-Pretty:SMD-0805
- removed C248: 1u, OHDSP-Footprints-Pretty:SMD-0805
- removed C250, R419, R516, R517, R518, R520, R529, R530, R531, R532, R533, R534, R535, R536, R543: N/F, OHDSP-Footprints-Pretty:SMD-0805
- removed C308: 35ZL470MEFC10X20, OHDSP-Footprints-Pretty:CAP-TH-D10mmP5mm
- removed C309: 1n5, OHDSP-Footprints-Pretty:SMD-0805
- removed C310: 10ZL470MEFC8X11.5, OHDSP-Footprints-Pretty:CAP-TH-D8mmP3.5mm
- removed C311, C312, C313, C329, C330, C331: 220u, OHDSP-Footprints-Pretty:CAP-TH-D6.3mmP2.5mm
- removed C317, C318, C319: 10n, OHDSP-Footprints-Pretty:SMD-0805
- removed C326, C327, C328: 22u, OHDSP-Footprints-Pretty:SMD-0805
- removed CN401, CN402: COAX, OHDSP-Footprints-Pretty:CONN-RF-UFL
- removed D301: 1N914, OHDSP-Footprints-Pretty:DIODE-DO-35
- removed D302, D303: MBRS330T3, OHDSP-Footprints-Pretty:DIODE-SMC
- removed D304, D305, D306: LED, OHDSP-Footprints-Pretty:SMD-0805
- removed D501, D502, D503, D504: 1N5818, OHDSP-Footprints-Pretty:DIODE-DO-41
- removed P301, P302, P303, P306: PIN, OHDSP-Footprints-Pretty:MNT_HOLE_2.5mm
- removed P305, P512, P513, P514, P515: CONN_2x1, OHDSP-Footprints-Pretty:CONN_SIL_2
- removed P508: CONN_02X20, OHDSP-Footprints-Pretty:CONN_DIL_2X20
- removed P509, P510, P511: CONN_02X05, OHDSP-Footprints-Pretty:CONN_DIL_2X5
- removed R241, R242, R243, R528, R539, R540, R542, R544, R545, R546: 0R, OHDSP-Footprints-Pretty:SMD-0805
- removed R519, R541, R559: 1k, OHDSP-Footprints-Pretty:SMD-0805
- removed R521, R522, R523, R524, R525, R526, R527: 27R, OHDSP-Footprints-Pretty:SMD-0805
- removed R537, R538: 18k, OHDSP-Footprints-Pretty:SMD-1206
- removed R547, R548, R549, R550: 560R, OHDSP-Footprints-Pretty:SMD-1206
- removed R551, R552, R553, R554, R555, R556, R560, R561: 0R, OHDSP-Footprints-Pretty:SMD-1206
- removed R557, R558: 47R, OHDSP-Footprints-Pretty:SMD-0805
- removed U302, U303: NCP700BSN33T1G, OHDSP-Footprints-Pretty:IC-SOT23-5
- removed U304: NCP700BSN18T1G, OHDSP-Footprints-Pretty:IC-SOT23-5
- removed XTAL401: XTAL-OSC-4PIN, OHDSP-Footprints-Pretty:XTAL_8_DIL
- added C1000: 100u, OHDSP-Footprints-Pretty:CAP-TH-D10mmP5mm, F.Cu at (422.2, 177.6)
- added C1001: 100n, OHDSP-Footprints-Pretty:CAP_TH_5mm, F.Cu at (487.7, 124.3)
- added C1002: 100u, OHDSP-Footprints-Pretty:CAP-TH-D10mmP5mm, F.Cu at (464.3, 138.3)
- added C1003: 100n, OHDSP-Footprints-Pretty:CAP_TH_5mm, F.Cu at (466.0, 149.4)
- added C1004: 100u, OHDSP-Footprints-Pretty:CAP-TH-D10mmP5mm, F.Cu at (522.1, 82.1)
- added C1005: 100n, OHDSP-Footprints-Pretty:CAP-TH-D10mmP5mm, F.Cu at (434.4, 164.9)
- added C1006: 100n, OHDSP-Footprints-Pretty:SMD-0805, F.Cu at (525.4, 108.5)
- added C1007: 100n, OHDSP-Footprints-Pretty:SMD-0805, F.Cu at (526.9, 102.1)
- added C1008: 100n, OHDSP-Footprints-Pretty:SMD-0805, F.Cu at (409.6, 158.5)
- added C1009: 100u, OHDSP-Footprints-Pretty:CAP-TH-D10mmP5mm, F.Cu at (389.1, 164.5)
- added C1010: 100u, OHDSP-Footprints-Pretty:CAP-TH-D10mmP5mm, F.Cu at (460.6, 92.7)
- added C1011: 100u, OHDSP-Footprints-Pretty:CAP-TH-D10mmP5mm, F.Cu at (358.1, 184.5)
- added C1012: 100u, OHDSP-Footprints-Pretty:CAP-TH-D10mmP5mm, F.Cu at (385.8, 177.3)
- added C1013: 100n, OHDSP-Footprints-Pretty:SMD-0805, F.Cu at (527.3, 96.3)
- added C1014: 100n, OHDSP-Footprints-Pretty:SMD-0805, F.Cu at (527.3, 90.6)
- added C1015: 100n, OHDSP-Footprints-Pretty:SMD-0805, F.Cu at (472.6, 108.6)
- added C1016: 100n, OHDSP-Footprints-Pretty:SMD-0805, F.Cu at (409.6, 164.2)
- added C1017: 1n, OHDSP-Footprints-Pretty:CAP_TH_5mm, F.Cu at (430.6, 194.0)
- added C1018: 1n, OHDSP-Footprints-Pretty:CAP_TH_5mm, F.Cu at (487.7, 133.3)
- added C1019: 1n, OHDSP-Footprints-Pretty:CAP_TH_5mm, F.Cu at (420.8, 197.7)
- added C1020: 1n, OHDSP-Footprints-Pretty:CAP_TH_5mm, F.Cu at (433.0, 185.0)
- added C1021: 1n, OHDSP-Footprints-Pretty:CAP_TH_5mm, F.Cu at (499.8, 118.7)
- added C1022: 1n, OHDSP-Footprints-Pretty:CAP_TH_5mm, F.Cu at (445.1, 172.3)
- added C1023: 1n, OHDSP-Footprints-Pretty:CAP_TH_5mm, F.Cu at (520.0, 102.2)
- added C1024: 1n, OHDSP-Footprints-Pretty:CAP_TH_5mm, F.Cu at (466.0, 158.4)
- added C1025: 1n, OHDSP-Footprints-Pretty:CAP_TH_5mm, F.Cu at (497.4, 127.6)
- added C1026: 1n, OHDSP-Footprints-Pretty:CAP_TH_5mm, F.Cu at (475.8, 146.0)
- added C1027: 1n, OHDSP-Footprints-Pretty:CAP_TH_5mm, F.Cu at (454.9, 168.5)
- added C1028: 1n, OHDSP-Footprints-Pretty:CAP_TH_5mm, F.Cu at (442.8, 181.2)
- added C1029: 100u, OHDSP-Footprints-Pretty:CAP-TH-D10mmP5mm, F.Cu at (394.6, 190.0)
- added C1030: 100u, OHDSP-Footprints-Pretty:CAP-TH-D10mmP5mm, F.Cu at (410.1, 175.4)
- added C1031: 100u, OHDSP-Footprints-Pretty:CAP-TH-D10mmP5mm, F.Cu at (464.3, 125.5)
- added C1032: 100u, OHDSP-Footprints-Pretty:CAP-TH-D10mmP5mm, F.Cu at (452.2, 126.8)
- added C1033: 100n, OHDSP-Footprints-Pretty:SMD-0805, F.Cu at (449.0, 99.6)
- added C1034: 100n, OHDSP-Footprints-Pretty:SMD-0805, F.Cu at (449.0, 93.9)
- added C1035: 100n, OHDSP-Footprints-Pretty:SMD-0805, F.Cu at (460.9, 101.3)
- added C1036: 100n, OHDSP-Footprints-Pretty:SMD-0805, F.Cu at (455.0, 101.3)
- added C1037: 100p, OHDSP-Footprints-Pretty:CAP_TH_5mm, F.Cu at (520.0, 93.2)
- added C1038: 100p, OHDSP-Footprints-Pretty:CAP_TH_5mm, F.Cu at (456.2, 150.6)
- added C1039: N/F, OHDSP-Footprints-Pretty:CAP_TH_5mm, F.Cu at (509.2, 114.9)
- added C1040: N/F, OHDSP-Footprints-Pretty:CAP_TH_5mm, F.Cu at (485.1, 142.2)
- added C1041: N/F, OHDSP-Footprints-Pretty:CAP_TH_5mm, F.Cu at (518.5, 111.1)
- added C1042: N/F, OHDSP-Footprints-Pretty:CAP_TH_5mm, F.Cu at (509.2, 123.8)
- added C1043: N/F, OHDSP-Footprints-Pretty:CAP_TH_5mm, F.Cu at (466.0, 167.3)
- added C1044: N/F, OHDSP-Footprints-Pretty:CAP_TH_5mm, F.Cu at (475.8, 154.9)
- added C1045: 100u, OHDSP-Footprints-Pretty:CAP-TH-D10mmP5mm, F.Cu at (497.8, 82.1)
- added C1046: 100n, OHDSP-Footprints-Pretty:CAP_TH_5mm, F.Cu at (475.1, 137.0)
- added C1047: 100u, OHDSP-Footprints-Pretty:CAP-TH-D10mmP5mm, F.Cu at (436.7, 139.5)
- added C1048: 100n, OHDSP-Footprints-Pretty:CAP_TH_5mm, F.Cu at (507.9, 105.9)
- added C1049: 100u, OHDSP-Footprints-Pretty:CAP-TH-D10mmP5mm, F.Cu at (421.2, 152.2)
- added C1050: 100n, OHDSP-Footprints-Pretty:CAP_TH_5mm, F.Cu at (433.0, 176.1)
- added C1051: 100u, OHDSP-Footprints-Pretty:CAP-TH-D10mmP5mm, F.Cu at (397.9, 177.3)
- added C1052: 100n, OHDSP-Footprints-Pretty:CAP_TH_5mm, F.Cu at (445.1, 163.3)
- added C1053: 100u, OHDSP-Footprints-Pretty:CAP-TH-D10mmP5mm, F.Cu at (382.4, 190.0)
- added C1054: 100n, OHDSP-Footprints-Pretty:CAP_TH_5mm, F.Cu at (420.8, 188.8)
- added C1055: 100u, OHDSP-Footprints-Pretty:CAP-TH-D10mmP5mm, F.Cu at (510.0, 82.1)
- added C1056: 100n, OHDSP-Footprints-Pretty:CAP_TH_5mm, F.Cu at (456.2, 159.6)
- added C1057: 220u, OHDSP-Footprints-Pretty:CAP-TH-D6.3mmP2.5mm, F.Cu at (692.6, 272.7)
- added C1058: 22u, OHDSP-Footprints-Pretty:SMD-0805, F.Cu at (699.0, 276.0)
- added C1059: 100n, OHDSP-Footprints-Pretty:SMD-0805, F.Cu at (713.7, 259.6)
- added C1060: 1u, OHDSP-Footprints-Pretty:SMD-0805, F.Cu at (707.7, 266.4)
- added C1061: 100n, OHDSP-Footprints-Pretty:SMD-0805, F.Cu at (728.3, 248.1)
- added C1062: 1u, OHDSP-Footprints-Pretty:SMD-0805, F.Cu at (723.7, 253.8)
- added C1063: 100n, OHDSP-Footprints-Pretty:SMD-0805, F.Cu at (696.3, 281.8)
- added C1064: 220u, OHDSP-Footprints-Pretty:CAP-TH-D6.3mmP2.5mm, F.Cu at (701.3, 263.0)
- added C1065: 220u, OHDSP-Footprints-Pretty:CAP-TH-D6.3mmP2.5mm, F.Cu at (692.6, 263.0)
- added C1066: 22u, OHDSP-Footprints-Pretty:SMD-0805, F.Cu at (713.7, 265.3)
- added C1067: 22u, OHDSP-Footprints-Pretty:SMD-0805, F.Cu at (722.4, 248.1)
- added C1068: 100n, OHDSP-Footprints-Pretty:SMD-0805, F.Cu at (717.8, 253.8)
- added C1069: 100n, OHDSP-Footprints-Pretty:SMD-0805, F.Cu at (719.6, 259.6)
- added C1070: 1u, OHDSP-Footprints-Pretty:SMD-0805, F.Cu at (734.3, 248.1)
- added C1071: 100n, OHDSP-Footprints-Pretty:SMD-0805, F.Cu at (710.9, 272.1)
- added C1072: 1u, OHDSP-Footprints-Pretty:SMD-0805, F.Cu at (705.0, 277.8)
- added C1073: 100n, OHDSP-Footprints-Pretty:SMD-0805, F.Cu at (729.7, 253.8)
- added C1074: 22p, OHDSP-Footprints-Pretty:SMD-0805, F.Cu at (719.6, 265.3)
- added C1075: 22p, OHDSP-Footprints-Pretty:SMD-0805, F.Cu at (725.6, 259.6)
- added C1076: 1n, OHDSP-Footprints-Pretty:SMD-0805, F.Cu at (710.9, 277.8)
- added C1077: 1u, OHDSP-Footprints-Pretty:SMD-0805, F.Cu at (716.9, 271.1)
- added C1078: 10u, OHDSP-Footprints-Pretty:SMD-0805, F.Cu at (735.6, 253.8)
- added C1079: 100n, OHDSP-Footprints-Pretty:SMD-0805, F.Cu at (716.9, 276.8)
- added C1080: 100n, OHDSP-Footprints-Pretty:SMD-0805, F.Cu at (705.0, 272.1)
- added C204: 220u, OHDSP-Footprints-Pretty:CAP-TH-D6.3mmP2.5mm, F.Cu at (575.0, 310.4)
- added C219: 100n, OHDSP-Footprints-Pretty:SMD-0805, F.Cu at (592.7, 292.7)
- added C222: 22u, OHDSP-Footprints-Pretty:SMD-0805, F.Cu at (557.1, 321.1)
- added C225: 3n3, OHDSP-Footprints-Pretty:SMD-0805, F.Cu at (589.0, 328.5)
- added C234: 220u, OHDSP-Footprints-Pretty:CAP-TH-D6.3mmP2.5mm, F.Cu at (551.1, 325.5)
- added C401: 22u, OHDSP-Footprints-Pretty:SMD-0805, F.Cu at (776.3, 210.6)
- added C403: 1000u, OHDSP-Footprints-Pretty:CAP-TH-D12.5mmP5mm, F.Cu at (714.3, 184.2)
- added C409: 100p, OHDSP-Footprints-Pretty:SMD-0805, F.Cu at (773.4, 193.4)
- added C410: 220u, OHDSP-Footprints-Pretty:CAP-TH-D10mmP5mm, F.Cu at (707.2, 230.0)
- added C411: 220u, OHDSP-Footprints-Pretty:CAP-TH-D10mmP5mm, F.Cu at (756.9, 182.9)
- added C412: 220u, OHDSP-Footprints-Pretty:CAP-TH-D12.5mmP5mm, F.Cu at (711.7, 199.4)
- added C413: 10n, OHDSP-Footprints-Pretty:CAP_TH_5mm, F.Cu at (729.2, 231.9)
- added C414: 10n, OHDSP-Footprints-Pretty:SMD-0805, F.Cu at (735.6, 229.2)
- added C415: 10n, OHDSP-Footprints-Pretty:CAP_TH_5mm, F.Cu at (762.0, 194.1)
- added C416: 22u, OHDSP-Footprints-Pretty:SMD-0805, F.Cu at (768.4, 194.1)
- added C417: 100n, OHDSP-Footprints-Pretty:SMD-0805, F.Cu at (727.0, 238.2)
- added C418: 22u, OHDSP-Footprints-Pretty:SMD-0805, F.Cu at (771.3, 211.4)
- added C419: 220u, OHDSP-Footprints-Pretty:CAP-TH-D12.5mmP5mm, F.Cu at (697.3, 191.5)
- added C420: 220u, OHDSP-Footprints-Pretty:CAP-TH-D12.5mmP5mm, F.Cu at (678.6, 228.4)
- added C421: 220u, OHDSP-Footprints-Pretty:CAP-TH-D6.3mmP2.5mm, F.Cu at (719.2, 223.8)
- added C422: 10n, OHDSP-Footprints-Pretty:CAP_TH_5mm, F.Cu at (739.6, 222.2)
- added C423: 10n, OHDSP-Footprints-Pretty:CAP_TH_5mm, F.Cu at (748.8, 213.7)
- added C424: 100n, OHDSP-Footprints-Pretty:SMD-0805, F.Cu at (756.0, 217.6)
- added C425: 22u, OHDSP-Footprints-Pretty:SMD-0805, F.Cu at (709.9, 238.5)
- added C426: 22u, OHDSP-Footprints-Pretty:SMD-0805, F.Cu at (776.3, 199.2)
- added C427: 22u, OHDSP-Footprints-Pretty:SMD-0805, F.Cu at (745.6, 231.5)
- added C428: 22u, OHDSP-Footprints-Pretty:SMD-0805, F.Cu at (745.6, 237.3)
- added C429: 100n, OHDSP-Footprints-Pretty:SMD-0805, F.Cu at (750.6, 231.5)
- added C430: 100n, OHDSP-Footprints-Pretty:SMD-0805, F.Cu at (781.3, 204.9)
- added C431: 100n, OHDSP-Footprints-Pretty:SMD-0805, F.Cu at (761.0, 223.3)
- added C432: 100n, OHDSP-Footprints-Pretty:SMD-0805, F.Cu at (756.0, 229.1)
- added C433: 1u, OHDSP-Footprints-Pretty:SMD-0805, F.Cu at (766.0, 217.6)
- added C434: 1u, OHDSP-Footprints-Pretty:SMD-0805, F.Cu at (756.0, 223.3)
- added C435: 1u, OHDSP-Footprints-Pretty:SMD-0805, F.Cu at (768.4, 188.4)
- added C436: 1u, OHDSP-Footprints-Pretty:SMD-0805, F.Cu at (735.6, 235.0)
- added C437: 100n, OHDSP-Footprints-Pretty:SMD-0805, F.Cu at (740.6, 228.5)
- added C438: 100n, OHDSP-Footprints-Pretty:SMD-0805, F.Cu at (755.3, 210.8)
- added C439: 100n, OHDSP-Footprints-Pretty:SMD-0805, F.Cu at (766.3, 200.4)
- added C440: 100n, OHDSP-Footprints-Pretty:SMD-0805, F.Cu at (746.0, 220.0)
- added C441: 22u, OHDSP-Footprints-Pretty:SMD-0805, F.Cu at (761.3, 200.4)
- added C442: 22u, OHDSP-Footprints-Pretty:SMD-0805, F.Cu at (782.0, 178.7)
- added C443: 22u, OHDSP-Footprints-Pretty:SMD-0805, F.Cu at (778.4, 187.7)
- added C444: 22u, OHDSP-Footprints-Pretty:SMD-0805, F.Cu at (740.6, 234.3)
- added C445: 220u, OHDSP-Footprints-Pretty:CAP-TH-D6.3mmP2.5mm, F.Cu at (731.4, 222.0)
- added C446: 220u, OHDSP-Footprints-Pretty:CAP-TH-D6.3mmP2.5mm, F.Cu at (767.4, 181.1)
- added C447: 220u, OHDSP-Footprints-Pretty:CAP-TH-D6.3mmP2.5mm, F.Cu at (753.8, 194.6)
- added C448: 220u, OHDSP-Footprints-Pretty:CAP-TH-D6.3mmP2.5mm, F.Cu at (740.1, 199.7)
- added C501: 220u, OHDSP-Footprints-Pretty:CAP-TH-D6.3mmP2.5mm, F.Cu at (728.5, 107.5)
- added C502: 22u, OHDSP-Footprints-Pretty:SMD-0805, F.Cu at (774.0, 89.4)
- added C503: 100n, OHDSP-Footprints-Pretty:SMD-0805, F.Cu at (764.0, 100.9)
- added C504: 1u, OHDSP-Footprints-Pretty:SMD-0805, F.Cu at (756.6, 106.6)
- added C505: 100n, OHDSP-Footprints-Pretty:SMD-0805, F.Cu at (769.0, 100.9)
- added C518: 100n, OHDSP-Footprints-Pretty:SMD-0805, F.Cu at (777.7, 83.6)
- added C519: 1u, OHDSP-Footprints-Pretty:SMD-0805, F.Cu at (718.2, 110.7)
- added C520: 100n, OHDSP-Footprints-Pretty:SMD-0805, F.Cu at (749.0, 95.0)
- added C521: 1u, OHDSP-Footprints-Pretty:SMD-0805, F.Cu at (754.0, 99.1)
- added C522: 100n, OHDSP-Footprints-Pretty:SMD-0805, F.Cu at (759.0, 89.4)
- added C523: 100n, OHDSP-Footprints-Pretty:SMD-0805, F.Cu at (772.7, 77.9)
- added C524: 100n, OHDSP-Footprints-Pretty:SMD-0805, F.Cu at (767.7, 83.6)
- added C525: 10u, OHDSP-Footprints-Pretty:SMD-0805, F.Cu at (739.4, 109.9)
- added C526: 10u, OHDSP-Footprints-Pretty:SMD-0805, F.Cu at (746.6, 100.8)
- added C527: 220u, OHDSP-Footprints-Pretty:CAP-TH-D6.3mmP2.5mm, F.Cu at (740.6, 102.6)
- added C528: 220u, OHDSP-Footprints-Pretty:CAP-TH-D6.3mmP2.5mm, F.Cu at (756.8, 80.3)
- added C601: 100n, OHDSP-Footprints-Pretty:CAP_TH_5mm, F.Cu at (633.4, 229.0)
- added C602: 47u, OHDSP-Footprints-Pretty:CAP-TH-D10mmP5mm, F.Cu at (607.8, 235.3)
- added C603: 470p, OHDSP-Footprints-Pretty:CAP_TH_5mm, F.Cu at (656.6, 210.6)
- added C604: 470p, OHDSP-Footprints-Pretty:CAP_TH_5mm, F.Cu at (642.4, 229.0)
- added C605: 470p, OHDSP-Footprints-Pretty:CAP_TH_5mm, F.Cu at (605.4, 259.2)
- added C606: 470p, OHDSP-Footprints-Pretty:CAP_TH_5mm, F.Cu at (651.5, 228.5)
- added C607: 150p, OHDSP-Footprints-Pretty:CAP_TH_5mm, F.Cu at (592.9, 272.3)
- added C608: 150p, OHDSP-Footprints-Pretty:CAP_TH_5mm, F.Cu at (614.5, 259.6)
- added C609: 150p, OHDSP-Footprints-Pretty:CAP_TH_5mm, F.Cu at (626.2, 250.7)
- added C610: 150p, OHDSP-Footprints-Pretty:CAP_TH_5mm, F.Cu at (639.5, 238.0)
- added C611: 100n, OHDSP-Footprints-Pretty:CAP_TH_5mm, F.Cu at (656.6, 219.6)
- added C612: 47u, OHDSP-Footprints-Pretty:CAP-TH-D10mmP5mm, F.Cu at (634.4, 212.2)
- added C613: 100n, OHDSP-Footprints-Pretty:CAP_TH_5mm, F.Cu at (605.4, 268.1)
- added C614: 220u, OHDSP-Footprints-Pretty:CAP-TH-D10mmP5mm, F.Cu at (595.0, 242.8)
- added C615: 100n, OHDSP-Footprints-Pretty:CAP_TH_5mm, F.Cu at (617.2, 250.7)
- added C616: 220u, OHDSP-Footprints-Pretty:CAP-TH-D10mmP5mm, F.Cu at (611.2, 222.6)
- added C617: 100n, OHDSP-Footprints-Pretty:CAP_TH_5mm, F.Cu at (630.4, 238.0)
- added C618: 220u, OHDSP-Footprints-Pretty:CAP-TH-D10mmP5mm, F.Cu at (570.7, 266.1)
- added C619: 100n, OHDSP-Footprints-Pretty:CAP_TH_5mm, F.Cu at (617.9, 241.7)
- added C620: 220u, OHDSP-Footprints-Pretty:CAP-TH-D10mmP5mm, F.Cu at (646.5, 212.2)
- added C621: 5n6, OHDSP-Footprints-Pretty:CAP_TH_5mm, F.Cu at (601.9, 277.1)
- added C622: 5n6, OHDSP-Footprints-Pretty:CAP_TH_5mm, F.Cu at (623.5, 259.6)
- added C623: 5n6, OHDSP-Footprints-Pretty:CAP_TH_5mm, F.Cu at (635.3, 246.9)
- added C624: 5n6, OHDSP-Footprints-Pretty:CAP_TH_5mm, F.Cu at (614.5, 268.6)
- added C625: 100u, OHDSP-Footprints-Pretty:CAP-TH-D10mmP5mm, F.Cu at (582.8, 268.2)
- added C626: 100u, OHDSP-Footprints-Pretty:CAP-TH-D10mmP5mm, F.Cu at (595.7, 228.2)
- added C627: 100u, OHDSP-Footprints-Pretty:CAP-TH-D10mmP5mm, F.Cu at (607.1, 248.0)
- added C628: 100u, OHDSP-Footprints-Pretty:CAP-TH-D10mmP5mm, F.Cu at (623.3, 224.9)
- added C629: 100u, OHDSP-Footprints-Pretty:CAP-TH-D10mmP5mm, F.Cu at (595.0, 255.5)
- added C630: 100u, OHDSP-Footprints-Pretty:CAP-TH-D10mmP5mm, F.Cu at (570.7, 253.4)
- added C631: 100u, OHDSP-Footprints-Pretty:CAP-TH-D10mmP5mm, F.Cu at (582.8, 242.8)
- added C632: 100u, OHDSP-Footprints-Pretty:CAP-TH-D10mmP5mm, F.Cu at (582.8, 255.5)
- added C633: 100n, OHDSP-Footprints-Pretty:SMD-0805, F.Cu at (646.3, 235.3)
- added C634: 100n, OHDSP-Footprints-Pretty:SMD-0805, F.Cu at (658.3, 225.9)
- added C635: 100n, OHDSP-Footprints-Pretty:SMD-0805, F.Cu at (663.4, 219.5)
- added C636: 100n, OHDSP-Footprints-Pretty:SMD-0805, F.Cu at (663.4, 213.8)
- added C637: 100n, OHDSP-Footprints-Pretty:SMD-0805, F.Cu at (663.4, 208.0)
- added C638: 100n, OHDSP-Footprints-Pretty:SMD-0805, F.Cu at (620.9, 265.9)
- added C639: 100n, OHDSP-Footprints-Pretty:SMD-0805, F.Cu at (576.0, 276.7)
- added C640: 100n, OHDSP-Footprints-Pretty:SMD-0805, F.Cu at (581.0, 276.7)
- added C701: 100p, OHDSP-Footprints-Pretty:CAP_TH_5mm, F.Cu at (700.7, 80.5)
- added C702: 100p, OHDSP-Footprints-Pretty:CAP_TH_5mm, F.Cu at (701.6, 98.4)
- added C703: 100u, OHDSP-Footprints-Pretty:CAP-TH-D10mmP5mm, F.Cu at (602.6, 142.8)
- added C704: 100n, OHDSP-Footprints-Pretty:CAP_TH_5mm, F.Cu at (646.0, 151.0)
- added C705: 100u, OHDSP-Footprints-Pretty:CAP-TH-D10mmP5mm, F.Cu at (666.4, 82.1)
- added C706: 100n, OHDSP-Footprints-Pretty:CAP_TH_5mm, F.Cu at (636.9, 151.0)
- added C707: 100p, OHDSP-Footprints-Pretty:CAP_TH_5mm, F.Cu at (691.8, 111.1)
- added C708: 100p, OHDSP-Footprints-Pretty:CAP_TH_5mm, F.Cu at (683.4, 93.2)
- added C709: 100u, OHDSP-Footprints-Pretty:CAP-TH-D10mmP5mm, F.Cu at (618.1, 119.4)
- added C710: 100n, OHDSP-Footprints-Pretty:CAP_TH_5mm, F.Cu at (636.9, 142.0)
- added C711: 100u, OHDSP-Footprints-Pretty:CAP-TH-D10mmP5mm, F.Cu at (649.1, 92.7)
- added C712: 100n, OHDSP-Footprints-Pretty:CAP_TH_5mm, F.Cu at (619.8, 160.1)
- added C713: 100u, OHDSP-Footprints-Pretty:CAP-TH-D10mmP5mm, F.Cu at (602.6, 130.1)
- added C714: 100n, OHDSP-Footprints-Pretty:CAP_TH_5mm, F.Cu at (628.8, 160.1)
- added C715: 10u, OHDSP-Footprints-Pretty:CAP-TH-D10mmP5mm, F.Cu at (626.9, 136.2)
- added C716: 10u, OHDSP-Footprints-Pretty:CAP-TH-D10mmP5mm, F.Cu at (657.9, 107.5)
- added C717: 10u, OHDSP-Footprints-Pretty:CAP-TH-D10mmP5mm, F.Cu at (670.0, 107.5)
- added C718: 10u, OHDSP-Footprints-Pretty:CAP-TH-D10mmP5mm, F.Cu at (642.4, 118.2)
- added C719: 100n, OHDSP-Footprints-Pretty:CAP_TH_5mm, F.Cu at (646.0, 142.0)
- added C720: 100n, OHDSP-Footprints-Pretty:CAP_TH_5mm, F.Cu at (683.4, 102.2)
- added C721: 100n, OHDSP-Footprints-Pretty:CAP_TH_5mm, F.Cu at (692.5, 93.2)
- added C722: 100n, OHDSP-Footprints-Pretty:CAP_TH_5mm, F.Cu at (652.4, 131.4)
- added C723: 47p, OHDSP-Footprints-Pretty:CAP_TH_5mm, F.Cu at (664.1, 145.5)
- added C724: 47p, OHDSP-Footprints-Pretty:CAP_TH_5mm, F.Cu at (681.8, 138.0)
- added C725: 47p, OHDSP-Footprints-Pretty:CAP_TH_5mm, F.Cu at (691.3, 129.0)
- added C726: 47p, OHDSP-Footprints-Pretty:CAP_TH_5mm, F.Cu at (672.8, 145.5)
- added C727: 1n, OHDSP-Footprints-Pretty:CAP_TH_5mm, F.Cu at (655.6, 167.2)
- added C728: 1n, OHDSP-Footprints-Pretty:CAP_TH_5mm, F.Cu at (682.7, 120.1)
- added C729: 1n, OHDSP-Footprints-Pretty:CAP_TH_5mm, F.Cu at (637.9, 168.9)
- added C730: 1n, OHDSP-Footprints-Pretty:CAP_TH_5mm, F.Cu at (655.1, 149.3)
- added C731: 100u, OHDSP-Footprints-Pretty:CAP-TH-D10mmP5mm, F.Cu at (690.7, 82.1)
- added C732: 100u, OHDSP-Footprints-Pretty:CAP-TH-D10mmP5mm, F.Cu at (642.4, 130.9)
- added C733: 100n, OHDSP-Footprints-Pretty:SMD-0805, F.Cu at (667.0, 157.6)
- added C734: 100n, OHDSP-Footprints-Pretty:SMD-0805, F.Cu at (679.2, 144.3)
- added C735: 100p, OHDSP-Footprints-Pretty:CAP_TH_5mm, F.Cu at (619.8, 169.0)
- added C736: 100p, OHDSP-Footprints-Pretty:CAP_TH_5mm, F.Cu at (701.6, 89.5)
- added C737: 100u, OHDSP-Footprints-Pretty:CAP-TH-D10mmP5mm, F.Cu at (633.6, 98.1)
- added C738: 100n, OHDSP-Footprints-Pretty:CAP_TH_5mm, F.Cu at (655.1, 140.3)
- added C739: 100u, OHDSP-Footprints-Pretty:CAP-TH-D10mmP5mm, F.Cu at (614.7, 144.8)
- added C740: 100n, OHDSP-Footprints-Pretty:CAP_TH_5mm, F.Cu at (628.8, 169.0)
- added C741: 100p, OHDSP-Footprints-Pretty:CAP_TH_5mm, F.Cu at (637.9, 159.9)
- added C742: 100p, OHDSP-Footprints-Pretty:CAP_TH_5mm, F.Cu at (664.6, 118.7)
- added C743: 100u, OHDSP-Footprints-Pretty:CAP-TH-D10mmP5mm, F.Cu at (654.5, 120.2)
- added C744: 100n, OHDSP-Footprints-Pretty:CAP_TH_5mm, F.Cu at (673.6, 127.6)
- added C745: 100u, OHDSP-Footprints-Pretty:CAP-TH-D10mmP5mm, F.Cu at (626.9, 148.9)
- added C746: 100n, OHDSP-Footprints-Pretty:CAP_TH_5mm, F.Cu at (664.1, 136.6)
- added C747: 10u, OHDSP-Footprints-Pretty:CAP-TH-D10mmP5mm, F.Cu at (608.0, 157.5)
- added C748: 10u, OHDSP-Footprints-Pretty:CAP-TH-D10mmP5mm, F.Cu at (595.9, 155.9)
- added C749: 10u, OHDSP-Footprints-Pretty:CAP-TH-D10mmP5mm, F.Cu at (678.5, 82.1)
- added C750: 10u, OHDSP-Footprints-Pretty:CAP-TH-D10mmP5mm, F.Cu at (583.7, 159.2)
- added C751: 100n, OHDSP-Footprints-Pretty:CAP_TH_5mm, F.Cu at (682.7, 111.1)
- added C752: 100n, OHDSP-Footprints-Pretty:CAP_TH_5mm, F.Cu at (692.5, 102.2)
- added C753: 100n, OHDSP-Footprints-Pretty:CAP_TH_5mm, F.Cu at (673.6, 118.7)
- added C754: 100n, OHDSP-Footprints-Pretty:CAP_TH_5mm, F.Cu at (664.6, 127.6)
- added C755: 47p, OHDSP-Footprints-Pretty:CAP_TH_5mm, F.Cu at (646.5, 168.9)
- added C756: 47p, OHDSP-Footprints-Pretty:CAP_TH_5mm, F.Cu at (700.8, 116.3)
- added C757: 47p, OHDSP-Footprints-Pretty:CAP_TH_5mm, F.Cu at (655.6, 158.2)
- added C758: 47p, OHDSP-Footprints-Pretty:CAP_TH_5mm, F.Cu at (682.7, 129.0)
- added C759: 1n, OHDSP-Footprints-Pretty:CAP_TH_5mm, F.Cu at (691.3, 120.1)
- added C760: 1n, OHDSP-Footprints-Pretty:CAP_TH_5mm, F.Cu at (673.2, 136.6)
- added C761: 1n, OHDSP-Footprints-Pretty:CAP_TH_5mm, F.Cu at (701.6, 107.4)
- added C762: 1n, OHDSP-Footprints-Pretty:CAP_TH_5mm, F.Cu at (646.9, 159.9)
- added C763: 100u, OHDSP-Footprints-Pretty:CAP-TH-D10mmP5mm, F.Cu at (587.1, 143.2)
- added C764: 100u, OHDSP-Footprints-Pretty:CAP-TH-D10mmP5mm, F.Cu at (571.6, 159.2)
- added C765: 100u, OHDSP-Footprints-Pretty:CAP-TH-D10mmP5mm, F.Cu at (673.4, 94.8)
- added C766: 100u, OHDSP-Footprints-Pretty:CAP-TH-D10mmP5mm, F.Cu at (661.2, 94.8)
- added C767: 100u, OHDSP-Footprints-Pretty:CAP-TH-D10mmP5mm, F.Cu at (614.7, 132.1)
- added C768: 100u, OHDSP-Footprints-Pretty:CAP-TH-D10mmP5mm, F.Cu at (630.2, 123.5)
- added C769: 100u, OHDSP-Footprints-Pretty:CAP-TH-D10mmP5mm, F.Cu at (645.7, 105.5)
- added C770: 100u, OHDSP-Footprints-Pretty:CAP-TH-D10mmP5mm, F.Cu at (630.2, 110.8)
- added C771: 100n, OHDSP-Footprints-Pretty:SMD-0805, F.Cu at (672.0, 151.8)
- added C772: 100n, OHDSP-Footprints-Pretty:SMD-0805, F.Cu at (688.2, 135.4)
- added C773: 100n, OHDSP-Footprints-Pretty:SMD-0805, F.Cu at (621.5, 99.2)
- added C774: 100n, OHDSP-Footprints-Pretty:SMD-0805, F.Cu at (662.0, 163.3)
- added C775: 100n, OHDSP-Footprints-Pretty:SMD-0805, F.Cu at (662.0, 151.8)
- added C776: 100n, OHDSP-Footprints-Pretty:SMD-0805, F.Cu at (667.0, 151.8)
- added C777: 100n, OHDSP-Footprints-Pretty:SMD-0805, F.Cu at (697.8, 122.6)
- added C778: 100n, OHDSP-Footprints-Pretty:SMD-0805, F.Cu at (662.0, 157.6)
- added C801: 100u, OHDSP-Footprints-Pretty:CAP-TH-D10mmP5mm, F.Cu at (410.1, 305.5)
- added C802: 100n, OHDSP-Footprints-Pretty:CAP_TH_5mm, F.Cu at (464.6, 279.5)
- added C803: 100u, OHDSP-Footprints-Pretty:CAP-TH-D10mmP5mm, F.Cu at (394.6, 320.1)
- added C804: 100n, OHDSP-Footprints-Pretty:CAP_TH_5mm, F.Cu at (486.9, 257.7)
- added C805: 100u, OHDSP-Footprints-Pretty:CAP-TH-D10mmP5mm, F.Cu at (510.0, 212.2)
- added C806: 100n, OHDSP-Footprints-Pretty:CAP_TH_5mm, F.Cu at (474.4, 267.1)
- added C807: 100u, OHDSP-Footprints-Pretty:CAP-TH-D10mmP5mm, F.Cu at (484.9, 237.6)
- added C808: 100n, OHDSP-Footprints-Pretty:CAP_TH_5mm, F.Cu at (455.5, 280.8)
- added C809: 100u, OHDSP-Footprints-Pretty:CAP-TH-D10mmP5mm, F.Cu at (497.8, 212.2)
- added C810: 100u, OHDSP-Footprints-Pretty:CAP-TH-D10mmP5mm, F.Cu at (382.4, 320.1)
- added C811: 100u, OHDSP-Footprints-Pretty:CAP-TH-D10mmP5mm, F.Cu at (452.2, 244.2)
- added C812: 100u, OHDSP-Footprints-Pretty:CAP-TH-D10mmP5mm, F.Cu at (421.2, 282.3)
- added C813: 100n, OHDSP-Footprints-Pretty:SMD-0805, F.Cu at (472.1, 238.8)
- added C814: 100n, OHDSP-Footprints-Pretty:SMD-0805, F.Cu at (409.1, 294.3)
- added C815: 100n, OHDSP-Footprints-Pretty:SMD-0805, F.Cu at (440.6, 326.6)
- added C816: 100n, OHDSP-Footprints-Pretty:SMD-0805, F.Cu at (445.6, 326.6)
- added C817: 1n, OHDSP-Footprints-Pretty:CAP_TH_5mm, F.Cu at (479.8, 302.9)
- added C818: 1n, OHDSP-Footprints-Pretty:CAP_TH_5mm, F.Cu at (464.2, 325.5)
- added C819: 1n, OHDSP-Footprints-Pretty:CAP_TH_5mm, F.Cu at (518.4, 271.9)
- added C820: 1n, OHDSP-Footprints-Pretty:CAP_TH_5mm, F.Cu at (499.6, 289.8)
- added C821: 100u, OHDSP-Footprints-Pretty:CAP-TH-D10mmP5mm, F.Cu at (433.3, 282.3)
- added C822: 1n, OHDSP-Footprints-Pretty:CAP_TH_5mm, F.Cu at (473.6, 285.0)
- added C823: 1n, OHDSP-Footprints-Pretty:CAP_TH_5mm, F.Cu at (492.5, 266.7)
- added C824: 1n, OHDSP-Footprints-Pretty:CAP_TH_5mm, F.Cu at (462.5, 298.7)
- added C825: 1n, OHDSP-Footprints-Pretty:CAP_TH_5mm, F.Cu at (438.2, 320.3)
- added C826: 100u, OHDSP-Footprints-Pretty:CAP-TH-D10mmP5mm, F.Cu at (448.8, 269.6)
- added C827: 1n, OHDSP-Footprints-Pretty:CAP_TH_5mm, F.Cu at (505.1, 262.9)
- added C828: 1n, OHDSP-Footprints-Pretty:CAP_TH_5mm, F.Cu at (446.9, 320.3)
- added C829: 100u, OHDSP-Footprints-Pretty:CAP-TH-D10mmP5mm, F.Cu at (370.3, 318.0)
- added C830: 100u, OHDSP-Footprints-Pretty:CAP-TH-D10mmP5mm, F.Cu at (464.3, 243.0)
- added C831: 1n, OHDSP-Footprints-Pretty:CAP_TH_5mm, F.Cu at (482.3, 294.0)
- added C832: 1n, OHDSP-Footprints-Pretty:CAP_TH_5mm, F.Cu at (471.2, 302.9)
- added C833: 100n, OHDSP-Footprints-Pretty:SMD-0805, F.Cu at (409.1, 288.6)
- added C834: 100n, OHDSP-Footprints-Pretty:SMD-0805, F.Cu at (458.6, 231.4)
- added C835: 100n, OHDSP-Footprints-Pretty:SMD-0805, F.Cu at (453.6, 231.4)
- added C836: 100n, OHDSP-Footprints-Pretty:SMD-0805, F.Cu at (448.6, 229.7)
- added C837: 100u, OHDSP-Footprints-Pretty:CAP-TH-D10mmP5mm, F.Cu at (484.9, 224.9)
- added C838: 100u, OHDSP-Footprints-Pretty:CAP-TH-D10mmP5mm, F.Cu at (409.0, 280.1)
- added C839: 100u, OHDSP-Footprints-Pretty:CAP-TH-D10mmP5mm, F.Cu at (472.8, 230.2)
- added C840: 100u, OHDSP-Footprints-Pretty:CAP-TH-D10mmP5mm, F.Cu at (440.0, 244.2)
- added C841: 100n, OHDSP-Footprints-Pretty:SMD-0805, F.Cu at (497.3, 296.1)
- added C842: 100n, OHDSP-Footprints-Pretty:SMD-0805, F.Cu at (486.2, 300.3)
- added C843: 100n, OHDSP-Footprints-Pretty:SMD-0805, F.Cu at (470.6, 315.0)
- added C844: 100n, OHDSP-Footprints-Pretty:SMD-0805, F.Cu at (475.6, 309.3)
- added C845: 100p, OHDSP-Footprints-Pretty:CAP_TH_5mm, F.Cu at (520.0, 216.3)
- added C846: 100p, OHDSP-Footprints-Pretty:CAP_TH_5mm, F.Cu at (464.6, 288.5)
- added C847: N/F, OHDSP-Footprints-Pretty:CAP_TH_5mm, F.Cu at (464.2, 316.6)
- added C848: N/F, OHDSP-Footprints-Pretty:CAP_TH_5mm, F.Cu at (525.3, 243.1)
- added C849: N/F, OHDSP-Footprints-Pretty:CAP_TH_5mm, F.Cu at (455.5, 325.5)
- added C850: N/F, OHDSP-Footprints-Pretty:CAP_TH_5mm, F.Cu at (490.9, 294.0)
- added C851: N/F, OHDSP-Footprints-Pretty:CAP_TH_5mm, F.Cu at (509.8, 271.9)
- added C852: N/F, OHDSP-Footprints-Pretty:CAP_TH_5mm, F.Cu at (522.3, 262.9)
- added C853: 100u, OHDSP-Footprints-Pretty:CAP-TH-D10mmP5mm, F.Cu at (452.2, 256.9)
- added C854: 100n, OHDSP-Footprints-Pretty:CAP_TH_5mm, F.Cu at (486.5, 248.8)
- added C855: 100u, OHDSP-Footprints-Pretty:CAP-TH-D10mmP5mm, F.Cu at (436.7, 269.6)
- added C856: 100n, OHDSP-Footprints-Pretty:CAP_TH_5mm, F.Cu at (496.0, 257.7)
- added C857: 100u, OHDSP-Footprints-Pretty:CAP-TH-D10mmP5mm, F.Cu at (427.9, 244.2)
- added C858: 100n, OHDSP-Footprints-Pretty:CAP_TH_5mm, F.Cu at (441.3, 311.4)
- added C859: 100u, OHDSP-Footprints-Pretty:CAP-TH-D10mmP5mm, F.Cu at (427.9, 256.9)
- added C860: 100n, OHDSP-Footprints-Pretty:CAP_TH_5mm, F.Cu at (516.2, 236.1)
- added C861: 100u, OHDSP-Footprints-Pretty:CAP-TH-D10mmP5mm, F.Cu at (389.1, 294.7)
- added C862: 100n, OHDSP-Footprints-Pretty:CAP_TH_5mm, F.Cu at (455.5, 289.7)
- added C863: 100u, OHDSP-Footprints-Pretty:CAP-TH-D10mmP5mm, F.Cu at (485.7, 212.2)
- added C864: 100n, OHDSP-Footprints-Pretty:CAP_TH_5mm, F.Cu at (483.4, 267.1)
- added C865: 100u, OHDSP-Footprints-Pretty:CAP-TH-D10mmP5mm, F.Cu at (401.3, 292.8)
- added C866: 100u, OHDSP-Footprints-Pretty:CAP-TH-D10mmP5mm, F.Cu at (385.8, 307.4)
- added C867: 100u, OHDSP-Footprints-Pretty:CAP-TH-D10mmP5mm, F.Cu at (440.0, 256.9)
- added C868: 100n, OHDSP-Footprints-Pretty:CAP_TH_5mm, F.Cu at (429.2, 318.9)
- added C869: 100u, OHDSP-Footprints-Pretty:CAP-TH-D10mmP5mm, F.Cu at (472.8, 217.5)
- added C870: 100n, OHDSP-Footprints-Pretty:CAP_TH_5mm, F.Cu at (453.5, 298.7)
- added C871: 100u, OHDSP-Footprints-Pretty:CAP-TH-D10mmP5mm, F.Cu at (424.5, 269.6)
- added C872: 100u, OHDSP-Footprints-Pretty:CAP-TH-D10mmP5mm, F.Cu at (412.4, 264.1)
- added C873: 100n, OHDSP-Footprints-Pretty:CAP_TH_5mm, F.Cu at (432.3, 306.2)
- added C874: 100u, OHDSP-Footprints-Pretty:CAP-TH-D10mmP5mm, F.Cu at (397.9, 307.4)
- added C875: 100n, OHDSP-Footprints-Pretty:CAP_TH_5mm, F.Cu at (507.1, 236.1)
- added C876: 100u, OHDSP-Footprints-Pretty:CAP-TH-D10mmP5mm, F.Cu at (396.9, 280.1)
- added C877: 100n, OHDSP-Footprints-Pretty:SMD-0805, F.Cu at (435.6, 326.6)
- added C878: 100n, OHDSP-Footprints-Pretty:SMD-0805, F.Cu at (506.0, 287.1)
- added C879: 100n, OHDSP-Footprints-Pretty:SMD-0805, F.Cu at (480.6, 309.3)
- added C880: 100n, OHDSP-Footprints-Pretty:SMD-0805, F.Cu at (470.6, 320.7)
- added C881: 100u, OHDSP-Footprints-Pretty:CAP-TH-D10mmP5mm, F.Cu at (358.1, 314.6)
- added C882: 100u, OHDSP-Footprints-Pretty:CAP-TH-D10mmP5mm, F.Cu at (464.3, 255.7)
- added C883: 100u, OHDSP-Footprints-Pretty:CAP-TH-D10mmP5mm, F.Cu at (373.6, 305.3)
- added C884: 100u, OHDSP-Footprints-Pretty:CAP-TH-D10mmP5mm, F.Cu at (460.6, 222.9)
- added C885: 100n, OHDSP-Footprints-Pretty:SMD-0805, F.Cu at (491.2, 300.3)
- added C886: 100n, OHDSP-Footprints-Pretty:SMD-0805, F.Cu at (470.6, 309.3)
- added C887: 100n, OHDSP-Footprints-Pretty:SMD-0805, F.Cu at (475.6, 315.0)
- added C888: 100n, OHDSP-Footprints-Pretty:SMD-0805, F.Cu at (448.6, 224.0)
- added C889: 1n, OHDSP-Footprints-Pretty:CAP_TH_5mm, F.Cu at (513.7, 262.9)
- added C890: 1n, OHDSP-Footprints-Pretty:CAP_TH_5mm, F.Cu at (522.3, 254.0)
- added C891: 1n, OHDSP-Footprints-Pretty:CAP_TH_5mm, F.Cu at (501.1, 271.9)
- added C892: 1n, OHDSP-Footprints-Pretty:CAP_TH_5mm, F.Cu at (462.1, 307.6)
- added C893: 1n, OHDSP-Footprints-Pretty:CAP_TH_5mm, F.Cu at (483.4, 276.1)
- added C894: 1n, OHDSP-Footprints-Pretty:CAP_TH_5mm, F.Cu at (505.1, 254.0)
- added C895: 1n, OHDSP-Footprints-Pretty:CAP_TH_5mm, F.Cu at (453.5, 307.6)
- added C896: 1n, OHDSP-Footprints-Pretty:CAP_TH_5mm, F.Cu at (516.2, 245.0)
- added C897: 1n, OHDSP-Footprints-Pretty:CAP_TH_5mm, F.Cu at (525.3, 234.2)
- added C898: 1n, OHDSP-Footprints-Pretty:CAP_TH_5mm, F.Cu at (429.2, 327.8)
- added C899: 1n, OHDSP-Footprints-Pretty:CAP_TH_5mm, F.Cu at (513.7, 254.0)
- added C900: 1n, OHDSP-Footprints-Pretty:CAP_TH_5mm, F.Cu at (473.6, 294.0)
- added C901: 100u, OHDSP-Footprints-Pretty:CAP-TH-D10mmP5mm, F.Cu at (509.2, 224.9)
- added C902: 100u, OHDSP-Footprints-Pretty:CAP-TH-D10mmP5mm, F.Cu at (464.3, 268.4)
- added C903: 100u, OHDSP-Footprints-Pretty:CAP-TH-D10mmP5mm, F.Cu at (497.1, 224.9)
- added C904: 100u, OHDSP-Footprints-Pretty:CAP-TH-D10mmP5mm, F.Cu at (422.2, 307.7)
- added C905: 100n, OHDSP-Footprints-Pretty:SMD-0805, F.Cu at (486.2, 306.0)
- added C906: 100n, OHDSP-Footprints-Pretty:SMD-0805, F.Cu at (526.8, 213.7)
- added C907: 100n, OHDSP-Footprints-Pretty:SMD-0805, F.Cu at (526.1, 225.1)
- added C908: 100n, OHDSP-Footprints-Pretty:SMD-0805, F.Cu at (526.8, 219.4)
- added C909: 100p, OHDSP-Footprints-Pretty:CAP_TH_5mm, F.Cu at (444.4, 293.5)
- added C910: 100p, OHDSP-Footprints-Pretty:CAP_TH_5mm, F.Cu at (420.1, 318.9)
- added C911: N/F, OHDSP-Footprints-Pretty:CAP_TH_5mm, F.Cu at (509.8, 280.8)
- added C912: N/F, OHDSP-Footprints-Pretty:CAP_TH_5mm, F.Cu at (490.9, 285.0)
- added C913: N/F, OHDSP-Footprints-Pretty:CAP_TH_5mm, F.Cu at (482.3, 285.0)
- added C914: N/F, OHDSP-Footprints-Pretty:CAP_TH_5mm, F.Cu at (492.5, 275.6)
- added C915: N/F, OHDSP-Footprints-Pretty:CAP_TH_5mm, F.Cu at (455.5, 316.6)
- added C916: N/F, OHDSP-Footprints-Pretty:CAP_TH_5mm, F.Cu at (501.1, 280.8)
- added C917: 100u, OHDSP-Footprints-Pretty:CAP-TH-D10mmP5mm, F.Cu at (434.4, 295.0)
- added C918: 100n, OHDSP-Footprints-Pretty:CAP_TH_5mm, F.Cu at (507.1, 245.0)
- added C919: 100u, OHDSP-Footprints-Pretty:CAP-TH-D10mmP5mm, F.Cu at (445.5, 282.3)
- added C920: 100n, OHDSP-Footprints-Pretty:CAP_TH_5mm, F.Cu at (495.6, 248.8)
- added C921: 100u, OHDSP-Footprints-Pretty:CAP-TH-D10mmP5mm, F.Cu at (476.5, 250.3)
- added C922: 100n, OHDSP-Footprints-Pretty:CAP_TH_5mm, F.Cu at (474.4, 276.1)
- added C923: 100u, OHDSP-Footprints-Pretty:CAP-TH-D10mmP5mm, F.Cu at (497.1, 237.6)
- added C924: 100n, OHDSP-Footprints-Pretty:CAP_TH_5mm, F.Cu at (519.3, 225.2)
- added C925: 100u, OHDSP-Footprints-Pretty:CAP-TH-D10mmP5mm, F.Cu at (422.2, 295.0)
- added C926: 100n, OHDSP-Footprints-Pretty:CAP_TH_5mm, F.Cu at (420.1, 327.8)
- added C927: 100u, OHDSP-Footprints-Pretty:CAP-TH-D10mmP5mm, F.Cu at (410.1, 318.2)
- added C928: 100n, OHDSP-Footprints-Pretty:CAP_TH_5mm, F.Cu at (444.4, 302.4)
- added C929: 100u, OHDSP-Footprints-Pretty:CAP-TH-D10mmP5mm, F.Cu at (497.1, 94.8)
- added C930: 100n, OHDSP-Footprints-Pretty:CAP_TH_5mm, F.Cu at (441.6, 190.2)
- added C931: 100u, OHDSP-Footprints-Pretty:CAP-TH-D10mmP5mm, F.Cu at (401.3, 162.7)
- added C932: 100n, OHDSP-Footprints-Pretty:CAP_TH_5mm, F.Cu at (517.8, 120.1)
- added C933: 100u, OHDSP-Footprints-Pretty:CAP-TH-D10mmP5mm, F.Cu at (485.7, 82.1)
- added C934: 100n, OHDSP-Footprints-Pretty:CAP_TH_5mm, F.Cu at (474.6, 163.9)
- added C935: 100u, OHDSP-Footprints-Pretty:CAP-TH-D10mmP5mm, F.Cu at (440.0, 114.1)
- added C936: 100n, OHDSP-Footprints-Pretty:CAP_TH_5mm, F.Cu at (463.5, 176.3)
- added C937: 100u, OHDSP-Footprints-Pretty:CAP-TH-D10mmP5mm, F.Cu at (412.4, 134.0)
- added C938: 100u, OHDSP-Footprints-Pretty:CAP-TH-D10mmP5mm, F.Cu at (427.9, 114.1)
- added C939: 100u, OHDSP-Footprints-Pretty:CAP-TH-D10mmP5mm, F.Cu at (433.3, 152.2)
- added C940: 100u, OHDSP-Footprints-Pretty:CAP-TH-D10mmP5mm, F.Cu at (484.9, 107.5)
- added C941: 100n, OHDSP-Footprints-Pretty:SMD-0805, F.Cu at (522.9, 144.3)
- added C942: 100n, OHDSP-Footprints-Pretty:SMD-0805, F.Cu at (508.5, 159.0)
- added C943: 100n, OHDSP-Footprints-Pretty:SMD-0805, F.Cu at (513.5, 153.3)
- added C944: 100n, OHDSP-Footprints-Pretty:SMD-0805, F.Cu at (508.5, 153.3)
- added C945: 1n, OHDSP-Footprints-Pretty:CAP_TH_5mm, F.Cu at (493.5, 163.4)
- added C946: 1n, OHDSP-Footprints-Pretty:CAP_TH_5mm, F.Cu at (502.1, 154.5)
- added C947: 1n, OHDSP-Footprints-Pretty:CAP_TH_5mm, F.Cu at (459.7, 195.4)
- added C948: 1n, OHDSP-Footprints-Pretty:CAP_TH_5mm, F.Cu at (483.3, 178.0)
- added C949: 100u, OHDSP-Footprints-Pretty:CAP-TH-D10mmP5mm, F.Cu at (448.8, 139.5)
- added C950: 1n, OHDSP-Footprints-Pretty:CAP_TH_5mm, F.Cu at (515.1, 138.0)
- added C951: 1n, OHDSP-Footprints-Pretty:CAP_TH_5mm, F.Cu at (483.7, 169.1)
- added C952: 1n, OHDSP-Footprints-Pretty:CAP_TH_5mm, F.Cu at (493.5, 154.5)
- added C953: 1n, OHDSP-Footprints-Pretty:CAP_TH_5mm, F.Cu at (502.8, 145.5)
- added C954: 100u, OHDSP-Footprints-Pretty:CAP-TH-D10mmP5mm, F.Cu at (509.2, 94.8)
- added C955: 1n, OHDSP-Footprints-Pretty:CAP_TH_5mm, F.Cu at (474.6, 172.8)
- added C956: 1n, OHDSP-Footprints-Pretty:CAP_TH_5mm, F.Cu at (526.8, 120.1)
- added C957: 100u, OHDSP-Footprints-Pretty:CAP-TH-D10mmP5mm, F.Cu at (476.5, 120.2)
- added C958: 100u, OHDSP-Footprints-Pretty:CAP-TH-D10mmP5mm, F.Cu at (472.8, 100.1)
- added C959: 1n, OHDSP-Footprints-Pretty:CAP_TH_5mm, F.Cu at (478.1, 187.0)
- added C960: 1n, OHDSP-Footprints-Pretty:CAP_TH_5mm, F.Cu at (492.3, 172.4)
- added C961: 100n, OHDSP-Footprints-Pretty:SMD-0805, F.Cu at (442.0, 196.5)
- added C962: 100n, OHDSP-Footprints-Pretty:SMD-0805, F.Cu at (437.0, 196.5)
- added C963: 100n, OHDSP-Footprints-Pretty:SMD-0805, F.Cu at (517.9, 144.3)
- added C964: 100n, OHDSP-Footprints-Pretty:SMD-0805, F.Cu at (489.7, 178.7)
- added C965: 100u, OHDSP-Footprints-Pretty:CAP-TH-D10mmP5mm, F.Cu at (484.9, 94.8)
- added C966: 100u, OHDSP-Footprints-Pretty:CAP-TH-D10mmP5mm, F.Cu at (464.3, 112.8)
- added C967: 100u, OHDSP-Footprints-Pretty:CAP-TH-D10mmP5mm, F.Cu at (409.0, 150.0)
- added C968: 100u, OHDSP-Footprints-Pretty:CAP-TH-D10mmP5mm, F.Cu at (472.8, 87.4)
- added C969: 100n, OHDSP-Footprints-Pretty:SMD-0805, F.Cu at (513.5, 159.0)
- added C970: 100n, OHDSP-Footprints-Pretty:SMD-0805, F.Cu at (498.8, 169.7)
- added C971: 100n, OHDSP-Footprints-Pretty:SMD-0805, F.Cu at (484.6, 184.3)
- added C972: 100n, OHDSP-Footprints-Pretty:SMD-0805, F.Cu at (475.9, 193.3)
- added C973: 100p, OHDSP-Footprints-Pretty:CAP_TH_5mm, F.Cu at (460.4, 186.4)
- added C974: 100p, OHDSP-Footprints-Pretty:CAP_TH_5mm, F.Cu at (506.1, 132.8)
- added C975: N/F, OHDSP-Footprints-Pretty:CAP_TH_5mm, F.Cu at (526.8, 129.0)
- added C976: N/F, OHDSP-Footprints-Pretty:CAP_TH_5mm, F.Cu at (469.5, 185.2)
- added C977: N/F, OHDSP-Footprints-Pretty:CAP_TH_5mm, F.Cu at (511.5, 146.9)
- added C978: N/F, OHDSP-Footprints-Pretty:CAP_TH_5mm, F.Cu at (523.8, 138.0)
- added C979: N/F, OHDSP-Footprints-Pretty:CAP_TH_5mm, F.Cu at (469.5, 194.2)
- added C980: N/F, OHDSP-Footprints-Pretty:CAP_TH_5mm, F.Cu at (502.1, 163.4)
- added C981: 100u, OHDSP-Footprints-Pretty:CAP-TH-D10mmP5mm, F.Cu at (440.0, 126.8)
- added C982: 100n, OHDSP-Footprints-Pretty:CAP_TH_5mm, F.Cu at (451.4, 186.4)
- added C983: 100u, OHDSP-Footprints-Pretty:CAP-TH-D10mmP5mm, F.Cu at (396.9, 150.0)
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Connections:
- C201 pad 1: /ADAU1701/FILTA -> /ADAU1701/DVDD
- C202 pad 1: /ADAU1701/FILTD -> /ADAU1701/FILTA
- C203 pad 1: /ADAU1701/CM -> /ADAU1701/FILTD
- C205 pad 1: /ADAU1701/FILTA -> Net-(C205-Pad1)
- C206 pad 1: /ADAU1701/FILTD -> /ADAU1701/DVDD
- C207 pad 1: /ADAU1701/CM -> Net-(C207-Pad1)
- C208 pad 1: /ADAU1701/DVDD -> /ADAU1701/FILTA
- C209 pad 1: Net-(C209-Pad1) -> /ADAU1701/FILTD
- C210 pad 1: /ADAU1701/FILTA -> /ADAU1701/CM
- C211 pad 1: /ADAU1701/FILTD -> Net-(C207-Pad1)
- C212 pad 1: /ADAU1701/CM -> /ADAU1701/DVDD
- C213 pad 1: Net-(C213-Pad1) -> /ADAU1701/FILTA
- C214 pad 1: /ADAU1701/DVDD -> /ADAU1701/FILTD
- C215 pad 1: Net-(C213-Pad1) -> /ADAU1701/CM
- C220 pad 1: /ADAU1701/DVDD -> Net-(C220-Pad1)
- C221 pad 1: /ADAU1701/DVDD -> /AD1937 CODEC/CODEC_RST
- C223 pad 2: Net-(C223-Pad2) -> GNDD
- C224 pad 1: Net-(C223-Pad1) -> Net-(C224-Pad1)
- C224 pad 2: /ADAU1701/PVDD -> Net-(C224-Pad2)
- C226 pad 1: Net-(C226-Pad1) -> /ADAU1701/IOVDD
- C228 pad 1: /Connectors/ADC_RESET -> /ADAU1701/IOVDD
- C230 pad 1: /ADAU1701/IOVDD -> /ADAU1701/PVDD
- C231 pad 1: /ADAU1701/IOVDD -> /ADAU1701/PVDD
- C232 pad 1: Net-(C232-Pad1) -> /ADAU1701/PVDD
- C233 pad 1: /ADAU1701/IOVDD -> Net-(C233-Pad1)
- C235 pad 1: /ADAU1701/PVDD -> /ADAU1701/AVDD
- C236 pad 1: /ADAU1701/PVDD -> /ADAU1701/AVDD
- C237 pad 1: /ADAU1701/PVDD -> /ADAU1701/AVDD
- C238 pad 1: /ADAU1701/AVDD -> /ADAU1701/DVDD
- C239 pad 1: Net-(C239-Pad1) -> /ADAU1701/AVDD
- C243 pad 1: /ADAU1701/AVDD -> /ADAU1701/IOVDD
- C244 pad 1: /ADAU1701/AVDD -> /ADAU1701/IOVDD
- C245 pad 1: /ADAU1701/AVDD -> VPP
- C301 pad 1: GNDD -> Net-(C301-Pad1)
- C301 pad 2: VCC -> GNDD
- C302 pad 1: GNDD -> Net-(C301-Pad1)
- C302 pad 2: VCC -> GNDD
- C304 pad 1: VCC -> Net-(C304-Pad1)
- C305 pad 1: Net-(C305-Pad1) -> Net-(C303-Pad1)
- C305 pad 2: Net-(C305-Pad2) -> GNDD
- C306 pad 1: GNDD -> Net-(C303-Pad1)
- C306 pad 2: VCC -> GNDD
- C402 pad 1: Net-(C402-Pad1) -> GNDD
- C402 pad 2: GNDD -> VCC
- C405 pad 1: Net-(C404-Pad1) -> Net-(C405-Pad1)
- C406 pad 1: Net-(C404-Pad1) -> GNDD
- C406 pad 2: GNDD -> Net-(C406-Pad2)
- C407 pad 1: Net-(C407-Pad1) -> GNDD
- C407 pad 2: GNDD -> Net-(C405-Pad1)
- C408 pad 1: Net-(C407-Pad1) -> GNDD
- C408 pad 2: GNDD -> Net-(C406-Pad2)
- C506 pad 1: Net-(C506-Pad1) -> /AD1937 CODEC/CDVDD
- C506 pad 2: Net-(C506-Pad2) -> GNDD
- C507 pad 1: Net-(C507-Pad1) -> /AD1937 CODEC/CDVDD
- C507 pad 2: Net-(C507-Pad2) -> GNDD
- C508 pad 2: Net-(C508-Pad2) -> GNDD
- C510 pad 1: Net-(C510-Pad1) -> Net-(C509-Pad1)
- C510 pad 2: Net-(C510-Pad2) -> /AD1937 CODEC/CAVDD
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Routing:
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- removed copper zone on F.Cu, net GNDD
Other:
- board size 100 x 100 mm -> 200 x 100 mm
