File: Schematics/OHDSP-XOVER.sch (KiCad schematic (older format))
At the start: 0 parts

Commit message: WIP
Changed lines of the file:
@@
 LIBS:power
 LIBS:OHDSP-Lib
-LIBS:OHDSP-ADAU1701-cache
+LIBS:OHDSP-XOVER-cache
 EELAYER 25 0
 EELAYER END
 $Descr A4 11693 8268
 encoding utf-8
-Sheet 1 5
+Sheet 1 7
 Title ""
 Date "10 feb 2015"
@@
 Wire Wire Line
 	950  3450 1600 3450
+$Sheet
+S 5750 1500 1500 1050
+U 5574D2FB
+F0 "PSU" 60
+F1 "PSU.sch" 60
+$EndSheet
+$Sheet
+S 6100 3400 1650 800
+U 5574D5A4
+F0 "SPDIF" 60
+F1 "SPDIF.sch" 60
+$EndSheet
 $EndSCHEMATC

Commit message: WIP
Changed lines of the file:
@@
 LIBS:power
 LIBS:OHDSP-Lib
-LIBS:OHDSP-XOVER-cache
 EELAYER 25 0
 EELAYER END
@@
 $EndSheet
 $Sheet
-S 8900 1100 1650 1500
-U 54DA50D9
-F0 "ADAU1701 PSU" 60
-F1 "ADAU1701 PSU.sch" 60
-$EndSheet
-$Sheet
 S 8950 4800 1650 1200
 U 54E20ECF
@@
 Wire Wire Line
 	3400 1400 4000 1400
-$Sheet
-S 1600 2650 1800 1550
-U 54E8D6A6
-F0 "Connectors" 60
-F1 "Connectors.sch" 60
-F2 "ADC_LRCLK0" O L 1600 2750 60
-F3 "ADC_BCLK0" O L 1600 2850 60
-F4 "ADC_SDATA0" O L 1600 2950 60
-F5 "DAC_LRCLK0" I R 3400 2750 60
-F6 "DAC_BCLK0" I R 3400 2850 60
-F7 "DAC_SDATA0" I R 3400 2950 60
-F8 "I2C_SCL" B L 1600 3950 60
-F9 "I2C_SDA" B L 1600 3850 60
-F10 "ADC_SDATA1" O L 1600 3050 60
-F11 "ADC_SDATA2" O L 1600 3150 60
-F12 "ADC_SDATA3" O L 1600 3250 60
-F13 "DAC_SDATA1" I R 3400 3050 60
-F14 "DAC_SDATA2" I R 3400 3150 60
-F15 "DAC_SDATA3" I R 3400 3250 60
-F16 "PI_RST" O L 1600 4100 60
-F17 "ADC_MCLK" I L 1600 3350 60
-F18 "DAC_MCLK" I R 3400 3350 60
-F19 "DAC_RESET" I R 3400 3450 60
-F20 "ADC_RESET" I L 1600 3450 60
-F21 "ADI_RST" O R 3400 4100 60
-F22 "ANA_IN1" O L 1600 3600 60
-F23 "ANA_IN2" O L 1600 3700 60
-F24 "ANA_OUT1" I R 3400 3600 60
-F25 "ANA_OUT2" I R 3400 3700 60
-F26 "ANA_OUT3" I R 3400 3800 60
-F27 "ANA_OUT4" I R 3400 3900 60
-$EndSheet
-Text Label 950  2750 0    60   ~ 0
-IN_LRCLK0
-Text Label 950  2850 0    60   ~ 0
-IN_BCLK0
-Text Label 950  2950 0    60   ~ 0
-IN_SDATA0
-Text Label 950  3050 0    60   ~ 0
-IN_SDATA1
-Text Label 950  3250 0    60   ~ 0
-IN_SDATA3
-Text Label 950  3150 0    60   ~ 0
-IN_SDATA2
-Wire Wire Line
-	950  2750 1600 2750
-Wire Wire Line
-	1600 2850 950  2850
-Wire Wire Line
-	950  2950 1600 2950
-Wire Wire Line
-	1600 3050 950  3050
-Wire Wire Line
-	1600 3150 950  3150
-Wire Wire Line
-	950  3250 1600 3250
-Text Label 4000 2750 2    60   ~ 0
-OUT_LRCLK0
-Text Label 4000 2850 2    60   ~ 0
-OUT_BCLK0
-Text Label 4000 2950 2    60   ~ 0
-OUT_SDATA0
-Wire Wire Line
-	3400 2750 4000 2750
-Wire Wire Line
-	3400 2850 4000 2850
-Wire Wire Line
-	3400 2950 4000 2950
-Text Label 4000 3050 2    60   ~ 0
-OUT_SDATA1
-Wire Wire Line
-	3400 3050 4000 3050
-Text Label 4000 3150 2    60   ~ 0
-OUT_SDATA2
-Wire Wire Line
-	3400 3150 4000 3150
-Text Label 4000 3250 2    60   ~ 0
-OUT_SDATA3
-Wire Wire Line
-	3400 3250 4000 3250
 Text Label 3650 1700 2    60   ~ 0
 SDA
@@
 Wire Wire Line
 	3400 1600 3650 1600
-Text Label 950  3850 0    60   ~ 0
+Text Label 4200 4200 2    60   ~ 0
 SDA
-Text Label 950  3950 0    60   ~ 0
+Text Label 4200 4100 2    60   ~ 0
 SCL
 Wire Wire Line
-	1600 3850 950  3850
-Wire Wire Line
-	1600 3950 950  3950
+	3650 4200 4200 4200
+Wire Wire Line
+	3650 4100 4200 4100
 Text Notes 7000 7100 0    59   ~ 0
 Copyright Paul Janicki 2015\n\nLicensed under the TAPR Open Hardware License (www.tapr.org/OHL).\n\nThis documentation is distributed\nWITHOUT ANY EXPRESS OR IMPLIED WARRANTY, INCLUDING OF\nMERCHANTABILITY, SATISFACTORY QUALITY AND FITNESS FOR A\nPARTICULAR PURPOSE.\n
-Text Label 950  4100 0    60   ~ 0
-PI_RESET
-Wire Wire Line
-	950  4100 1600 4100
 Text Label 950  1600 0    60   ~ 0
 PI_RESET
 Wire Wire Line
 	950  1600 1600 1600
-Text Label 4000 4100 2    60   ~ 0
-ADI_RESET
-Wire Wire Line
-	3400 4100 4000 4100
 Text Label 950  1700 0    60   ~ 0
 ADI_RESET
@@
 Wire Wire Line
 	3400 2200 3950 2200
-Text Label 4000 3600 2    60   ~ 0
+Text Label 4000 2750 2    60   ~ 0
 ANA_OUT1
-Text Label 4000 3700 2    60   ~ 0
+Text Label 4000 2850 2    60   ~ 0
 ANA_OUT2
-Text Label 4000 3800 2    60   ~ 0
+Text Label 4000 2950 2    60   ~ 0
 ANA_OUT3
-Text Label 4000 3900 2    60   ~ 0
+Text Label 4000 3050 2    60   ~ 0
 ANA_OUT4
 Wire Wire Line
-	3400 3600 4000 3600
-Wire Wire Line
-	3400 3700 4000 3700
-Wire Wire Line
-	3400 3800 4000 3800
-Wire Wire Line
-	3400 3900 4000 3900
-Text Label 950  3600 0    60   ~ 0
+	3400 2750 4000 2750
+Wire Wire Line
+	3400 2850 4000 2850
+Wire Wire Line
+	3400 2950 4000 2950
+Wire Wire Line
+	3400 3050 4000 3050
+Text Label 950  2750 0    60   ~ 0
 ANA_IN1
-Text Label 950  3700 0    60   ~ 0
+Text Label 950  2850 0    60   ~ 0
 ANA_IN2
 Wire Wire Line
-	950  3600 1600 3600
-Wire Wire Line
-	1600 3700 950  3700
+	950  2750 1600 2750
+Wire Wire Line
+	1600 2850 950  2850
 Text Label 8550 5250 0    60   ~ 0
 MCLK1
@@
 Wire Wire Line
 	950  1950 1600 1950
-Text Label 950  3350 0    60   ~ 0
-MCLK2
-Wire Wire Line
-	950  3350 1600 3350
-Text Label 4000 3350 2    60   ~ 0
-MCLK3
-Wire Wire Line
-	4000 3350 3400 3350
 Text Label 950  1800 0    60   ~ 0
 GLB_RESET
 Wire Wire Line
 	950  1800 1600 1800
-Text Label 950  3450 0    60   ~ 0
-GLB_RESET
-Text Label 4000 3450 2    60   ~ 0
-GLB_RESET
-Wire Wire Line
-	4000 3450 3400 3450
-Wire Wire Line
-	950  3450 1600 3450
-$Sheet
-S 5750 1500 1500 1050
+$Sheet
+S 9250 900  1500 1050
 U 5574D2FB
 F0 "PSU" 60
@@
 $EndSheet
 $Sheet
-S 6100 3400 1650 800
+S 7150 1000 1650 800
 U 5574D5A4
 F0 "SPDIF" 60
 F1 "SPDIF.sch" 60
 $EndSheet
+$Sheet
+S 1600 3550 2050 2550
+U 55781C1C
+F0 "AD1937 CODEC" 60
+F1 "AD1937 CODEC.sch" 60
+F2 "CODECDAC_LRCLK" I L 1600 3650 60
+F3 "CODECDAC_BCLK" I L 1600 3750 60
+F4 "CODECDAC_SDATA0" I L 1600 3850 60
+F5 "CODECDAC_SDATA1" I L 1600 3950 60
+F6 "CODECDAC_SDATA2" I L 1600 4050 60
+F7 "CODECDAC_SDATA3" I L 1600 4150 60
+F8 "CODECADC_LRCLK" O R 3650 3650 60
+F9 "CODECADC_BCLK" O R 3650 3750 60
+F10 "CODECADC_SDATA0" O R 3650 3850 60
+F11 "CODECADC_SDATA1" O R 3650 3950 60
+F12 "I2C_SCL" B R 3650 4100 60
+F13 "I2C_SDA" B R 3650 4200 60
+F14 "DAC_OUT1_LP" O L 1600 4350 60
+F15 "CODEC_MCLK" I R 3650 4350 60
+F16 "ADC_IN1_LP" I R 3650 4500 60
+F17 "ADC_IN1_LN" I R 3650 4600 60
+F18 "ADC_IN2_LP" I R 3650 4950 60
+F19 "ADC_IN2_LN" I R 3650 5050 60
+F20 "ADC_IN1_RP" I R 3650 4700 60
+F21 "ADC_IN1_RN" I R 3650 4800 60
+F22 "ADC_IN2_RP" I R 3650 5150 60
+F23 "ADC_IN2_RN" I R 3650 5250 60
+F24 "DAC_OUT1_LN" O L 1600 4450 60
+F25 "DAC_OUT1_RP" O L 1600 4550 60
+F26 "DAC_OUT1_RN" O L 1600 4650 60
+F27 "DAC_OUT2_LP" O L 1600 4750 60
+F28 "DAC_OUT2_LN" O L 1600 4850 60
+F29 "DAC_OUT2_RP" O L 1600 4950 60
+F30 "DAC_OUT2_RN" O L 1600 5050 60
+F31 "DAC_OUT3_LP" O L 1600 5200 60
+F32 "DAC_OUT3_LN" O L 1600 5300 60
+F33 "DAC_OUT3_RP" O L 1600 5400 60
+F34 "DAC_OUT3_RN" O L 1600 5500 60
+F35 "DAC_OUT4_LP" O L 1600 5600 60
+F36 "DAC_OUT4_LN" O L 1600 5700 60
+F37 "DAC_OUT4_RP" O L 1600 5800 60
+F38 "DAC_OUT4_RN" O L 1600 5900 60
+F39 "CODEC_RST" I R 3650 5900 60
+$EndSheet
+$Sheet
+S 1600 2650 1800 550
+U 54E8D6A6
+F0 "Connectors" 60
+F1 "Connectors.sch" 60
+F22 "ANA_IN1" O L 1600 2750 60
+F23 "ANA_IN2" O L 1600 2850 60
+F24 "ANA_OUT1" I R 3400 2750 60
+F25 "ANA_OUT2" I R 3400 2850 60
+F26 "ANA_OUT3" I R 3400 2950 60
+F27 "ANA_OUT4" I R 3400 3050 60
+$EndSheet
+Text Label 4200 3650 2    60   ~ 0
+IN_LRCLK0
+Text Label 4200 3750 2    60   ~ 0
+IN_BCLK0
+Text Label 4200 3850 2    60   ~ 0
+IN_SDATA0
+Text Label 4200 3950 2    60   ~ 0
+IN_SDATA1
+Wire Wire Line
+	4200 3650 3650 3650
+Wire Wire Line
+	3650 3750 4200 3750
+Wire Wire Line
+	4200 3850 3650 3850
+Wire Wire Line
+	3650 3950 4200 3950
+Text Label 1000 3650 0    60   ~ 0
+OUT_LRCLK0
+Text Label 1000 3750 0    60   ~ 0
+OUT_BCLK0
+Text Label 1000 3850 0    60   ~ 0
+OUT_SDATA0
+Wire Wire Line
+	1600 3650 1000 3650
+Wire Wire Line
+	1000 3750 1600 3750
+Wire Wire Line
+	1600 3850 1000 3850
+Text Label 1000 3950 0    60   ~ 0
+OUT_SDATA1
+Wire Wire Line
+	1600 3950 1000 3950
+Text Label 1000 4050 0    60   ~ 0
+OUT_SDATA2
+Wire Wire Line
+	1600 4050 1000 4050
+Text Label 1000 4150 0    60   ~ 0
+OUT_SDATA3
+Wire Wire Line
+	1600 4150 1000 4150
+Text Label 4200 4350 2    60   ~ 0
+MCLK2
+Wire Wire Line
+	4200 4350 3650 4350
+Text Label 4200 5900 2    60   ~ 0
+GLB_RESET
+Wire Wire Line
+	3650 5900 4200 5900
 $EndSCHEMATC

Commit message: WIP
Changed lines of the file:
@@
 LIBS:power
 LIBS:OHDSP-Lib
+LIBS:OHDSP-XOVER-cache
 EELAYER 25 0
 EELAYER END
 $Descr A4 11693 8268
 encoding utf-8
-Sheet 1 7
+Sheet 1 9
 Title ""
 Date "10 feb 2015"
@@
 F38 "DAC_OUT4_RN" O L 1600 5900 60
 F39 "CODEC_RST" I R 3650 5900 60
+F40 "AD1937_CM" O R 3650 5550 60
 $EndSheet
 $Sheet
@@
 F0 "Connectors" 60
 F1 "Connectors.sch" 60
-F22 "ANA_IN1" O L 1600 2750 60
-F23 "ANA_IN2" O L 1600 2850 60
-F24 "ANA_OUT1" I R 3400 2750 60
-F25 "ANA_OUT2" I R 3400 2850 60
-F26 "ANA_OUT3" I R 3400 2950 60
-F27 "ANA_OUT4" I R 3400 3050 60
+F2 "ANA_IN1" O L 1600 2750 60
+F3 "ANA_IN2" O L 1600 2850 60
+F4 "ANA_OUT1" I R 3400 2750 60
+F5 "ANA_OUT2" I R 3400 2850 60
+F6 "ANA_OUT3" I R 3400 2950 60
+F7 "ANA_OUT4" I R 3400 3050 60
 $EndSheet
 Text Label 4200 3650 2    60   ~ 0
@@
 Wire Wire Line
 	3650 5900 4200 5900
+$Sheet
+S 6500 2400 1800 1300
+U 55785217
+F0 "AD1937_AnaIn" 60
+F1 "AD1937_AnaIn.sch" 60
+$EndSheet
+$Sheet
+S 5600 4250 2200 1550
+U 557A1433
+F0 "AD1937_DigiOut_1To4" 60
+F1 "AD1937_DigiOut_1To4.sch" 60
+$EndSheet
 $EndSCHEMATC

Commit message: WIP
Other:
- note added: "12 Opamps"
- note added: "4 Opamps"
- note added: "5 Opamps"
- note added: "Total 33 Opamps - 13 Singles - 20 Dual - \nAssume OPA134/OPA2134 - \nMax 5mA per opamp - +/-12V current (per rail) is 165mA"

Commit message: WIP
Changed lines of the file:
@@
 $Descr A4 11693 8268
 encoding utf-8
-Sheet 1 10
+Sheet 1 9
 Title ""
 Date "10 feb 2015"
@@
 $EndSheet
 $Sheet
-S 7150 1000 1650 800
-U 5574D5A4
-F0 "SPDIF" 60
-F1 "SPDIF.sch" 60
-$EndSheet
-$Sheet

Commit message: WIP
Changed lines of the file:
@@
 $Descr A4 11693 8268
 encoding utf-8
-Sheet 1 9
+Sheet 1 10
 Title ""
 Date "10 feb 2015"
@@
 $EndDescr
 $Sheet
-S 1600 800  1800 1550
+S 1600 800  1800 1650
 U 54BE4270
 F0 "ADAU1701" 50
@@
 F12 "DACOUT_SDATA2" O R 3400 1300 60
 F13 "DACOUT_SDATA3" O R 3400 1400 60
-F14 "I2C_SCL" B R 3400 1600 60
-F15 "I2C_SDA" B R 3400 1700 60
-F16 "DAC_VOUT0" O R 3400 1900 60
+F14 "I2C_SCL" B R 3400 1550 60
+F15 "I2C_SDA" B R 3400 1650 60
+F16 "DAC_VOUT0" O R 3400 1800 60
 F17 "RST_OUT" O L 1600 1800 60
 F18 "RST_IN1" I L 1600 1700 60
-F19 "DAC_VOUT1" O R 3400 2000 60
-F20 "DAC_VOUT2" O R 3400 2100 60
-F21 "DAC_VOUT3" O R 3400 2200 60
+F19 "DAC_VOUT1" O R 3400 1900 60
+F20 "DAC_VOUT2" O R 3400 2000 60
+F21 "DAC_VOUT3" O R 3400 2100 60
 F22 "ADC_IN0" I L 1600 2100 60
 F23 "ADC_IN1" I L 1600 2200 60
 F24 "RST_IN2" I L 1600 1600 60
 F25 "MCLK" I L 1600 1950 60
+F26 "SELFBOOT_WP" I R 3400 2350 60
+F27 "SELFBOOT_EN" I R 3400 2250 60
 $EndSheet
 $Sheet
@@
 Wire Wire Line
 	3400 1400 4000 1400
-Text Label 3650 1700 2    60   ~ 0
+Text Label 3650 1650 2    60   ~ 0
 SDA
-Text Label 3650 1600 2    60   ~ 0
+Text Label 3650 1550 2    60   ~ 0
 SCL
 Wire Wire Line
-	3400 1700 3650 1700
-Wire Wire Line
-	3400 1600 3650 1600
+	3400 1650 3650 1650
+Wire Wire Line
+	3400 1550 3650 1550
 Text Label 7450 4250 2    60   ~ 0
 SDA
@@
 Wire Wire Line
 	1600 2200 950  2200
+Text Label 3950 1800 2    60   ~ 0
+ANA_OUT1
 Text Label 3950 1900 2    60   ~ 0
-ANA_OUT1
+ANA_OUT2
 Text Label 3950 2000 2    60   ~ 0
-ANA_OUT2
+ANA_OUT3
 Text Label 3950 2100 2    60   ~ 0
-ANA_OUT3
-Text Label 3950 2200 2    60   ~ 0
 ANA_OUT4
 Wire Wire Line
+	3400 1800 3950 1800
+Wire Wire Line
 	3400 1900 3950 1900
 Wire Wire Line
@@
 Wire Wire Line
 	3400 2100 3950 2100
-Wire Wire Line
-	3400 2200 3950 2200
 Text Label 4000 2750 2    60   ~ 0
 ANA_OUT1
@@
 Text Notes 700  7150 0    60   ~ 0
 Total 33 Opamps - 13 Singles - 20 Dual - \nAssume OPA134/OPA2134 - \nMax 5mA per opamp - +/-12V current (per rail) is 165mA
+$Sheet
+S 5100 1450 1750 1350
+U 55787687
+F0 "ATmega32U4" 60
+F1 "ATmega32U4.sch" 60
+$EndSheet
 $EndSCHEMATC
