File: Schematics/PSU.sch (KiCad schematic (older format))
At the start: 51 parts, among them P301 PIN, P302 PIN, P303 PIN, P305 CONN_2x1, P306 PIN, U301 IC-REG-XRP7659ISTR-F, U303 XC6222D331MR-G

Commit message: WIP
Other:
- note added: "12V to 15V Input"
- note added: "External Power"
- note removed: "Power from Pi or External"
- note removed: "Two sets of screw terminals\nOne for 5V-16V self power\nOne set for 5V - will power the Pi as well\nDo not put 16V up the Pi!"
- moved on the sheet: C307, C308, C310, C311, D302, D305, L301, P301, P302, P303, P305, P306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

Commit message: WIP
Parts:
- added D? (x2): SS24T3G, OHDSP-Footprints-Pretty:DIODE-SMB, symbol DIODE
- added P? (x2): CONN_2x1, OHDSP-Footprints-Pretty:CONN-SCREW-2WAY-5mm-5.08mm, symbol CONN_2x1
Connections:
- net GNDD: now also P?.1 (P1), P?.2 (P2)
- new net: D?.1 (A), P?.1 (P1)
- new net: D?.2 (K), P?.2 (P2)
Changed lines of the file:
@@
 $Descr A4 11693 8268
 encoding utf-8
-Sheet 4 9
+Sheet 4 10
 Title ""
 Date "10 feb 2015"
@@
 	3900 2100 3900 1800
 Wire Wire Line
-	3550 1800 3900 1800
-Wire Wire Line
-	3900 1800 4150 1800
-Wire Wire Line
-	4150 1800 4250 1800
+	3550 1800 4250 1800
 Connection ~ 3900 1800
 Wire Wire Line
@@
 Connection ~ 4150 1800
 Wire Wire Line
-	5350 1800 5350 1900
-Wire Wire Line
-	5350 1900 5350 2000
+	5350 1800 5350 2000
 Connection ~ 5350 1900
 Wire Wire Line
-	4950 2500 4950 2550
-Wire Wire Line
-	4950 2550 4950 2600
+	4950 2500 4950 2600
 Wire Wire Line
 	4950 2550 4250 2550
@@
 	1000 1850 1000 1600
 Wire Wire Line
-	900  1600 1000 1600
-Wire Wire Line
-	1000 1600 1350 1600
-Wire Wire Line
-	1350 1600 1500 1600
-Wire Wire Line
-	1500 1600 2150 1600
+	900  1600 2150 1600
 Connection ~ 1000 1600
 Wire Wire Line
@@
 	7700 1800 7700 1950
 Wire Wire Line
-	4850 1800 5350 1800
-Wire Wire Line
-	5350 1800 5850 1800
-Wire Wire Line
-	5850 1800 6350 1800
-Wire Wire Line
-	6350 1800 6900 1800
-Wire Wire Line
-	6900 1800 7150 1800
-Wire Wire Line
-	7150 1800 7400 1800
-Wire Wire Line
-	7400 1800 7700 1800
-Wire Wire Line
-	7700 1800 7850 1800
-Wire Wire Line
-	7850 1800 8550 1800
+	4850 1800 8550 1800
 Wire Wire Line
 	7400 1950 7400 1800
@@
 Connection ~ 7400 1800
 Wire Wire Line
-	10650 1700 10650 1800
-Wire Wire Line
-	10650 1800 10650 1900
-Wire Wire Line
-	9900 1800 10150 1800
-Wire Wire Line
-	10150 1800 10300 1800
-Wire Wire Line
-	10300 1800 10400 1800
-Wire Wire Line
-	10400 1800 10650 1800
+	10650 1700 10650 1900
+Wire Wire Line
+	9900 1800 10650 1800
 Wire Wire Line
 	10150 1900 10150 1800
@@
 	5850 2450 5850 2400
 Wire Wire Line
-	7400 2350 7400 2400
-Wire Wire Line
-	7400 2400 7400 2450
+	7400 2350 7400 2450
 Wire Wire Line
 	7700 2400 7700 2350
 Connection ~ 7400 2400
 Wire Wire Line
-	10650 2300 10650 2400
-Wire Wire Line
-	10650 2400 10650 2450
-Wire Wire Line
-	10000 2400 10150 2400
-Wire Wire Line
-	10150 2400 10400 2400
-Wire Wire Line
-	10400 2400 10650 2400
+	10650 2300 10650 2450
+Wire Wire Line
+	10000 2400 10650 2400
 Wire Wire Line
 	10400 2400 10400 2300
@@
 Connection ~ 1500 1600
 Wire Wire Line
-	8400 2000 8450 2000
-Wire Wire Line
-	8450 2000 8550 2000
+	8400 2000 8550 2000
 Connection ~ 7850 1800
 Wire Wire Line
@@
 	3850 3550 3850 3450
 Wire Wire Line
-	2950 3550 3200 3550
-Wire Wire Line
-	3200 3550 3650 3550
-Wire Wire Line
-	3650 3550 3850 3550
-Wire Wire Line
-	3850 3550 4050 3550
-Wire Wire Line
-	4050 3550 4400 3550
+	2950 3550 4400 3550
 Text Notes 700  3150 0    118  ~ 0
 External Power
@@
 $EndComp
 Wire Wire Line
-	3650 4050 3650 4100
-Wire Wire Line
-	3650 4100 3650 4150
-Wire Wire Line
-	3650 4100 4050 4100
-Wire Wire Line
-	4050 4100 4400 4100
+	3650 4050 3650 4150
+Wire Wire Line
+	3650 4100 4400 4100
 Wire Wire Line
 	4050 4100 4050 4050
@@
 Connection ~ 7400 5050
 Wire Wire Line
-	10650 4950 10650 5050
-Wire Wire Line
-	10650 5050 10650 5150
-Wire Wire Line
-	9900 5050 10150 5050
-Wire Wire Line
-	10150 5050 10300 5050
-Wire Wire Line
-	10300 5050 10400 5050
-Wire Wire Line
-	10400 5050 10650 5050
+	10650 4950 10650 5150
+Wire Wire Line
+	9900 5050 10650 5050
 Wire Wire Line
 	10150 5150 10150 5050
@@
 Connection ~ 10400 5050
 Wire Wire Line
-	7400 5600 7400 5650
-Wire Wire Line
-	7400 5650 7400 5700
+	7400 5600 7400 5700
 Wire Wire Line
 	7700 5650 7700 5600
 Connection ~ 7400 5650
 Wire Wire Line
-	10650 5550 10650 5650
-Wire Wire Line
-	10650 5650 10650 5700
-Wire Wire Line
-	10000 5650 10150 5650
-Wire Wire Line
-	10150 5650 10400 5650
-Wire Wire Line
-	10400 5650 10650 5650
+	10650 5550 10650 5700
+Wire Wire Line
+	10000 5650 10650 5650
 Wire Wire Line
 	10400 5650 10400 5550
@@
 Connection ~ 10150 5650
 Wire Wire Line
-	8400 5250 8450 5250
-Wire Wire Line
-	8450 5250 8550 5250
+	8400 5250 8550 5250
 Connection ~ 7850 5050
 Connection ~ 10650 5050
@@
 	7900 5250 7850 5250
 Wire Wire Line
-	7850 5050 7850 5250
+	7850 5250 7850 5050
 Wire Wire Line
 	8450 5900 8450 5850
@@
 $EndComp
 Wire Wire Line
-	6900 5050 7400 5050
-Wire Wire Line
-	7400 5050 7700 5050
-Wire Wire Line
-	7700 5050 7850 5050
-Wire Wire Line
-	7850 5050 8550 5050
-Wire Wire Line
-	6900 5050 6900 3300
-Wire Wire Line
-	6900 3300 6900 1800
+	6900 5050 8550 5050
+Wire Wire Line
+	6900 1800 6900 5050
 Connection ~ 6900 1800
 $Comp
@@
 	7700 3300 7700 3450
 Wire Wire Line
-	6900 3300 7400 3300
-Wire Wire Line
-	7400 3300 7700 3300
-Wire Wire Line
-	7700 3300 7850 3300
-Wire Wire Line
-	7850 3300 8550 3300
+	6900 3300 8550 3300
 Wire Wire Line
 	7400 3450 7400 3300
@@
 Connection ~ 7400 3300
 Wire Wire Line
-	10650 3200 10650 3300
-Wire Wire Line
-	10650 3300 10650 3400
-Wire Wire Line
-	9900 3300 10150 3300
-Wire Wire Line
-	10150 3300 10300 3300
-Wire Wire Line
-	10300 3300 10400 3300
-Wire Wire Line
-	10400 3300 10650 3300
+	10650 3200 10650 3400
+Wire Wire Line
+	9900 3300 10650 3300
 Wire Wire Line
 	10150 3400 10150 3300
@@
 Connection ~ 10400 3300
 Wire Wire Line
-	7400 3850 7400 3900
-Wire Wire Line
-	7400 3900 7400 3950
+	7400 3850 7400 3950
 Wire Wire Line
 	7700 3900 7700 3850
 Connection ~ 7400 3900
 Wire Wire Line
-	10650 3800 10650 3900
-Wire Wire Line
-	10650 3900 10650 3950
-Wire Wire Line
-	10000 3900 10150 3900
-Wire Wire Line
-	10150 3900 10400 3900
-Wire Wire Line
-	10400 3900 10650 3900
+	10650 3800 10650 3950
+Wire Wire Line
+	10000 3900 10650 3900
 Wire Wire Line
 	10400 3900 10400 3800
@@
 Connection ~ 10150 3900
 Wire Wire Line
-	8400 3500 8450 3500
-Wire Wire Line
-	8450 3500 8550 3500
+	8400 3500 8550 3500
 Connection ~ 7850 3300
 Connection ~ 10650 3300
@@
 Text Notes 700  3350 0    60   ~ 0
 12V to 15V Input
+$Comp
+L CONN_2x1 P?
+U 1 1 558024D3
+P 1150 5550
+F 0 "P?" V 1645 5395 40  0000 C CNN
+F 1 "CONN_2x1" V 1590 5510 40  0000 C CNN
+F 2 "OHDSP-Footprints-Pretty:CONN-SCREW-2WAY-5mm-5.08mm" H 1490 5440 60  0001 C CNN
+F 3 "" H 1490 5440 60  0000 C CNN
+	1    1150 5550
+	-1   0    0    -1
+$EndComp
+$Comp
+L CONN_2x1 P?
+U 1 1 5580257D
+P 1150 6250
+F 0 "P?" V 1645 6095 40  0000 C CNN
+F 1 "CONN_2x1" V 1590 6210 40  0000 C CNN
+F 2 "OHDSP-Footprints-Pretty:CONN-SCREW-2WAY-5mm-5.08mm" H 1490 6140 60  0001 C CNN
+F 3 "" H 1490 6140 60  0000 C CNN
+	1    1150 6250
+	-1   0    0    -1
+$EndComp
+$Comp
+L DIODE D?
+U 1 1 55802637
+P 1600 5550
+F 0 "D?" H 1600 5650 40  0000 C CNN
+F 1 "SS24T3G" H 1600 5450 40  0000 C CNN
+F 2 "OHDSP-Footprints-Pretty:DIODE-SMB" H 1600 5550 60  0001 C CNN
+F 3 "" H 1600 5550 60  0000 C CNN
+	1    1600 5550
+	1    0    0    -1
+$EndComp
+$Comp
+L DIODE D?
+U 1 1 558026E9
+P 1600 6350
+F 0 "D?" H 1600 6450 40  0000 C CNN
+F 1 "SS24T3G" H 1600 6250 40  0000 C CNN
+F 2 "OHDSP-Footprints-Pretty:DIODE-SMB" H 1600 6350 60  0001 C CNN
+F 3 "" H 1600 6350 60  0000 C CNN
+	1    1600 6350
+	-1   0    0    1
+$EndComp
+Wire Wire Line
+	1150 5550 1400 5550
+Wire Wire Line
+	1150 5650 1250 5650
+Wire Wire Line
+	1250 5650 1250 6250
+Wire Wire Line
+	1250 6250 1150 6250
+Wire Wire Line
+	1400 6350 1150 6350
+$Comp
+L GNDD #PWR?
+U 1 1 55802D2A
+P 1400 5950
+F 0 "#PWR?" H 1400 5700 60  0001 C CNN
+F 1 "GNDD" H 1400 5800 60  0000 C CNN
+F 2 "" H 1400 5950 60  0000 C CNN
+F 3 "" H 1400 5950 60  0000 C CNN
+	1    1400 5950
+	1    0    0    -1
+$EndComp
+Wire Wire Line
+	1400 5950 1400 5850
+Wire Wire Line
+	1400 5850 1250 5850
+Connection ~ 1250 5850
 $EndSCHEMATC

Commit message: WIP
Parts:
- removed D302: SS24T3G, OHDSP-Footprints-Pretty:DIODE-SMB, symbol DIODE
- added C? (x4): 1000u, OHDSP-Footprints-Pretty:CAP-TH-D6.3mmP2.5mm, symbol CP1
- added C? (x6): 10n, OHDSP-Footprints-Pretty:SMD-0805, symbol C
- added C? (x4): 220u, OHDSP-Footprints-Pretty:CAP-TH-D6.3mmP2.5mm, symbol CP1
- added D? (x5): 1N4001, OHDSP-Footprints-Pretty:DIODE-SMB, symbol DIODE
- added R? (x2): 120R, OHDSP-Footprints-Pretty:SMD-0805, symbol R
- added R? (x2): 1k, OHDSP-Footprints-Pretty:SMD-0805, symbol R
- added R? (x2): 1R, OHDSP-Footprints-Pretty:SMD-0805, symbol R
- added U?: IC-REG-LM317AT, TO-220, symbol IC-REG-LM317AT
- added U?: IC-REG-LM337-TO220, TO-220, symbol IC-REG-LM337-TO220
- D? (x2): value SS24T3G -> 1N4001
Connections:
- net GNDD: now also C?.1, C?.1, C?.1, C?.1, C?.1, C?.1, C?.1, C?.1, C?.2, C?.2, C?.2, C?.2, C?.2, C?.2, D?.1 (A), D?.2 (K), R?.1, R?.1
- net at P305.1 (P1): now also D?.1 (A)
- net at L301.1: now also D?.2 (K)
- net at D?.2 (K): now also C?.1, R?.2
- net at D?.1 (A): now also C?.2, R?.2
- new net: C?.1, C?.2, R?.2, R?.2, U?.1 (ADJ)
- new net: C?.1, C?.2, D?.2 (K), R?.1, U?.3 (IN)
- new net: C?.1, C?.2, R?.1, R?.2, U?.1 (ADJ)
- new net: C?.2, C?.2, D?.1 (A), R?.1, U?.2 (IN)
- new net +12VA: C?.1, C?.1, D?.1 (A), D?.2 (K), R?.1, U?.2 (OUT)
- new net -12VA: C?.2, C?.2, D?.1 (A), D?.2 (K), R?.2, U?.3 (OUT)
Other:
- moved on the sheet: C319, C321, C323, C325, C327, C329, C?, D?, P301, P302, P303, P306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

Commit message: WIP
Parts:
- added C428, C444: 22u, OHDSP-Footprints-Pretty:SMD-0805, symbol C
- added C432, C440: 100n, OHDSP-Footprints-Pretty:SMD-0805, symbol C
- added C436: 1u, OHDSP-Footprints-Pretty:SMD-0805, symbol C
- added C448: 220u, OHDSP-Footprints-Pretty:CAP-TH-D6.3mmP2.5mm, symbol CP1
- added R416: 100k, OHDSP-Footprints-Pretty:SMD-0805, symbol R
- added U407: XC6222D331MR-G, OHDSP-Footprints-Pretty:IC-SOT25, symbol IC-REG-XC6210B332MR
- C403, C404, C405, C406, C419, C420: renamed from C?; footprint OHDSP-Footprints-Pretty:CAP-TH-D6.3mmP2.5mm -> OHDSP-Footprints-Pretty:CAP-TH-D12.5mmP5mm
- C407, C408, C413, C415, C422, C423: renamed from C?; footprint OHDSP-Footprints-Pretty:SMD-0805 -> OHDSP-Footprints-Pretty:CAP_TH_5mm
- C410, C411: renamed from C?; footprint OHDSP-Footprints-Pretty:CAP-TH-D6.3mmP2.5mm -> OHDSP-Footprints-Pretty:CAP-TH-D10mmP5mm
- C412: renamed from C308; footprint OHDSP-Footprints-Pretty:CAP-TH-D6.3mmP2.5mm -> OHDSP-Footprints-Pretty:CAP-TH-D12.5mmP5mm
- D401, D402, D403, D405, D406, D407, D408: renamed from D?; footprint OHDSP-Footprints-Pretty:DIODE-SMB -> OHDSP-Footprints-Pretty:DIODE-DO-41
- U402, U403: renamed from U?; footprint TO-220 -> OHDSP-Footprints-Pretty:IC-TO220
- gave numbers to parts that had none: 24
- renumbered C303 to C401, C305 to C402, C307 to C409, C309 to C414, C310 to C416, C311 to C417, C314 to C418, C316 to C421, C318 to C424, C319 to C425, C321 to C429, C323 to C433, C325 to C437, C327 to C441, C329 to C445, D303 to D404, D305 to D409, L301 to L401, L302 to L402, P305 to P401, P301 to P404, P302 to P405, P303 to P406, P306 to P407, R302 to R401, R303 to R404, R306 to R407, R307 to R408, R308 to R409, R309 to R412, R310 to R413, U301 to U401, U303 to U404
Connections:
- net GNDD: now also C428.2, C432.2, C436.2, C440.2, C444.2, C448.2, U407.2 (VSS)
- net at C418.1, C421.1, C424.1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: now also C428.1, C432.1, R416.1, U407.1 (VIN); no longer C427.1, C431.1, R415.1, U406.1 (VIN)
- new net: C427.1, C431.1, R415.1, U406.1 (VIN)
- new net: C436.1, R416.2, U407.3 (CE)
- new net VMEM: C440.1, C444.1, C448.1, U407.5 (VOUT)
- no-connect marks 3 -> 4
Other:
- note added: "Atmel 3v3"
